Commit message: adapt

File: src/b166er_robot/urdf/pioneer3at/pioneer3at.urdf (robot description, URDF)
Before this commit: robot pioneer_3at, 8 links, 7 joints
Links:
- removed link camera_mount
- removed link front_left_wheel
- removed link front_right_wheel
- removed link front_sonar_array
- removed link laser_mount
- removed link rear_left_wheel
- removed link rear_right_wheel
- added link back_sonar, mass 0.1; visual mesh filename=package://amr_robots_description/meshes/p3at_meshes/back_so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
- added link front_sonar, mass 0.1; visual mesh filename=package://amr_robots_description/meshes/p3at_meshes/front_s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
- added link p3at_back_left_axle, mass 0.1; collision mesh filename=package://amr_robots_description/meshes/p3at_meshes/axle.stl; visual mesh filename=package://amr_robots_description/meshes/p3at_meshes/axle.stl
- added link p3at_back_left_hub, mass 0.1; collision mesh filename=package://amr_robots_description/meshes/p3at_meshes/left_hu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; visual mesh filename=package://amr_robots_description/meshes/p3at_meshes/left_hu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
- added link p3at_back_left_wheel, mass 1.2; collision cylinder length=0.075 radius=0.111; visual mesh filename=package://amr_robots_description/meshes/p3at_meshes/wheel.s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
- added link p3at_back_right_axle, mass 0.1; collision mesh filename=package://amr_robots_description/meshes/p3at_meshes/axle.stl; visual mesh filename=package://amr_robots_description/meshes/p3at_meshes/axle.stl
- added link p3at_back_right_hub, mass 0.1; collision mesh filename=package://amr_robots_description/meshes/p3at_meshes/right_h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; visual mesh filename=package://amr_robots_description/meshes/p3at_meshes/right_h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
- added link p3at_back_right_wheel, mass 1.2; collision cylinder length=0.075 radius=0.111; visual mesh filename=package://amr_robots_description/meshes/p3at_meshes/wheel.s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
- added link p3at_front_left_axle, mass 0.1; visual mesh filename=package://amr_robots_description/meshes/p3at_meshes/axle.stl
- added link p3at_front_left_hub, mass 0.1; visual mesh filename=package://amr_robots_description/meshes/p3at_meshes/left_hu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
- added link p3at_front_left_wheel, mass 1.2; collision cylinder length=0.075 radius=0.111; visual mesh filename=package://amr_robots_description/meshes/p3at_meshes/wheel.s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
- added link p3at_front_right_axle, mass 0.1; visual mesh filename=package://amr_robots_description/meshes/p3at_meshes/axle.stl
- added link p3at_front_right_hub, mass 0.1; visual mesh filename=package://amr_robots_description/meshes/p3at_meshes/right_h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
- added link p3at_front_right_wheel, mass 1.2; collision cylinder length=0.075 radius=0.111; visual mesh filename=package://amr_robots_description/meshes/p3at_meshes/wheel.s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
- added link top_plate, mass 0.1; visual mesh filename=package://amr_robots_description/meshes/p3at_meshes/top.stl
- link base_link: mass 16.0 -> 21.5; geometry collision mesh filename=package://amr_robots_description/meshes/p3at_meshes/chassis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; visual mesh filename=package://amr_robots_description/meshes/p3at_meshes/chassis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
Joints:
- removed joint camera_mount_joint
- removed joint front_left_wheel_joint
- removed joint front_right_wheel_joint
- removed joint front_sonar_joint
- removed joint laser_mount_joint
- removed joint rear_left_wheel_joint
- removed joint rear_right_wheel_joint
- added joint base_back_joint: type fixed, parent base_link, child back_sonar, origin xyz=-0.187 0 0.247 rpy=0 0 0
- added joint base_front_joint: type fixed, parent base_link, child front_sonar, origin xyz=0.193 0 0.25 rpy=0 0 0
- added joint base_front_left_axle_joint: type fixed, parent base_link, child p3at_front_left_axle, origin xyz=0.135 0.156 0.111 rpy=0 0 0
- added joint base_front_left_hub_joint: type fixed, parent p3at_front_left_axle, child p3at_front_left_hub, origin xyz=0 0.041 0 rpy=0 0 0
- added joint base_front_right_axle_joint: type fixed, parent base_link, child p3at_front_right_axle, origin xyz=0.135 -0.156 0.111 rpy=0 0 0
- added joint base_front_right_hub_joint: type fixed, parent p3at_front_right_axle, child p3at_front_right_hub, origin xyz=0 -0.041 0 rpy=0 0 0
- added joint base_top_joint: type fixed, parent base_link, child top_plate, origin xyz=0.003 0 0.274 rpy=0 0 0
- added joint p3at_back_left_axle_joint: type fixed, parent base_link, child p3at_back_left_axle, origin xyz=-0.134 0.156 0.111 rpy=0 0 0
- added joint p3at_back_left_hub_joint: type fixed, parent p3at_back_left_axle, child p3at_back_left_hub, origin xyz=-0 0.041 0 rpy=0 0 0
- added joint p3at_back_left_wheel_joint: type continuous, parent p3at_back_left_hub, child p3at_back_left_wheel, origin xyz=0 0 0 rpy=0 0 0, axis 0 1 0, limit effort=100 velocity=100
- added joint p3at_back_right_axle_joint: type fixed, parent base_link, child p3at_back_right_axle, origin xyz=-0.134 -0.156 0.111 rpy=0 0 0
- added joint p3at_back_right_hub_joint: type fixed, parent p3at_back_right_axle, child p3at_back_right_hub, origin xyz=-0 -0.041 0 rpy=0 0 0
- added joint p3at_back_right_wheel_joint: type continuous, parent p3at_back_right_hub, child p3at_back_right_wheel, origin xyz=0 0 0 rpy=0 0 0, axis 0 1 0, limit effort=100 velocity=100
- added joint p3at_front_left_wheel_joint: type continuous, parent p3at_front_left_hub, child p3at_front_left_wheel, origin xyz=0 0 0 rpy=0 0 0, axis 0 1 0, limit effort=100 velocity=100
- added joint p3at_front_right_wheel_joint: type continuous, parent p3at_front_right_hub, child p3at_front_right_wheel, origin xyz=0 0 0 rpy=0 0 0, axis 0 1 0, limit effort=100 velocity=100
