Commit message: fix(sim): corrige malhas do Pioneer e a config do RViz
O xacro do Pioneer referenciava package://pioneer3at_simulation/meshes/,
um pacote que não existe neste workspace (resquício do template de
origem) — isso fazia o chassi/rodas falharem ao carregar no RobotModel
do RViz. Corrigido para package://b166er_robot/meshes/pioneer3at/,
onde as malhas realmente estão.

Também corrige config/b166er.rviz: o QMainWindow State (blob binário
do Qt) estava corrompido por uma edição manual anterior, escondendo os
painéis Displays/Views; removido para usar o layout padrão. O TF
Marker Scale estava em 1 metro (gigante para este robô), cobrindo o
modelo com setas/rótulos sobrepostos — reduzido para 0.15.

Confirmado visualmente no RViz: chassi vermelho, rodas com aro
dourado, torre e braço na postura correta, batendo com foto do robô
real.

Co-Authored-By: Claude Sonnet 4.6 <noreply@anthropic.com>

File: src/b166er_robot/urdf/pioneer3at/pioneer3at-m.urdf.xacro (robot description, xacro)
@@ -22,5 +22,5 @@
       <origin xyz="0 0 0.177" rpy="0 0 0"/>
       <geometry name="pioneer_geom">
-        <mesh filename="package://pioneer3at_simulation/meshes/chassis.stl"/>
+        <mesh filename="package://b166er_robot/meshes/pioneer3at/chassis.stl"/>
       </geometry>
       <material name="ChassisRed">
@@ -31,5 +31,5 @@
       <origin xyz="0 0 0.177" rpy="0 0 0"/>
       <geometry>
-        <mesh filename="package://pioneer3at_simulation/meshes/chassis.stl"/>
+        <mesh filename="package://b166er_robot/meshes/pioneer3at/chassis.stl"/>
       </geometry>
     </collision>
@@ -55,5 +55,5 @@
       <origin xyz="0 0 0" rpy="0 0 0"/>
       <geometry name="pioneer_geom">
-        <mesh filename="package://pioneer3at_simulation/meshes/top.stl"/>
+        <mesh filename="package://b166er_robot/meshes/pioneer3at/top.stl"/>
       </geometry>
       <material name="TopBlack">
@@ -86,5 +86,5 @@
       <origin xyz="0 0 0" rpy="0 0 0"/>
       <geometry name="pioneer_geom">
-        <mesh filename="package://pioneer3at_simulation/meshes/front_sonar.stl"/>
+        <mesh filename="package://b166er_robot/meshes/pioneer3at/front_sonar.stl"/>
       </geometry>
       <material name="SonarYellow">
@@ -111,5 +111,5 @@
       <origin xyz="0 0 0" rpy="0 0 0"/>
       <geometry name="pioneer_geom">
-        <mesh filename="package://pioneer3at_simulation/meshes/back_sonar.stl"/>
+        <mesh filename="package://b166er_robot/meshes/pioneer3at/back_sonar.stl"/>
       </geometry>
       <material name="SonarYellow">
@@ -138,5 +138,5 @@
         <origin xyz="0 0 0" rpy="0 0 0"/>
         <geometry name="pioneer_geom">
-          <mesh filename="package://pioneer3at_simulation/meshes/axle.stl"/>
+          <mesh filename="package://b166er_robot/meshes/pioneer3at/axle.stl"/>
         </geometry>
         <material name="AxleGrey">
@@ -162,5 +162,5 @@
         <origin xyz="0 0 0" rpy="0 0 0"/>
         <geometry name="pioneer_geom">
-          <mesh filename="package://pioneer3at_simulation/meshes/${side}_hubcap.stl"/>
+          <mesh filename="package://b166er_robot/meshes/pioneer3at/${side}_hubcap.stl"/>
         </geometry>
         <material name="HubcapYellow">
@@ -192,5 +192,5 @@
         <origin xyz="0 0 0" rpy="0 0 0"/>
         <geometry name="pioneer_geom">
-          <mesh filename="package://pioneer3at_simulation/meshes/wheel.stl" scale="0.75 0.66 0.75"/>
+          <mesh filename="package://b166er_robot/meshes/pioneer3at/wheel.stl" scale="0.75 0.66 0.75"/>
         </geometry>
         <material name="WheelBlack">
@@ -201,5 +201,5 @@
         <origin xyz="0 0 0" rpy="${-3.1415927/2} 0 0"/>
         <geometry>
-          <!--mesh filename="package://pioneer3at_simulation/meshes/wheel.stl"/-->
+          <!--mesh filename="package://b166er_robot/meshes/pioneer3at/wheel.stl"/-->
           <cylinder radius="0.085" length="0.05"/>
         </geometry>
@@ -229,5 +229,5 @@
         <origin xyz="0 0 0" rpy="0 0 0"/>
         <geometry name="pioneer_geom">
-          <mesh filename="package://pioneer3at_simulation/meshes/axle.stl"/>
+          <mesh filename="package://b166er_robot/meshes/pioneer3at/axle.stl"/>
         </geometry>
         <material name="AxleGrey">
@@ -238,5 +238,5 @@
         <origin xyz="0 0 0" rpy="0 0 0"/>
         <geometry>
-          <mesh filename="package://pioneer3at_simulation/meshes/axle.stl"/>
+          <mesh filename="package://b166er_robot/meshes/pioneer3at/axle.stl"/>
         </geometry>
       </collision>
@@ -259,5 +259,5 @@
         <origin xyz="0 0 0" rpy="0 0 0"/>
         <geometry name="pioneer_geom">
-          <mesh filename="package://pioneer3at_simulation/meshes/${side}_hubcap.stl"/>
+          <mesh filename="package://b166er_robot/meshes/pioneer3at/${side}_hubcap.stl"/>
         </geometry>
         <material name="HubcapYellow"/>
@@ -266,5 +266,5 @@
         <origin xyz="0 0 0" rpy="0 0 0"/>
         <geometry>
-          <mesh filename="package://pioneer3at_simulation/meshes/${side}_hubcap.stl"/>
+          <mesh filename="package://b166er_robot/meshes/pioneer3at/${side}_hubcap.stl"/>
         </geometry>
       </collision>
@@ -293,5 +293,5 @@
         <origin xyz="0 0 0" rpy="0 0 0"/>
         <geometry name="pioneer_geom">
-          <mesh filename="package://pioneer3at_simulation/meshes/wheel.stl" scale="0.75 0.66 0.75"/>
+          <mesh filename="package://b166er_robot/meshes/pioneer3at/wheel.stl" scale="0.75 0.66 0.75"/>
         </geometry>
         <material name="WheelBlack"/>
@@ -300,5 +300,5 @@
         <origin xyz="0 0 0" rpy="${-3.1415927/2} 0 0"/>
         <geometry>
-          <!--mesh filename="package://pioneer3at_simulation/meshes/wheel.stl"/-->
+          <!--mesh filename="package://b166er_robot/meshes/pioneer3at/wheel.stl"/-->
           <cylinder radius="0.085" length="0.05"/>
         </geometry>

Commit message: fix(sim): remove câmeras e lasers fictícios herdados do template
O xacro do Pioneer trazia 4 câmeras RGB simuladas e 2 lasers dummy de
3 amostras no top_plate, resquício do template original — sem
correspondência com nenhum hardware real do b166er e confundindo a
inspeção visual no RViz com a T265 (visualmente pareciam duas
câmeras coladas perto do gripper). Removidas as 6 instâncias e o
macro custom_camera, que ficou sem uso. O top_plate agora só tem o
laser_hokuyo_link, como no robô real.

Co-Authored-By: Claude Sonnet 4.6 <noreply@anthropic.com>

File: src/b166er_robot/urdf/pioneer3at/pioneer3at-m.urdf.xacro (robot description, xacro)
@@ -363,73 +363,4 @@
     </gazebo>
   </xacro:macro>
-  <xacro:macro name="custom_camera" params="name color x y z roll pitch yaw h_fov width height near far">
-    <joint name="camera_${name}_joint" type="fixed">
-      <axis xyz = "1 0 0"/>
-      <origin xyz="${x} ${y} ${z}" rpy="${roll} ${pitch} ${yaw}"/>
-      <parent link="top_plate"/>
-      <child link="camera_${name}_link"/>
-    </joint>
-    <link name="camera_${name}_link">
-        <collision>
-          <origin xyz="0 0 0" rpy="0 0 0"/>
-          <geometry>
-            <box size="0.025 0.025 0.025"/>
-          </geometry>
-        </collision>
-        <visual>
-          <origin xyz="0 0 0" rpy="0 0 0"/>
-          <geometry>
-            <box size="0.025 0.025 0.025"/>
-          </geometry>
-          <material name="red"/>
-        </visual>
-        <inertial>
-          <mass value="1e-5" />
-          <origin xyz="0 0 0" rpy="0 0 0"/>
-          <inertia ixx="1e-6" ixy="0" ixz="0" iyy="1e-6" iyz="0" izz="1e-6" />
-        </inertial>
-    </link>
-    <gazebo reference="camera_${name}_link">
-      <material value="Gazebo/${color}"/>
-      <sensor type="camera" name="camera_${name}">
-        <update_rate>30.0</update_rate>
-        <camera name="camera_${name}">
-          <pose> 0.025 0 0 0 0 0</pose>
-          <horizontal_fov>${h_fov}</horizontal_fov>
-          <image>
-            <width>${width}</width>
-            <height>${height}</height>
-            <format>R8G8B8</format>
-          </image>
-          <clip>
-            <near>${near}</near>
-            <far>${far}</far>
-          </clip>
-          <noise>
-            <type>gaussian</type>
-            <!-- Noise is sampled independently per pixel on each frame.
-                 That pixel's noise value is added to each of its color
-                 channels, which at that point lie in the range [0,1]. -->
-            <mean>0.0</mean>
-            <stddev>0.007</stddev>
-          </noise>
-        </camera>
-        <plugin name="camera_controller" filename="libgazebo_ros_camera.so">
-          <alwaysOn>true</alwaysOn>
-          <updateRate>0.0</updateRate>
-          <cameraName>/${robot_name}/camera_${name}</cameraName>
-          <imageTopicName>image_raw</imageTopicName>
-          <cameraInfoTopicName>camera_info</cameraInfoTopicName>
-          <frameName>camera_${name}_link</frameName>
-          <hackBaseline>0.07</hackBaseline>
-          <distortionK1>0.0</distortionK1>
-          <distortionK2>0.0</distortionK2>
-          <distortionK3>0.0</distortionK3>
-          <distortionT1>0.0</distortionT1>
-          <distortionT2>0.0</distortionT2>
-        </plugin>
-      </sensor>
-    </gazebo>
-  </xacro:macro>
   <xacro:macro name="custom_laser" params="name color x y z roll pitch yaw samples resolution min_angle max_angle min_range max_range range_resolution">
     <joint name="laser_${name}_joint" type="fixed">
@@ -531,13 +462,4 @@
     </gazebo>
   </xacro:macro>
-  <!-- RGB cameras -->
-  <xacro:custom_camera name="one" color="Red" x="0.24" y="0" z="0.04" roll="0" pitch="0.0" yaw="0" h_fov="1.3962634" width="800" height="800" near="0.02" far="100"/>
-  <xacro:custom_camera name="two" color="Blue" x="0.22" y="0.09" z="0.015" roll="0.2" pitch="0.1" yaw="-0.1" h_fov="1.3962634" width="800" height="800" near="0.02" far="100"/>
-  <xacro:custom_camera name="three" color="Yellow" x="0.22" y="-0.1" z="0.015" roll="-0.2" pitch="0.1" yaw="0.2" h_fov="1.3962634" width="800" height="800" near="0.02" far="100"/>
-  <!-- 'RGB' downward sensor -->
-  <xacro:custom_camera name="down" color="White" x="0.0" y="0.0" z="-0.17" roll="0.0" pitch="1.57" yaw="0.0" h_fov="1.0" width="100" height="100" near="0.01" far="1.0"/>
-  <!-- laser sensors -->
-  <xacro:custom_laser name="one" color="White" x="0.24" y="0" z="0.014" roll="0" pitch="0" yaw="0" samples="3" resolution="1" min_angle="${-PI/100}" max_angle="${PI/100}" min_range="0.10" max_range="5.0" range_resolution="0.01"/>
-  <xacro:custom_laser name="two" color="White" x="-0.22" y="0" z="0.014" roll="0" pitch="0" yaw="${PI}" samples="3" resolution="1" min_angle="${-PI/100}" max_angle="${PI/100}" min_range="0.10" max_range="5.0" range_resolution="0.01"/>
   <!-- skid steer controller -->
   <xacro:p3at_drive_side side="left" reflect="1"/>

Commit message: fix(sim): elimina disco branco das rodas e raios do laser no Gazebo/RViz
Três causas do artefato visual "uma roda branca" encontradas e corrigidas:

1. pioneer_wheel_state_pub: polling rápido (2ms) durante Gazebo pausado
   em vez de WallRate(10). Ao detectar o clock avançar publica imediata-
   mente os 4 joint states das rodas — eliminando a janela de ~100ms em
   que robot_state_publisher desconhecia a posição das rodas e o RViz as
   renderizava na origem do fixed_frame como disco branco centralizado.
   Taxa de manutenção elevada de 10 Hz para 50 Hz.

2. pioneer3at-m.urdf.xacro (custom_laser): material "red" não possuía
   <color> → RViz renderizava o link do laser (caixa 2.5cm) em branco
   (material indefinido). Adicionado rgba="0.8 0.1 0.1 1".

3. pioneer3at-m.urdf.xacro (custom_laser): <visualize>true</visualize>
   fazia o Gazebo renderizar os 1081 raios do Hokuyo como um disco
   branco de 270° ao redor do sensor. Desativado.

Co-Authored-By: Claude Sonnet 4.6 <noreply@anthropic.com>

File: src/b166er_robot/urdf/pioneer3at/pioneer3at-m.urdf.xacro (robot description, xacro)
@@ -386,5 +386,9 @@
             <box size="0.025 0.025 0.025"/>
           </geometry>
-          <material name="red"/>
+          <!-- "red" sem <color> = material indefinido no RViz → link renderizado branco.
+               Definição explícita garante cor vermelha em vez do branco padrão. -->
+          <material name="red">
+            <color rgba="0.8 0.1 0.1 1"/>
+          </material>
         </visual>
         <inertial>
@@ -398,5 +402,7 @@
         <sensor type="gpu_ray" name="laser_${name}">
           <pose>0 0 0 0 0 0</pose>
-          <visualize>true</visualize>
+          <!-- visualize=true desenha os 1081 raios como disco branco no Gazebo,
+               confundindo a inspeção visual do robô. Desabilitado. -->
+          <visualize>false</visualize>
           <update_rate>40</update_rate>
           <ray>

Commit message: fix(sim): corrige movimento do Pioneer e disco branco no RViz/Gazebo
- <joint_properties damping="0.7"/> → <dynamics damping="1.0" friction="3.0"/>
  nas 4 juntas de roda: tag padrão URDF que o Gazebo aplica corretamente.
  friction=3 N·m impede rotação passiva das rodas sob força do braço.
- sensor type="gpu_ray" → "ray" + libgazebo_ros_gpu_laser.so → _laser.so:
  gpu_ray ignora <visualize>false</visualize> no Gazebo 11, causando o
  disco branco de 270° dos raios do laser no Gazebo. Ray CPU honra o tag.
- Adiciona <color rgba> explícito nas referências HubcapYellow e WheelBlack
  do lado traseiro: RViz sem cor explícita pode usar branco como fallback.
- Remove chamada a <xacro:p3at_gazebo_contacts/>: libgazeboRosPioneer3ATContacts.so
  não existe em nenhum sistema, gerava erro de carregamento de plugin no log.

Co-Authored-By: Claude Sonnet 4.6 <noreply@anthropic.com>

File: src/b166er_robot/urdf/pioneer3at/pioneer3at-m.urdf.xacro (robot description, xacro)
@@ -217,5 +217,5 @@
       <anchor xyz="0 0 0"/>
       <limit effort="10" velocity="10"/>
-      <joint_properties damping="0.7"/>
+      <dynamics damping="1.0" friction="3.0"/>
       <origin xyz="0 0 0" rpy="0 0 0"/>
       <parent link="p3at_front_${side}_hub"/>
@@ -265,5 +265,7 @@
           <mesh filename="package://b166er_robot/meshes/pioneer3at/${side}_hubcap.stl"/>
         </geometry>
-        <material name="HubcapYellow"/>
+        <material name="HubcapYellow">
+          <color rgba="1.0 0.811 0.151 1.0"/>
+        </material>
       </visual>
       <collision>
@@ -299,5 +301,7 @@
           <mesh filename="package://b166er_robot/meshes/pioneer3at/wheel.stl" scale="0.75 0.66 0.75"/>
         </geometry>
-        <material name="WheelBlack"/>
+        <material name="WheelBlack">
+          <color rgba="0.117 0.117 0.117 1"/>
+        </material>
       </visual>
       <collision>
@@ -316,5 +320,5 @@
       <anchor xyz="0 0 0"/>
       <limit effort="10" velocity="10"/>
-      <joint_properties damping="0.7"/>
+      <dynamics damping="1.0" friction="3.0"/>
       <origin xyz="0 0 0" rpy="0 0 0"/>
       <parent link="p3at_back_${side}_hub"/>
@@ -400,5 +404,5 @@
     <gazebo reference="laser_${name}_link">
         <material value="Gazebo/${color}"/>
-        <sensor type="gpu_ray" name="laser_${name}">
+        <sensor type="ray" name="laser_${name}">
           <pose>0 0 0 0 0 0</pose>
           <!-- visualize=true desenha os 1081 raios como disco branco no Gazebo,
@@ -430,5 +434,5 @@
             </noise>
           </ray>
-          <plugin name="gazebo_ros_head_hokuyo_controller" filename="libgazebo_ros_gpu_laser.so">
+          <plugin name="gazebo_ros_head_hokuyo_controller" filename="libgazebo_ros_laser.so">
             <topicName>/${robot_name}/laser_${name}/scan</topicName>
             <frameName>laser_${name}_link</frameName>
@@ -480,5 +484,3 @@
   <xacro:p3at_drive_side side="right" reflect="-1"/>
   <xacro:p3at_gazebo_ext/>
-  <!-- contacts and extra robot_state -->
-  <xacro:p3at_gazebo_contacts/>
 </robot>

Commit message: fix(sim): amortece contato das rodas — elimina drift por locomoção vibratória
Diagnóstico ao vivo na simulação rodando:
- Chassi avançava ~20-30 mm/s com rodas paradas (FL 92 rad acumulados vs
  BL -0.02) e twist do corpo ~0 — movimento por correção de posição, não
  por rolagem.
- Snapshot de /gazebo/link_states: TODOS os links com vz≈-0.08 m/s — o
  robô inteiro em queda perpétua num ciclo-limite de quicar do contato.
- J2/J3 com taxas fantasma constantes (+0.42/-0.29 rad/s) e posição
  congelada: o braço balançando em sincronia com o quicar; estendido
  horizontal (pose zero do RV-M2), retificava a vibração em avanço.

Causa: kp=1e6 com kd=100 nas rodas → ζ≈1.6% para ~41 kg (kd crítico
≈6300). O contato ressoava a ~50 Hz sem dissipar energia.

Correções:
- kd 100 → 1e4 nas 4 rodas (ζ≈1.6, levemente sobreamortecido).
- Remove bloco <gazebo reference> duplicado das rodas dianteiras
  (introduzido em b2bec0f) que conflitava na fusão do SDF.
- Spawn z -0.02 → -0.025: queda inicial de 6 mm → 1 mm, sem excitar o
  modo vertical no unpause.

Co-Authored-By: Claude Fable 5 <noreply@anthropic.com>

File: src/b166er_robot/urdf/pioneer3at/pioneer3at-m.urdf.xacro (robot description, xacro)
@@ -206,11 +206,7 @@
       </collision>
     </link>
-    <gazebo reference="p3at_front_${side}_wheel">
-      <material value="Gazebo/Black"/>
-      <kp>1000000.0</kp>
-      <kd>100.0</kd>
-      <mu1>0.9</mu1>
-      <mu2>0.9</mu2>
-    </gazebo>
+    <!-- Parâmetros de contato ficam no bloco único mais abaixo (junto do
+         sensor de contato) — blocos <gazebo reference> duplicados para o
+         mesmo link conflitam na fusão do SDF. -->
     <joint name="p3at_front_${side}_wheel_joint" type="continuous">
       <axis xyz="0 1 0"/>
@@ -333,6 +329,9 @@
         </sensor>
         <kp>1000000.0</kp>
-        <!-- kp and kd for rubber -->
-        <kd>100.0</kd>
+        <!-- kd=100 dava razão de amortecimento ~1.6% para os ~41 kg do robô
+             (kd crítico ≈ 6300): o contato quicava a ~50 Hz sem dissipar e a
+             vibração era retificada pelo braço em deslocamento contínuo do
+             chassi (~20-30 mm/s). kd=1e4 → ζ≈1.6 (levemente sobreamortecido). -->
+        <kd>10000.0</kd>
         <mu1>0.9</mu1>
         <!-- was 10 -->
@@ -355,6 +354,6 @@
         </sensor>
         <kp>1000000.0</kp>
-        <!-- kp and kd for rubber -->
-        <kd>100.0</kd>
+        <!-- kd=1e4: ver comentário no bloco da roda traseira. -->
+        <kd>10000.0</kd>
         <mu1>0.9</mu1>
         <!-- was 10 -->

Commit message: fix(sim): reduz fricção das rodas 3.0 → 0.5 N·m para ajuste fino da base
Teste whole-body no Gazebo: alvo EE a 0.5 m de distância → base andou,
braço coordenou, orientação convergiu — mas estacionou com erro de 7.9 mm
(critério Fase 3: < 5 mm). O fuzzy_wb_controller ficou comandando
-2.1 mm/s em regime permanente sem a base responder: os 3 N·m de fricção
de junta (paliativo do drift) agem como stiction e bloqueiam comandos de
ajuste fino. Com a causa real do drift corrigida (kd=1e4 no contato),
0.5 N·m mantém frenagem passiva sem impedir micro-movimentos.

Co-Authored-By: Claude Fable 5 <noreply@anthropic.com>

File: src/b166er_robot/urdf/pioneer3at/pioneer3at-m.urdf.xacro (robot description, xacro)
@@ -213,5 +213,5 @@
       <anchor xyz="0 0 0"/>
       <limit effort="10" velocity="10"/>
-      <dynamics damping="1.0" friction="3.0"/>
+      <dynamics damping="1.0" friction="0.5"/>
       <origin xyz="0 0 0" rpy="0 0 0"/>
       <parent link="p3at_front_${side}_hub"/>
@@ -316,5 +316,5 @@
       <anchor xyz="0 0 0"/>
       <limit effort="10" velocity="10"/>
-      <dynamics damping="1.0" friction="3.0"/>
+      <dynamics damping="1.0" friction="0.5"/>
       <origin xyz="0 0 0" rpy="0 0 0"/>
       <parent link="p3at_back_${side}_hub"/>
