Commit message: fix(b166er_robot): placa da tag 165mm para o quadrado preto renderizar 132mm
A textura apriltag_36h11_id0.png tem quiet zone branca: o quadrado
preto ocupa exatamente 80% da imagem (medido pixel a pixel, bbox
100-899 numa textura de 1000px). O detector/PnP mede o quadrado
PRETO — é ele que deve ter os 132mm da tag física já validada em
hardware, não a placa inteira. Com a placa antiga de 132mm, o preto
renderizava 105,6mm e o PnP superestimava a distância em exatamente
25% (fator medido ao vivo na validação do apriltag_localizer,
2026-08-13). Placa agora mede tag_black_size/0.8 = 165mm.

Co-Authored-By: Claude Fable 5 <noreply@anthropic.com>

File: src/b166er_robot/urdf/fixtures/apriltag_mount.urdf.xacro (robot description, xacro)
@@ -14,5 +14,16 @@
        material OGRE em materials/scripts/apriltag.material. -->
   <xacro:macro name="apriltag_mount" params="parent prefix:=tag_ xyz:='0 0 0' rpy:='0 0 0'">
-    <xacro:property name="tag_size" value="0.132"/>          <!-- 132 mm — mesma tag física já validada -->
+    <!-- A textura apriltag_36h11_id0.png tem quiet zone branca: o
+         quadrado preto ocupa exatamente 80% da imagem (medido pixel a
+         pixel em 2026-08-13, bbox 100-899 numa textura de 1000px). O
+         que importa para o detector/PnP é o QUADRADO PRETO — é ele que
+         deve medir 132mm, igual à tag física do Marco já validada em
+         hardware (ver project_fase4_apriltag_validacao). Por isso a
+         PLACA mede tag_black_size/0.8 = 165mm, para o preto renderizar
+         os 132mm exatos. Descoberto ao vivo: o PnP superestimava a
+         distância em ~25% quando a placa media 132mm (preto = 105,6mm
+         renderizado, tratado como 132mm pelo detector). -->
+    <xacro:property name="tag_black_size" value="0.132"/>    <!-- 132 mm — quadrado preto, mesma tag física validada -->
+    <xacro:property name="tag_size" value="${tag_black_size/0.8}"/>  <!-- placa: preto + quiet zone da textura -->
     <xacro:property name="tag_plate_thickness" value="0.005"/>
     <xacro:property name="wall_standoff" value="0.02"/>

Commit message: feat: tag de 220mm, standoff 0.70 e correções de repetibilidade
Bateria de repetibilidade (pedido do Marco) rendeu quatro achados.

1. TAMANHO DA TAG (pergunta do Marco: "aumentando o tamanho da tag não
   melhora?" — melhora, e muito). De 132 para 220 mm. Medido em
   varredura, erro da pose da parede:
     distância   132 mm         220 mm
     2,80 m      sem detecção   59 mm
     2,30 m      —              26 mm
     1,80 m      —              17 mm
     1,30 m      ~40 mm         13 mm
     0,80 m      ~20 mm         17 mm
   O SEARCH acontece a ~3 m, onde a tag de 132 mm sequer detecta de
   forma útil — era essa a origem dos erros de meio metro que já
   mandaram o robô contra a parede. PARA A BANCADA REAL: precisa
   imprimir a tag de 220 mm.
   (Testei 320 mm também, mas ficou inconclusivo — o localizador não
   subiu direito naquela rodada; não afirmo nada sobre ele.)

2. TAG SOBREPONDO A CHAVE, notado pelo Marco: com 220 mm a PLACA foi
   para 27,5 cm de largura e, em -0.42, ficava a 2 mm da placa da
   chave. Movida para -0.50 (8 cm de folga).

3. DESEMPATE DA IK — bug meu, e o mais grave. A continuidade de ramo
   somava erro e distância num score único (e + w·dist), deixando a
   proximidade NEGOCIAR contra a precisão: quando a solução correta
   exigia reconfigurar o braço, perdia para uma solução ruim que
   estava perto, o resíduo estourava a tolerância e a missão abortava.
   Derrubou 8 de 8 execuções numa bateria. Agora é desempate de
   verdade: filtra quem alcança o alvo, e só entre esses escolhe o
   mais próximo da postura atual.

4. STANDOFF de 0,80 para 0,70 m. Com 0,80 sobravam 13 cm de margem de
   alcance e um erro de estacionamento de poucos centímetros bastava
   para o alvo sair do workspace (2 de 8 falharam assim). Atenção: o
   standoff é limitado dos DOIS lados — o pre_engage fica 18 cm à
   frente do olhal, então standoff pequeno demais o põe abaixo do
   alcance mínimo. Faixa viável medida: 0,58 a 0,90 m.

Também: mira-além da IK iterativa amortecida (0,8) e, se o ponto
extrapolado sair do alcance, recua para o alvo real em vez de abortar.

VISUALIZAÇÃO DA CÂMERA — o Marco relatou que nunca conseguia ver a
imagem. Eram dois problemas somados: (a) a imagem só era publicada se
já houvesse assinante, então o tópico parecia morto justamente quando
alguém ia olhar; (b) o localizador só subia junto com a missão, então
fora dela não havia imagem nenhuma. Agora publica sempre, a 15 Hz, e
sobe com o stack principal.
  rosrun image_view image_view image:=/b166er/tag_debug_image

Co-Authored-By: Claude Opus 5 <noreply@anthropic.com>

File: src/b166er_robot/urdf/fixtures/apriltag_mount.urdf.xacro (robot description, xacro)
@@ -20,9 +20,25 @@
          deve medir 132mm, igual à tag física do Marco já validada em
          hardware (ver project_fase4_apriltag_validacao). Por isso a
-         PLACA mede tag_black_size/0.8 = 165mm, para o preto renderizar
-         os 132mm exatos. Descoberto ao vivo: o PnP superestimava a
+         PLACA mede tag_black_size/0.8, para o preto renderizar o
+         tamanho nominal.
+         TAMANHO SUBIU DE 132 PARA 220 mm em 2026-08-21. A tag de
+         132 mm é a que o Marco tem impressa e validou em hardware,
+         mas ela limita a detecção confiável a 1,45 m (regra
+         lado ≥ d/11) — e o SEARCH da missão acontece a ~3 m, onde a
+         estimativa da parede errava mais de meio metro e chegou a
+         mandar o robô contra ela.
+         Medido em varredura (2026-08-21), erro da pose da parede:
+           distância   132 mm      220 mm
+           2,80 m      sem detecção  59 mm
+           2,30 m      —             26 mm
+           1,80 m      —             17 mm
+           1,30 m      ~40 mm        13 mm
+           0,80 m      ~20 mm        17 mm
+         PARA A BANCADA REAL: é preciso imprimir a tag de 220 mm. A de
+         132 mm continua válida, mas só a partir de ~1,4 m — o que
+         obriga a busca a acontecer mais perto da chave. Descoberto ao vivo: o PnP superestimava a
          distância em ~25% quando a placa media 132mm (preto = 105,6mm
          renderizado, tratado como 132mm pelo detector). -->
-    <xacro:property name="tag_black_size" value="0.132"/>    <!-- 132 mm — quadrado preto, mesma tag física validada -->
+    <xacro:property name="tag_black_size" value="0.220"/>   <!-- 220 mm — ver nota abaixo -->
     <xacro:property name="tag_size" value="${tag_black_size/0.8}"/>  <!-- placa: preto + quiet zone da textura -->
     <xacro:property name="tag_plate_thickness" value="0.005"/>

File: src/b166er_robot/urdf/fixtures/chave_com_tag.urdf.xacro (robot description, xacro)
@@ -25,10 +25,16 @@
        antes ficava em +0.20, com a chave em -0.20; agora do lado oposto.
        Aproximada da chave em seguida (também a pedido do Marco): a
-       separação caiu de 0,40 m para 0,22 m, com a tag em -0.42.
+       separação caiu de 0,40 m para 0,30 m, com a tag em -0.50.
+       Por que não mais perto: ao subir a tag de 132 para 220 mm, a
+       PLACA foi de 16,5 para 27,5 cm de largura, e em -0.42 a borda
+       dela ficava a 2 mm da placa da chave — visualmente encostadas
+       (o Marco notou: "a tag está em cima da chave"). Em -0.50 sobram
+       8 cm de folga. A conta que governa: meia-placa da tag (13,75 cm)
+       + meia-placa da chave (8 cm) + margem.
        Ficar perto importa para a percepção: quanto menor a distância
        entre a tag e o alvo de manipulação, menor o braço de alavanca
        do erro angular da detecção sobre a posição estimada do olhal.
        A parede segue com 1,6 m de largura. -->
-  <xacro:property name="tag_x_offset" value="-0.42"/>
+  <xacro:property name="tag_x_offset" value="-0.50"/>
   <!-- Altura de montagem do macro da chave = altura do PIVÔ (embaixo),
        não mais do bracket sob o isolador. Precisa bater com o cálculo

Commit message: fix(b166er_whole_body_control): tag a 17 cm do olhal e na mesma altura
Medido na bancada: o centro da tag fica 17 cm ao lado do olhal, na mesma
altura dele. A geometria anterior era arbitrada — 30 cm de separação e
22 cm acima.

Isso corta por 2,2 o braço de alavanca com que o erro angular da
detecção vira erro de posição no alvo (a missão estima a parede pela tag
e depois aplica offsets até o olhal).

Consequência: com 17 cm a placa da tag de 220 mm invade a placa da
chave. Só a de 132 mm cabe — e é a que o Marco tem impressa e
caracterizou contra a T265. O tamanho vira parâmetro do macro em vez de
constante escondida, porque agora ele interage com a geometria da
bancada.

task_sequencer para de manter a terceira cópia da geometria: ela tinha
apodrecido na mecânica de antes de 2026-08-13 (fechada = 20°, standoff
0,03) e agora importa de chave_task.

Co-Authored-By: Claude Opus 5 <noreply@anthropic.com>
Claude-Session: https://claude.ai/code/session_01Ra2BbYQxYWhbcCFkGE7vAN

File: src/b166er_robot/urdf/fixtures/apriltag_mount.urdf.xacro (robot description, xacro)
@@ -13,5 +13,5 @@
        ~/apriltag_36h11_id0.png, copiada para materials/textures/),
        material OGRE em materials/scripts/apriltag.material. -->
-  <xacro:macro name="apriltag_mount" params="parent prefix:=tag_ xyz:='0 0 0' rpy:='0 0 0'">
+  <xacro:macro name="apriltag_mount" params="parent prefix:=tag_ xyz:='0 0 0' rpy:='0 0 0' black_size:=0.132">
     <!-- A textura apriltag_36h11_id0.png tem quiet zone branca: o
          quadrado preto ocupa exatamente 80% da imagem (medido pixel a
@@ -39,6 +39,15 @@
          obriga a busca a acontecer mais perto da chave. Descoberto ao vivo: o PnP superestimava a
          distância em ~25% quando a placa media 132mm (preto = 105,6mm
-         renderizado, tratado como 132mm pelo detector). -->
-    <xacro:property name="tag_black_size" value="0.220"/>   <!-- 220 mm — ver nota abaixo -->
+         renderizado, tratado como 132mm pelo detector).
+         VIROU PARÂMETRO em 2026-08-27 (black_size). O tamanho deixou de
+         ser uma constante escondida aqui porque ele agora INTERAGE com
+         a geometria medida da bancada: a tag fica a 17 cm do olhal, e
+         nessa distância a placa de 220 mm invade a placa da chave. Quem
+         escolhe é chave_com_tag.urdf.xacro, onde as duas medidas se
+         encontram. Padrão 132 mm = a tag que o Marco tem impressa.
+         CURVA DE ALCANCE REAL (T265, 2026-08-26), tag de 132 mm:
+           detecta até ~1,8 m; mede bem só até ~1,2 m; colapsa em 2,5 m.
+         Extrapolando para 220 mm: ~3,0 m detecta, ~2,0 m mede bem. -->
+    <xacro:property name="tag_black_size" value="${black_size}"/>
     <xacro:property name="tag_size" value="${tag_black_size/0.8}"/>  <!-- placa: preto + quiet zone da textura -->
     <xacro:property name="tag_plate_thickness" value="0.005"/>

File: src/b166er_robot/urdf/fixtures/chave_com_tag.urdf.xacro (robot description, xacro)
@@ -22,29 +22,41 @@
   <xacro:property name="wall_height" value="1.40"/>
   <xacro:property name="chave_x_offset" value="-0.20"/>
-  <!-- Tag do OUTRO LADO da chave (pedido do Marco, 2026-08-13):
-       antes ficava em +0.20, com a chave em -0.20; agora do lado oposto.
-       Aproximada da chave em seguida (também a pedido do Marco): a
-       separação caiu de 0,40 m para 0,30 m, com a tag em -0.50.
-       Por que não mais perto: ao subir a tag de 132 para 220 mm, a
-       PLACA foi de 16,5 para 27,5 cm de largura, e em -0.42 a borda
-       dela ficava a 2 mm da placa da chave — visualmente encostadas
-       (o Marco notou: "a tag está em cima da chave"). Em -0.50 sobram
-       8 cm de folga. A conta que governa: meia-placa da tag (13,75 cm)
-       + meia-placa da chave (8 cm) + margem.
-       Ficar perto importa para a percepção: quanto menor a distância
-       entre a tag e o alvo de manipulação, menor o braço de alavanca
-       do erro angular da detecção sobre a posição estimada do olhal.
-       A parede segue com 1,6 m de largura. -->
-  <xacro:property name="tag_x_offset" value="-0.50"/>
-  <!-- Altura de montagem do macro da chave = altura do PIVÔ (embaixo),
-       não mais do bracket sob o isolador. Precisa bater com o cálculo
-       interno de chave_seccionadora_lf (pivot_z), que o xacro não
-       expõe para fora do macro: olhal_height=0.810, blade_length=0.200,
-       lâmina VERTICAL quando fechada. Mecânica invertida em 2026-08-13
-       (pivô embaixo, olhal em cima) e depois rotacionada 90° no eixo Z
-       (lâmina abre para fora da parede). O olhal segue a 0.810 m. -->
+  <!-- ═══ POSIÇÃO DA TAG — MEDIDA NA BANCADA (2026-08-26) ═══
+       olhal-dimension.png: o centro da tag fica a 17 cm do olhal, na
+       horizontal, e NA MESMA ALTURA dele. Toda a geometria anterior era
+       arbitrada: 30 cm de separação e 22 cm acima do olhal.
+       Isso muda o erro de percepção de forma direta. A missão estima a
+       pose da PAREDE pela tag e depois aplica offsets em YAML para
+       chegar ao olhal; quanto maior esse braço, mais o erro ANGULAR da
+       detecção vira erro de POSIÇÃO no alvo. Passar de 37 cm de
+       distância tag→olhal para 17 cm corta esse braço por 2,2.
+       CONSEQUÊNCIA QUE PRECISA DE DECISÃO: com 17 cm de separação a tag
+       de 220 mm não cabe mais ao lado da chave. Contas de meia-placa:
+         meia-placa da chave ......... 8,0 cm
+         meia-placa da tag 220 mm .... 13,75 cm  -> precisa de 21,75 cm
+         meia-placa da tag 132 mm .... 8,25 cm   -> precisa de 16,25 cm
+       Só a de 132 mm cabe nos 17 cm medidos — e é justamente a que o
+       Marco tem impressa. Por isso o padrão volta para 132 mm.
+       O preço é conhecido e já estava documentado: com 132 mm a
+       detecção confiável termina em ~1,8 m (T265 real, medido em
+       2026-08-26), e o SEARCH da missão acontece a 2,8 m. Ou a busca
+       desce para menos de 1,8 m, ou a bancada precisa afastar a tag do
+       olhal para caber a de 220 mm. As duas saídas são medições, não
+       chutes — mas são decisão do Marco. -->
+  <xacro:property name="tag_olhal_dx" value="0.17"/>
+  <xacro:property name="tag_x_offset" value="${chave_x_offset - tag_olhal_dx}"/>
+  <xacro:property name="tag_black_size" value="0.132"/>
+  <!-- Altura de montagem do macro da chave = altura do PIVÔ (embaixo).
+       Precisa bater com o cálculo interno de chave_seccionadora_lf
+       (pivot_z), que o xacro não expõe para fora do macro:
+       olhal_height=0.805 (MEDIDO), blade_length=0.200, lâmina VERTICAL
+       quando fechada. Mecânica invertida em 2026-08-13 (pivô embaixo,
+       olhal em cima) e depois rotacionada 90° no eixo Z (lâmina abre
+       para fora da parede). -->
+  <xacro:property name="olhal_z" value="0.805"/>
   <xacro:property name="chave_pivot_z"
-    value="${0.810 - 0.200}"/>  <!-- 0,610 m — lâmina VERTICAL na posição fechada -->
-  <xacro:property name="tag_mount_z" value="1.030"/>
+    value="${olhal_z - 0.200}"/>  <!-- 0,605 m — lâmina VERTICAL na posição fechada -->
+  <!-- Mesma altura do olhal (medido). Era 1.030. -->
+  <xacro:property name="tag_mount_z" value="${olhal_z}"/>
   <!-- ═══ Parede: base no chão, face frontal (mounting) em Y=0 do frame
        local, corpo se estendendo para -Y (atrás) ═══ -->
@@ -74,5 +86,6 @@
     xyz="${chave_x_offset} 0 ${chave_pivot_z}" rpy="0 0 0"/>
   <xacro:apriltag_mount parent="wall_link" prefix="tag_"
-    xyz="${tag_x_offset} 0 ${tag_mount_z}" rpy="0 0 0"/>
+    xyz="${tag_x_offset} 0 ${tag_mount_z}" rpy="0 0 0"
+    black_size="${tag_black_size}"/>
   <!-- A fixture NÃO pode mais ser <static>: modelo estático no Gazebo
        não simula juntas, e a lâmina precisa girar para a chave abrir
