Commit message: fix(b166er_robot): remove isolador do fixture da chave seccionadora
Por decisão explícita do Marco (documento "Descrição do movimento de
abertura da chave seccionadora", Google Docs, 2026-08-12): a bancada
de testes física fixa a chave direto na parede, sem o isolador tipo
bucha, e a simulação deve seguir o mesmo layout — a foto da bancada
real (mesmo documento) confirma isso, com a tag AprilTag já posicionada
exatamente como no nosso fixture.

A lâmina agora pivota direto no topo do bracket em vez de no topo do
isolador removido. bracket_mount_z recalculado (era ~0,788m com
isolador, agora ~0,938m sem) para que o olhal continue caindo em
exatamente 810mm do chão — verificado numericamente no URDF processado
pelo xacro.

Co-Authored-By: Claude Sonnet 5 <noreply@anthropic.com>

File: src/b166er_robot/urdf/fixtures/chave_com_tag.urdf.xacro (robot description, xacro)
@@ -28,7 +28,11 @@
        parâmetros dimensionais da chave mudarem lá, atualizar aqui
        também — olhal_height=0.810, blade_length=0.200,
-       blade_angle=0.349 rad, insulator_height=0.150, bracket_height=0.060. -->
+       blade_angle=0.349 rad, bracket_height=0.060. Sem isolador (ver
+       nota "SEM ISOLADOR" em chave_seccionadora_lf.urdf.xacro,
+       decisão do Marco em 2026-08-12): a lâmina pivota direto no
+       topo do bracket, então este valor subiu em relação à versão
+       anterior com isolador (que era ≈0,7879 m). -->
   <xacro:property name="chave_bracket_mount_z"
-    value="${0.810 + 0.200*cos(0.349) - 0.150 - 0.060}"/>  <!-- ≈ 0,7879 m -->
+    value="${0.810 + 0.200*cos(0.349) - 0.060}"/>  <!-- ≈ 0,9379 m -->
   <xacro:property name="tag_mount_z" value="1.030"/>
   <!-- ═══ Parede: base no chão, face frontal (mounting) em Y=0 do frame

File: src/b166er_robot/urdf/fixtures/chave_seccionadora_lf.urdf.xacro (robot description, xacro)
@@ -15,19 +15,27 @@
        IMPORTANTE: geometria de primitivas (caixas/cilindros), NÃO é
        uma réplica fiel de CAD — é uma aproximação proporcional
-       inspirada no desenho técnico do datasheet (isolador tipo bucha
-       nervurado, lâmina móvel a ~20° da vertical na posição fechada,
-       olhal na ponta da lâmina). O que É exato: a altura do olhal
-       acima do solo, fixada em 810 mm por especificação direta do
-       Marco — todo o resto da geometria é construído de baixo para
-       cima a partir desse ponto, não o contrário.
+       inspirada no desenho técnico do datasheet (lâmina móvel a ~20°
+       da vertical na posição fechada, olhal na ponta da lâmina). O
+       que É exato: a altura do olhal acima do solo, fixada em 810 mm
+       por especificação direta do Marco — todo o resto da geometria é
+       construído de baixo para cima a partir desse ponto, não o
+       contrário.
+       SEM ISOLADOR: por decisão explícita do Marco (documento
+       "Descrição do movimento de abertura da chave seccionadora",
+       Google Docs, compartilhado em 2026-08-12), o isolador tipo
+       bucha foi removido tanto da bancada de testes física quanto
+       desta simulação — a foto da bancada real (mesmo documento)
+       mostra a chave presa direto na parede, sem bucha, com a tag
+       AprilTag logo acima, exatamente como já modelávamos o resto do
+       fixture. A lâmina agora pivota direto no topo do bracket.
        Montagem: fixada direto numa parede (ver chave_com_tag.urdf.xacro),
        não num poste próprio — por isso este macro não tem link de base
        nem de suporte vertical, só o bracket "base C" que encosta na
-       parede e a cadeia bracket→isolador→lâmina→olhal por cima dele.
-       O afastamento de 3 cm da face da parede é aplicado uma única vez,
-       no joint bracket→isolador, e propaga por herança de frame para
-       todo o resto da cadeia (terminal, lâmina, olhal) — importante
-       para o TF do olhal_link bater exatamente com a geometria visual/
-       de colisão renderizada, já que é esse frame que o controlador
+       parede e a cadeia bracket→lâmina→olhal por cima dele. O
+       afastamento de 3 cm da face da parede é aplicado uma única vez,
+       no joint bracket→lâmina, e propaga por herança de frame para o
+       resto da cadeia (terminal, lâmina, olhal) — importante para o
+       TF do olhal_link bater exatamente com a geometria visual/de
+       colisão renderizada, já que é esse frame que o controlador
        whole-body vai mirar.
        Referências visuais usadas (não reproduzidas como imagem, só
@@ -40,5 +48,4 @@
     <xacro:property name="blade_length" value="0.200"/>       <!-- comprimento aprox. da lâmina móvel -->
     <xacro:property name="blade_angle" value="0.349"/>        <!-- 20° em rad, ângulo fechado (datasheet) -->
-    <xacro:property name="insulator_height" value="0.150"/>   <!-- altura aprox. do isolador tipo bucha -->
     <xacro:property name="bracket_height" value="0.060"/>     <!-- altura aprox. do suporte "base C" -->
     <xacro:property name="wall_standoff" value="0.03"/>       <!-- afastamento da face da parede -->
@@ -48,6 +55,7 @@
     <xacro:property name="pivot_x" value="${blade_length*sin(blade_angle)}"/>
     <!-- Altura em que o bracket precisa encostar na parede para que o
-         olhal, no fim da cadeia, caia exatamente em olhal_height. -->
-    <xacro:property name="bracket_mount_z" value="${olhal_height + pivot_z - insulator_height - bracket_height}"/>
+         olhal, no fim da cadeia, caia exatamente em olhal_height. Sem
+         isolador no meio, a lâmina pivota direto no topo do bracket. -->
+    <xacro:property name="bracket_mount_z" value="${olhal_height + pivot_z - bracket_height}"/>
     <!-- ═══ Suporte "base C" (bracket de fixação à parede) ═══ -->
     <link name="${prefix}bracket">
@@ -71,49 +79,17 @@
       <origin xyz="${xyz}" rpy="${rpy}"/>
     </joint>
-    <!-- ═══ Isolador tipo bucha (porcelana vitrificada), aproximado por
-         3 segmentos cilíndricos de raio alternado para sugerir as
-         nervuras — não é o perfil real, só a silhueta geral. O
-         afastamento da parede (wall_standoff) é aplicado aqui, uma
-         única vez — todo o resto da cadeia (terminal, lâmina, olhal)
-         herda esse deslocamento automaticamente por ser filho deste
-         link, sem precisar repetir o offset. ═══ -->
-    <xacro:property name="rib_h" value="${insulator_height/3}"/>
-    <link name="${prefix}insulator">
-      <visual>
-        <origin xyz="0 0 ${rib_h*0.5}"/>
-        <geometry><cylinder radius="0.045" length="${rib_h}"/></geometry>
-        <material name="porcelain"><color rgba="0.85 0.85 0.83 1"/></material>
-      </visual>
-      <visual>
-        <origin xyz="0 0 ${rib_h*1.5}"/>
-        <geometry><cylinder radius="0.038" length="${rib_h}"/></geometry>
-        <material name="porcelain"/>
-      </visual>
-      <visual>
-        <origin xyz="0 0 ${rib_h*2.5}"/>
-        <geometry><cylinder radius="0.045" length="${rib_h}"/></geometry>
-        <material name="porcelain"/>
-      </visual>
-      <collision>
-        <origin xyz="0 0 ${insulator_height/2}"/>
-        <geometry><cylinder radius="0.045" length="${insulator_height}"/></geometry>
-      </collision>
-      <inertial>
-        <mass value="1.5"/>
-        <inertia ixx="0.005" ixy="0" ixz="0" iyy="0.005" iyz="0" izz="0.002"/>
-      </inertial>
-    </link>
-    <joint name="${prefix}insulator_joint" type="fixed">
-      <parent link="${prefix}bracket"/>
-      <child link="${prefix}insulator"/>
-      <origin xyz="0 ${wall_standoff} ${bracket_height}" rpy="0 0 0"/>
-    </joint>
-    <!-- ═══ Terminal fixo (padrão NEMA) no topo do isolador ═══ -->
+    <!-- ═══ Terminal fixo (padrão NEMA) no topo do bracket. Sem
+         isolador para encadear o afastamento da parede (wall_standoff)
+         por herança, terminal e lâmina são agora irmãos, filhos diretos
+         do bracket — cada branch repete o offset Y explicitamente
+         (ver também blade_joint logo abaixo). ═══ -->
     <link name="${prefix}fixed_terminal">
       <visual>
+        <origin xyz="0 ${wall_standoff} 0"/>
         <geometry><box size="0.06 0.03 0.03"/></geometry>
         <material name="copper"><color rgba="0.72 0.45 0.20 1"/></material>
       </visual>
       <collision>
+        <origin xyz="0 ${wall_standoff} 0"/>
         <geometry><box size="0.06 0.03 0.03"/></geometry>
       </collision>
@@ -124,12 +100,13 @@
     </link>
     <joint name="${prefix}fixed_terminal_joint" type="fixed">
-      <parent link="${prefix}insulator"/>
+      <parent link="${prefix}bracket"/>
       <child link="${prefix}fixed_terminal"/>
-      <origin xyz="0 0 ${insulator_height}" rpy="0 0 0"/>
+      <origin xyz="0 0 ${bracket_height}" rpy="0 0 0"/>
     </joint>
     <!-- ═══ Lâmina móvel (posição fechada, ~20° da vertical) e olhal
          na ponta — este é o ponto que a garra deve alcançar para
-         operar a chave. Pivô no topo do isolador; a lâmina desce e se
-         inclina para fora até o olhal, em Z = 0.810 m do solo. ═══ -->
+         operar a chave. Pivô no topo do bracket (sem isolador no
+         meio); a lâmina desce e se inclina para fora até o olhal, em
+         Z = 0.810 m do solo. ═══ -->
     <link name="${prefix}blade">
       <visual>
@@ -148,7 +125,7 @@
     </link>
     <joint name="${prefix}blade_joint" type="fixed">
-      <parent link="${prefix}insulator"/>
+      <parent link="${prefix}bracket"/>
       <child link="${prefix}blade"/>
-      <origin xyz="0 0 ${insulator_height}" rpy="0 0 0"/>
+      <origin xyz="0 ${wall_standoff} ${bracket_height}" rpy="0 0 0"/>
     </joint>
     <!-- Olhal: anel de engate para a vara de manobra / garra do robô.
@@ -183,7 +160,4 @@
       <material>Gazebo/Grey</material>
     </gazebo>
-    <gazebo reference="${prefix}insulator">
-      <material>Gazebo/White</material>
-    </gazebo>
     <gazebo reference="${prefix}fixed_terminal">
       <material>Gazebo/Orange</material>
