Commit message: fix(b166er_robot): chave fechada = lâmina vertical, olhal vira anel, ferramenta ganha gancho
Três correções do Marco (2026-08-13):

1. FECHADA = LÂMINA VERTICAL. O modelo desenhava a lâmina inclinada
   20°, que é a posição ABERTA — "a inclinação que está é a posição
   da chave aberta". Fechada, a lâmina fica vertical encostando no
   contato fixo de cima; abrir é girá-la 30° para fora.
   Propagado: chave_pivot_z = 0.810 - 0.200 = 0.610 (era 0.622, com o
   cosseno do ângulo errado); OLHAL_OFFSET_FROM_WALL_LINK perde a
   componente de inclinação e vira (-0.20, 0.03, 0.810); os waypoints
   de abertura recalculados de 0°→15°→30° (dy=+0.052/+0.100,
   dz=-0.007/-0.027) em vez de partirem dos 20°.

2. OLHAL É UM ANEL, não uma barra — "não há a representação do
   olhal". É por dentro dele que o gancho passa. URDF não tem
   toroide, então são 10 cilindros curtos em círculo, no plano X-Z,
   com o furo voltado para o robô.

3. FERRAMENTA COM GANCHO na ponta — "para realizar a abertura a
   ferramenta deve ter na ponta um formato de gancho". Era um disco
   chato, que não engancharia nada. Agora um J aberto para o lado,
   desenhado EM VOLTA da origem de tool_tip: como é esse frame que o
   controlador mira, levar tool_tip ao centro do olhal põe o anel
   dentro do vão do gancho.

URDF e chave_task.py conferidos: olhal em (-0.20, 0.03, 0.810)
relativo a wall_link nos dois.

Co-Authored-By: Claude Opus 5 <noreply@anthropic.com>

File: src/b166er_robot/urdf/fixtures/chave_com_tag.urdf.xacro (robot description, xacro)
@@ -27,9 +27,9 @@
        interno de chave_seccionadora_lf (pivot_z), que o xacro não
        expõe para fora do macro: olhal_height=0.810, blade_length=0.200,
-       blade_angle=0.349 rad. Mecânica invertida em 2026-08-13 (pivô
-       embaixo, olhal em cima) — o OLHAL continua exatamente onde
-       estava, a 0.810 m; só a estrutura abaixo dele mudou. -->
+       lâmina VERTICAL quando fechada. Mecânica invertida em 2026-08-13
+       (pivô embaixo, olhal em cima) e depois rotacionada 90° no eixo Z
+       (lâmina abre para fora da parede). O olhal segue a 0.810 m. -->
   <xacro:property name="chave_pivot_z"
-    value="${0.810 - 0.200*cos(0.349)}"/>  <!-- ≈ 0,622 m -->
+    value="${0.810 - 0.200}"/>  <!-- 0,610 m — lâmina VERTICAL na posição fechada -->
   <xacro:property name="tag_mount_z" value="1.030"/>
   <!-- ═══ Parede: base no chão, face frontal (mounting) em Y=0 do frame

File: src/b166er_robot/urdf/fixtures/chave_seccionadora_lf.urdf.xacro (robot description, xacro)
@@ -1,55 +1,42 @@
 <?xml version="1.0"?>
 <robot xmlns:xacro="http://ros.org/wiki/xacro">
-  <!-- Chave seccionadora da BANCADA DE TESTES do Marco — remodelada em
-       2026-08-13 a partir da FOTO da bancada real (docs/img/
+  <!-- Chave seccionadora da BANCADA DE TESTES do Marco, modelada a
+       partir da FOTO da bancada real (docs/img/
        chave_bancada_teste_sem_isolador.jpg no pacote whole_body_control),
-       não mais do desenho técnico do datasheet STI.
-       Por que mudou: o desenho do datasheet inclui o isolador tipo bucha,
-       que a bancada não tem, e a silhueta resultante não lembrava a
-       chave real ("a renderização da chave não está parecido com o
-       real" — Marco). A foto mostra outra coisa: uma placa branca
-       parafusada na parede, um bracket metálico chato no topo, um
-       mecanismo escuro em forma de wishbone descendo, a barra
-       horizontal do olhal atravessando, e um segundo bracket metálico
-       na base.
-       INVERSÃO DA MECÂNICA (correção do Marco, 2026-08-13): o PIVÔ fica
-       EMBAIXO e o OLHAL EM CIMA. A versão anterior tinha isso ao
-       contrário (lâmina pendurada de um pivô superior), o que colocava
-       o alvo de manipulação na extremidade errada da chave — o robô
-       mirava a ponta de baixo.
-       O QUE NÃO MUDOU, de propósito: a posição do olhal no mundo
-       (810 mm do chão, mesmo offset lateral). É a esse ponto que o
-       pipeline de percepção e chave_task.py estão calibrados; inverter
-       a mecânica abaixo dele não mexe no alvo. Ver
-       OLHAL_OFFSET_FROM_WALL_LINK em chave_task.py.
+       não do desenho técnico do datasheet STI — o desenho inclui o
+       isolador tipo bucha, que a bancada não tem.
+       Geometria, depois das correções do Marco em 2026-08-13:
+       · PIVÔ EMBAIXO, OLHAL EM CIMA. A primeira versão tinha o
+         contrário e o robô mirava a extremidade errada.
+       · LÂMINA NO PLANO Y-Z (chave "rotacionada 90° no eixo Z"): abre
+         inclinando PARA FORA da parede, na direção de onde o robô se
+         aproxima. A barra do mecanismo corre paralela à face, como na
+         foto.
+       · FECHADA = LÂMINA VERTICAL. A versão anterior desenhava a
+         lâmina já inclinada 20°, que é a posição ABERTA ("a inclinação
+         que está é a posição da chave aberta" — Marco). Fechada, a
+         lâmina encosta no contato fixo de cima; abrir é girá-la 30°
+         para fora (curso confirmado pelo Marco).
+       · OLHAL É UM ANEL, não uma barra. É por dentro dele que o gancho
+         da ferramenta passa. URDF não tem primitiva de toroide, então
+         o anel é aproximado por segmentos cilíndricos em círculo, no
+         plano X-Z — furo voltado para o robô, para o gancho entrar de
+         frente e puxar.
        Continua sendo aproximação por primitivas, não réplica de CAD. -->
   <xacro:macro name="chave_seccionadora_lf" params="parent prefix:=chave_ xyz:='0 0 0' rpy:='0 0 0'">
-    <!-- ═══ Parâmetros ═══ -->
     <xacro:property name="olhal_height" value="0.810"/>      <!-- altura do olhal (spec do Marco) -->
     <xacro:property name="blade_length" value="0.200"/>      <!-- pivô → olhal -->
-    <xacro:property name="blade_angle" value="0.349"/>       <!-- 20° da vertical, posição fechada -->
     <xacro:property name="wall_standoff" value="0.03"/>      <!-- afastamento da face da parede -->
-    <!-- Placa branca de fundo (a que aparece na foto, parafusada na
-         parede e servindo de base para os dois brackets). -->
+    <!-- Placa de fundo (a branca da foto, parafusada na parede). -->
     <xacro:property name="plate_w" value="0.16"/>
     <xacro:property name="plate_h" value="0.62"/>
     <xacro:property name="plate_t" value="0.012"/>
-    <!-- Deslocamento do olhal em relação ao pivô, pela inclinação de
-         20° da lâmina fechada. Com o pivô EMBAIXO, o olhal sobe (+cos
-         em Z).
-         ROTAÇÃO DE 90° NO EIXO Z (correção do Marco, 2026-08-13): a
-         lâmina inclina no plano Y-Z, ou seja, PARA FORA da parede (na
-         direção de onde o robô se aproxima), não mais de lado ao longo
-         dela. Isso também põe a barra do olhal correndo paralela à
-         face da parede, como aparece na foto da bancada.
-         Implementado na geometria INTERNA do macro, não rotacionando a
-         instância: assim o wall_standoff continua empurrando a chave
-         para fora da parede (+Y). Rotacionar a instância giraria o
-         standoff junto e enfiaria a chave dentro da parede. -->
-    <xacro:property name="pivot_dz" value="${blade_length*cos(blade_angle)}"/>
-    <xacro:property name="pivot_dx" value="${blade_length*sin(blade_angle)}"/>
-    <!-- Origem do macro (bracket de montagem) = PIVÔ, embaixo. -->
-    <xacro:property name="pivot_z" value="${olhal_height - pivot_dz}"/>
-    <!-- ═══ Placa branca de fundo ═══ -->
+    <!-- Anel do olhal -->
+    <xacro:property name="ring_r" value="0.028"/>      <!-- raio do furo -->
+    <xacro:property name="ring_t" value="0.006"/>      <!-- espessura do arame -->
+    <xacro:property name="ring_seg" value="10"/>       <!-- segmentos do círculo -->
+    <!-- Fechada: lâmina vertical, olhal direto acima do pivô. -->
+    <xacro:property name="pivot_z" value="${olhal_height - blade_length}"/>
+    <!-- ═══ Placa de fundo ═══ -->
     <link name="${prefix}plate">
       <visual>
@@ -72,6 +59,5 @@
       <origin xyz="${xyz}" rpy="${rpy}"/>
     </joint>
-    <!-- ═══ Bracket inferior = PIVÔ da lâmina (chapa metálica chata,
-         parafusada na placa — a de baixo na foto) ═══ -->
+    <!-- ═══ Bracket inferior = PIVÔ ═══ -->
     <link name="${prefix}bracket">
       <visual>
@@ -94,6 +80,6 @@
       <origin xyz="0 0 0" rpy="0 0 0"/>
     </joint>
-    <!-- ═══ Bracket superior = contato fixo (a chapa de cima na foto,
-         com o furo no topo) ═══ -->
+    <!-- ═══ Bracket superior = contato fixo (a lâmina fechada encosta
+         nele) ═══ -->
     <link name="${prefix}fixed_terminal">
       <visual>
@@ -114,16 +100,15 @@
       <parent link="${prefix}plate"/>
       <child link="${prefix}fixed_terminal"/>
-      <origin xyz="0 0 ${pivot_dz + 0.16}" rpy="0 0 0"/>
+      <origin xyz="0 0 ${blade_length + 0.14}" rpy="0 0 0"/>
     </joint>
-    <!-- ═══ Lâmina móvel: SOBE do pivô até o olhal, inclinada ~20°
-         PARA FORA da parede (plano Y-Z) — o mecanismo escuro da foto ═══ -->
+    <!-- ═══ Lâmina móvel — VERTICAL (posição fechada) ═══ -->
     <link name="${prefix}blade">
       <visual>
-        <origin xyz="0 ${pivot_dx/2} ${blade_length/2}" rpy="${-blade_angle} 0 0"/>
+        <origin xyz="0 0 ${blade_length/2}"/>
         <geometry><box size="0.016 0.022 ${blade_length}"/></geometry>
         <material name="switch_dark"><color rgba="0.22 0.14 0.10 1"/></material>
       </visual>
       <collision>
-        <origin xyz="0 ${pivot_dx/2} ${blade_length/2}" rpy="${-blade_angle} 0 0"/>
+        <origin xyz="0 0 ${blade_length/2}"/>
         <geometry><box size="0.016 0.022 ${blade_length}"/></geometry>
       </collision>
@@ -138,17 +123,37 @@
       <origin xyz="0 ${wall_standoff} 0" rpy="0 0 0"/>
     </joint>
-    <!-- ═══ Olhal: a barra horizontal que atravessa o mecanismo na foto
-         — é onde a ferramenta engata. Este é o frame que o controlador
-         mira; fica no TOPO da lâmina, a 810 mm do chão. Eixo da barra
-         ao longo de X, ou seja, PARALELA à face da parede (é assim que
-         ela aparece na foto, atravessando o mecanismo de lado a lado). ═══ -->
+    <!-- ═══ OLHAL: anel no topo da lâmina, a 810 mm do chão. Este é o
+         frame que o controlador mira, e é por dentro dele que o gancho
+         da ferramenta passa.
+         O anel fica no plano X-Z (normal ao longo de Y), ou seja, com o
+         FURO VOLTADO PARA O ROBÔ — o gancho entra de frente e puxa.
+         Aproximado por ${ring_seg} cilindros curtos em círculo, já que
+         o URDF não tem toroide. A colisão é uma esfera única: o
+         contato fino do gancho no anel não é simulado nesta fase (a
+         tarefa é validada por posição do EE, não por contato). ═══ -->
     <link name="${prefix}olhal_link">
-      <visual>
-        <origin xyz="0 0 0" rpy="0 1.5708 0"/>
-        <geometry><cylinder radius="0.011" length="0.13"/></geometry>
-        <material name="galvanized"/>
-      </visual>
+      <xacro:macro name="ring_seg_vis" params="i">
+        <xacro:property name="a" value="${2*pi*i/ring_seg}"/>
+        <visual>
+          <origin xyz="${ring_r*cos(a)} 0 ${ring_r*sin(a)}"
+                  rpy="${pi/2} ${-a} 0"/>
+          <geometry>
+            <cylinder radius="${ring_t/2}" length="${2*pi*ring_r/ring_seg*1.15}"/>
+          </geometry>
+          <material name="galvanized"/>
+        </visual>
+      </xacro:macro>
+      <xacro:ring_seg_vis i="0"/>
+      <xacro:ring_seg_vis i="1"/>
+      <xacro:ring_seg_vis i="2"/>
+      <xacro:ring_seg_vis i="3"/>
+      <xacro:ring_seg_vis i="4"/>
+      <xacro:ring_seg_vis i="5"/>
+      <xacro:ring_seg_vis i="6"/>
+      <xacro:ring_seg_vis i="7"/>
+      <xacro:ring_seg_vis i="8"/>
+      <xacro:ring_seg_vis i="9"/>
       <collision>
-        <geometry><sphere radius="0.022"/></geometry>
+        <geometry><sphere radius="${ring_r}"/></geometry>
       </collision>
       <inertial>
@@ -160,9 +165,8 @@
       <parent link="${prefix}blade"/>
       <child link="${prefix}olhal_link"/>
-      <origin xyz="0 ${pivot_dx} ${pivot_dz}" rpy="0 0 0"/>
+      <origin xyz="0 0 ${blade_length}" rpy="0 0 0"/>
     </joint>
-    <!-- ═══ Materiais Gazebo explícitos — o <material><color> do URDF
-         some na fusão de corpo rígido da cadeia de juntas fixas
-         (comportamento confirmado ao vivo, ver histórico). ═══ -->
+    <!-- ═══ Materiais Gazebo explícitos (o <material><color> do URDF
+         some na fusão de corpo rígido da cadeia de juntas fixas) ═══ -->
     <gazebo reference="${prefix}plate">
       <material>Gazebo/White</material>
@@ -178,5 +182,5 @@
     </gazebo>
     <gazebo reference="${prefix}olhal_link">
-      <material>Gazebo/Grey</material>
+      <material>Gazebo/Orange</material>
     </gazebo>
   </xacro:macro>

File: src/b166er_robot/urdf/movemaster/movemaster.urdf.xacro (robot description, xacro)
@@ -362,16 +362,44 @@
       <child link="tool_tip"/>
     </joint>
-    <!-- tool_tip: frame na ponta do gancho — este é o frame que precisa
-         coincidir com chave_olhal_link quando a tarefa "engage"
-         converge. URDF não tem primitiva de toroide; o gancho é
-         aproximado por um disco fino, mesma convenção já usada em
-         chave_olhal_link (chave_seccionadora_lf.urdf.xacro). -->
+    <!-- tool_tip: frame no VÃO do gancho — o ponto onde o anel do
+         olhal se aloja quando engatado. É este frame que o controlador
+         mira, então o gancho é desenhado EM VOLTA da origem dele: se o
+         controlador leva tool_tip até o centro do olhal, o anel cai
+         dentro do vão.
+         Formato de gancho pedido pelo Marco (2026-08-13): "para
+         realizar a abertura a ferramenta deve ter na ponta um formato
+         de gancho". Antes era um disco chato, que não engancharia
+         nada. URDF não tem primitiva curva, então o gancho é
+         aproximado por segmentos retos: a haste continua um pouco além
+         do vão, curva e volta, formando um J aberto para o lado — o
+         anel entra pela abertura e fica preso no vão quando a
+         ferramenta puxa. -->
     <link name="tool_tip">
-      <visual>
-        <geometry><cylinder radius="0.015" length="0.006"/></geometry>
+      <!-- continuação da haste, passando o vão -->
+      <visual>
+        <origin xyz="0 0 -0.018" rpy="0 0 0"/>
+        <geometry><cylinder radius="0.006" length="0.05"/></geometry>
         <material name="ToolColor"/>
       </visual>
+      <!-- curva do gancho (dois segmentos inclinados) -->
+      <visual>
+        <origin xyz="0.016 0 -0.045" rpy="0 -0.9 0"/>
+        <geometry><cylinder radius="0.006" length="0.042"/></geometry>
+        <material name="ToolColor"/>
+      </visual>
+      <visual>
+        <origin xyz="0.038 0 -0.026" rpy="0 -2.0 0"/>
+        <geometry><cylinder radius="0.006" length="0.04"/></geometry>
+        <material name="ToolColor"/>
+      </visual>
+      <!-- bico do gancho, apontando de volta para a haste -->
+      <visual>
+        <origin xyz="0.040 0 0.003" rpy="0 -2.7 0"/>
+        <geometry><cylinder radius="0.005" length="0.026"/></geometry>
+        <material name="ToolColor"/>
+      </visual>
       <collision>
-        <geometry><sphere radius="0.018"/></geometry>
+        <origin xyz="0.018 0 -0.022"/>
+        <geometry><sphere radius="0.020"/></geometry>
       </collision>
     </link>

Commit message: feat(b166er_robot): a chave agora ABRE — junta revoluta na lâmina
O Marco observou que a chave não abria quando o robô puxava. Motivo:
ela não tinha junta nenhuma. O fixture inteiro era rígido
(blade_joint do tipo 'fixed') e o modelo era <static>true</static> —
modelo estático no Gazebo nem simula juntas. O robô podia encostar o
gancho no olhal com precisão perfeita que nada se moveria.

- blade_joint vira REVOLUTA em torno de X (lâmina gira no plano Y-Z,
  para fora da parede), curso 0 → 30°, com atrito alto (chave de
  manobra é dura, não cai sozinha nem oscila).
- O modelo deixa de ser <static> e passa a ser ancorado ao mundo por
  junta fixa ao link 'world' — mesmo efeito prático (a parede não sai
  do lugar) mas a lâmina fica livre.
- A missão gira a lâmina acompanhando o waypoint alcançado
  (set_blade_angle): 0° no engate, 15° em pos1, 30° em pos2.

O acoplamento é CINEMÁTICO, não por contato, e isso é uma escolha
deliberada documentada no código: puxar um anel com um gancho é
contato fino entre superfícies curvas, que o ODE com colisões
primitivas não resolve de forma confiável — a ferramenta atravessaria
ou escorregaria. O acoplamento cinemático mostra o movimento de
abertura corretamente, que é o que a missão precisa demonstrar, sem
mudar nada no que está sendo validado (navegação, percepção, alcance).

Verificado ao vivo: get_model_properties lista chave_blade_joint e
set_model_configuration responde success=True.

Co-Authored-By: Claude Opus 5 <noreply@anthropic.com>

File: src/b166er_robot/urdf/fixtures/chave_com_tag.urdf.xacro (robot description, xacro)
@@ -61,9 +61,17 @@
   <xacro:apriltag_mount parent="wall_link" prefix="tag_"
     xyz="${tag_x_offset} 0 ${tag_mount_z}" rpy="0 0 0"/>
-  <!-- Fixture inteira estática — nunca deve ser movida por física de
-       contato (é o alvo da tarefa, não um objeto manipulável nesta
-       fase). -->
-  <gazebo>
-    <static>true</static>
-  </gazebo>
+  <!-- A fixture NÃO pode mais ser <static>: modelo estático no Gazebo
+       não simula juntas, e a lâmina precisa girar para a chave abrir
+       (2026-08-13 — antes disso a chave era um bloco rígido e não
+       abria quando o robô puxava).
+       Em vez de 'static', a parede é ancorada ao mundo por uma junta
+       fixa ao link especial 'world'. Efeito prático igual — a parede
+       não sai do lugar por contato — mas a lâmina continua livre para
+       girar na sua junta revoluta. -->
+  <link name="world"/>
+  <joint name="world_anchor" type="fixed">
+    <parent link="world"/>
+    <child link="wall_link"/>
+    <origin xyz="0 0 0" rpy="0 0 0"/>
+  </joint>
 </robot>

File: src/b166er_robot/urdf/fixtures/chave_seccionadora_lf.urdf.xacro (robot description, xacro)
@@ -118,8 +118,19 @@
       </inertial>
     </link>
-    <joint name="${prefix}blade_joint" type="fixed">
+    <!-- JUNTA REAL DE ABERTURA (2026-08-13): era 'fixed', e por isso a
+         chave não abria de jeito nenhum quando o robô puxava — o Marco
+         notou. Agora é revoluta em torno de X, o que faz a lâmina
+         girar no plano Y-Z, para fora da parede. Curso 0 → 30°
+         (fechada → aberta), o mesmo confirmado pelo Marco. -->
+    <joint name="${prefix}blade_joint" type="revolute">
       <parent link="${prefix}bracket"/>
       <child link="${prefix}blade"/>
       <origin xyz="0 ${wall_standoff} 0" rpy="0 0 0"/>
+      <axis xyz="-1 0 0"/>
+      <limit lower="0.0" upper="0.60" effort="40" velocity="1.0"/>
+      <!-- Atrito alto: chave de manobra é dura, não cai sozinha pela
+           gravidade nem oscila. Também deixa a posição estável quando
+           o ângulo é imposto por set_model_configuration. -->
+      <dynamics damping="5.0" friction="8.0"/>
     </joint>
     <!-- ═══ OLHAL: anel no topo da lâmina, a 810 mm do chão. Este é o
