Commit message: feat: missão completa fecha de ponta a ponta (MISSION_OK)
Procura a tag, aproxima, abre a chave e volta ao ponto de partida.

TAG movida para o outro lado da chave e aproximada dela (pedidos do
Marco): de +0.20 para -0.42, separação de 0,40 m → 0,22 m. Parede
alargada para 1,6 m. Ficar perto reduz o braço de alavanca do erro
angular da detecção sobre a posição estimada do olhal.

BUG GRAVE que o Marco previu ao pedir a mudança ("ao mudar o lado da
tag, tem q alterar as direções no código também"):
apriltag_localizer.py tinha uma CÓPIA da constante TAG_OFFSET, ainda
com 0.20. A missão rodou inteira e terminou em MISSION_OK estimando a
parede 0,795 m fora do lugar — o robô "abriu a chave" a 80 cm de onde
ela está. Agora o localizador IMPORTA de chave_task; duplicar
geometria é exatamente o que aquele módulo existe para evitar.

IK ITERATIVA na manipulação fina (_reach_by_iterative_ik): mede a
ponta pelo T265, compara com o alvo e recomanda a IK mirando além, na
medida do que faltou. Fecha em 1-2 iterações.

E o controlador Cartesiano é DESLIGADO durante a manipulação: com ele
ativo seguia perseguindo o alvo antigo e movia a base enquanto a
missão comandava posturas, tirando a base do lugar para o qual a IK
tinha sido resolvida.

COLISÃO — a causa do engage nunca fechar, isolada por instrumentação
(logar q pedido vs q real) e por teste controlado (mesma postura longe
da parede: J4 falta 0,7°; no standoff: 6,3° — logo, colisão, não droop
nem IK):
· o olhal tinha colisão de ESFERA SÓLIDA de 28 mm "aproximando" o
  anel — para a física, uma bola maciça; o gancho batia nela em vez de
  atravessar. Removida (a abertura é acoplada cinematicamente).
· a lâmina idem, pelo mesmo motivo (o anel fica no topo dela).
· raiz geométrica: com wall_standoff de 3 cm o olhal ficava a 30 mm da
  face e o bracket ocupava até 28 mm — não cabia gancho nenhum. Subiu
  para 8 cm, o que também bate melhor com a foto da bancada (o
  mecanismo se projeta da placa). Folga passou de 2 mm para 52 mm.
· colisão do gancho afinada de 20 mm para 10 mm (é arame, não bola).

Medido: droop dos PIDs é pequeno nas posturas de trabalho (0,2-0,8°),
não os 3° que eu supunha — a hipótese de droop estava errada.
Modelo cinemático confere com o URDF em 0,2 mm.

Co-Authored-By: Claude Opus 5 <noreply@anthropic.com>

File: src/b166er_robot/urdf/fixtures/chave_com_tag.urdf.xacro (robot description, xacro)
@@ -18,9 +18,17 @@
   <xacro:include filename="$(find b166er_robot)/urdf/fixtures/apriltag_mount.urdf.xacro"/>
   <!-- ═══ Parâmetros da parede ═══ -->
-  <xacro:property name="wall_width" value="1.0"/>
+  <xacro:property name="wall_width" value="1.6"/>
   <xacro:property name="wall_thickness" value="0.10"/>
   <xacro:property name="wall_height" value="1.40"/>
   <xacro:property name="chave_x_offset" value="-0.20"/>
-  <xacro:property name="tag_x_offset" value="0.20"/>
+  <!-- Tag do OUTRO LADO da chave (pedido do Marco, 2026-08-13):
+       antes ficava em +0.20, com a chave em -0.20; agora do lado oposto.
+       Aproximada da chave em seguida (também a pedido do Marco): a
+       separação caiu de 0,40 m para 0,22 m, com a tag em -0.42.
+       Ficar perto importa para a percepção: quanto menor a distância
+       entre a tag e o alvo de manipulação, menor o braço de alavanca
+       do erro angular da detecção sobre a posição estimada do olhal.
+       A parede segue com 1,6 m de largura. -->
+  <xacro:property name="tag_x_offset" value="-0.42"/>
   <!-- Altura de montagem do macro da chave = altura do PIVÔ (embaixo),
        não mais do bracket sob o isolador. Precisa bater com o cálculo

File: src/b166er_robot/urdf/fixtures/chave_seccionadora_lf.urdf.xacro (robot description, xacro)
@@ -27,5 +27,15 @@
     <xacro:property name="olhal_height" value="0.810"/>      <!-- altura do olhal (spec do Marco) -->
     <xacro:property name="blade_length" value="0.200"/>      <!-- pivô → olhal -->
-    <xacro:property name="wall_standoff" value="0.03"/>      <!-- afastamento da face da parede -->
+    <!-- Afastamento do mecanismo em relação à placa. Subiu de 0,03 m
+         para 0,08 m em 2026-08-13, por dois motivos que convergem:
+         · FÍSICO: a foto da bancada mostra o mecanismo bem destacado da
+           placa (a barra e a articulação se projetam vários cm), não
+           colado como 3 cm sugeriam.
+         · FUNCIONAL: com 3 cm o olhal ficava a 30 mm da face, enquanto
+           o bracket ocupa até 28 mm — o gancho (esfera de colisão de
+           20 mm) não tinha por onde entrar. O J4 travava contra o
+           bracket e a ponta parava 5 cm aquém do alvo, sintoma que
+           levou horas a isolar porque parecia droop ou IK ruim. -->
+    <xacro:property name="wall_standoff" value="0.08"/>
     <!-- Placa de fundo (a branca da foto, parafusada na parede). -->
     <xacro:property name="plate_w" value="0.16"/>
@@ -109,8 +119,13 @@
         <material name="switch_dark"><color rgba="0.22 0.14 0.10 1"/></material>
       </visual>
-      <collision>
-        <origin xyz="0 0 ${blade_length/2}"/>
-        <geometry><box size="0.016 0.022 ${blade_length}"/></geometry>
-      </collision>
+      <!-- Lâmina SEM colisão, pelo mesmo motivo do olhal: o anel fica
+           no TOPO dela, então o gancho que mira o centro do anel
+           encosta na lâmina e trava. Medido: J4 cravado enquanto a IK
+           pedia de -41,9° a -2,9° (defasagem crescendo até 30,7°),
+           ponta congelada 5,7 cm aquém.
+           Colisão só faz sentido nas partes ESTRUTURAIS (placa,
+           brackets), que é onde o robô realmente não pode entrar. A
+           lâmina é o alvo da manipulação e sua abertura é acoplada
+           cinematicamente (set_blade_angle), não pelo contato. -->
       <inertial>
         <mass value="0.5"/>
@@ -165,7 +180,18 @@
       <xacro:ring_seg_vis i="8"/>
       <xacro:ring_seg_vis i="9"/>
-      <collision>
-        <geometry><sphere radius="${ring_r}"/></geometry>
-      </collision>
+      <!-- SEM COLISÃO no olhal (2026-08-13). Havia aqui uma esfera
+           sólida de raio ${ring_r} "aproximando" o anel — mas para a
+           física isso é uma BOLA MACIÇA, não um anel vazado: o gancho
+           batia nela em vez de atravessar. Sintoma medido: durante o
+           engate o J4 ficava cravado em ~-84° por mais que a IK
+           pedisse (-77,8° → -55,5°), a ponta congelada a 3 cm do alvo,
+           e a iteração só aumentava a defasagem (-5,1° → -29,8°).
+           Nada disso era droop nem IK ruim — era o gancho empurrando
+           uma esfera invisível.
+           Modelar o anel como toroide de colisão (vários cilindros)
+           seria caro e inútil aqui: a abertura da chave é acoplada
+           CINEMATICAMENTE (ver set_blade_angle em chave_mission.py),
+           não pelo contato gancho-anel. Sem colisão, o gancho alcança
+           o centro do anel, que é o que o controlador mira. -->
       <inertial>
         <mass value="0.08"/>

File: src/b166er_robot/urdf/movemaster/movemaster.urdf.xacro (robot description, xacro)
@@ -265,11 +265,24 @@
     </joint>
     <link name="task_camera_link">
-      <visual>
-        <geometry><box size="0.02 0.02 0.02"/></geometry>
-        <material name="ToolColor"/>
+      <!-- Corpo da câmera, deslocado para FORA da geometria do gripper.
+           Antes ficava na mesma origem do GripCube e sumia dentro dele
+           (o Marco: "a câmera não é visível na simulação") — o sensor
+           funcionava, mas não dava para ver onde estava nem para onde
+           apontava. O deslocamento é só VISUAL: o frame óptico, que é
+           o que importa para o PnP, continua na origem do link. -->
+      <visual>
+        <origin xyz="-0.03 0 0.035" rpy="0 0 0"/>
+        <geometry><box size="0.05 0.045 0.03"/></geometry>
+        <material name="CameraBody"><color rgba="0.05 0.05 0.05 1"/></material>
+      </visual>
+      <!-- Lente, apontando ao longo do eixo óptico (+X do link) -->
+      <visual>
+        <origin xyz="0.005 0 0.035" rpy="0 1.5708 0"/>
+        <geometry><cylinder radius="0.013" length="0.02"/></geometry>
+        <material name="CameraLens"><color rgba="0.15 0.3 0.55 1"/></material>
       </visual>
     </link>
     <gazebo reference="task_camera_link">
-      <material>Gazebo/Yellow</material>
+      <material>Gazebo/Blue</material>
       <sensor type="camera" name="task_camera">
         <update_rate>15.0</update_rate>
@@ -423,7 +436,10 @@
         <material name="ToolColor"/>
       </visual>
+      <!-- Colisão FINA (10 mm), condizente com um gancho de arame. A
+           esfera de 20 mm anterior tratava a ponta como uma bola e
+           batia em tudo perto do olhal. -->
       <collision>
         <origin xyz="0.018 0 -0.022"/>
-        <geometry><sphere radius="0.020"/></geometry>
+        <geometry><sphere radius="0.010"/></geometry>
       </collision>
     </link>
