Commit message: feat(lab): abertura por contato — anel com furo lateral, dedo fixo em L, seis fases
Remodela a manipulação a partir da geometria real da bancada, que o Marco
detalhou em desenho (Notebook 18, pág. 4) depois de eu errar a leitura
três vezes seguidas. O que estava modelado antes era invenção minha.

FIXTURE. O anel passa do plano XZ para o YZ: a normal vai de Y para X, ou
seja, o furo olha PARA O LADO e não para o robô. Não é aparência — é essa
normal que decide por onde a ferramenta entra. E o anel ganha colisão
segmento a segmento (10 cilindros), preservando o furo; a esfera
envolvente anterior fechava justamente o buraco por onde o gancho passa.
A lâmina também ganha colisão, mais estreita que o visual.

ATRITO DA JUNTA: 8,0 -> 1,5 N·m. Com abertura por contato o número deixa
de ser cosmético. O olhal fica a 200 mm do pivô, então 8 N·m exigiriam
40 N na ponta — muito acima do que um RV-M2 entrega (~12 N). O valor
antigo tornava a tarefa impossível pelo braço e ninguém percebia, porque
o ângulo era imposto por serviço do Gazebo.

FERRAMENTA. Sai o gancho em J (quatro cilindros de visual e UMA esfera de
colisão — uma esfera não engancha, empurra e escorrega) e entra o dedo
fixo do desenho do Marco: fixação, haste e degrau, 135 mm. Em vista
superior é um L — o degrau é um dedo HORIZONTAL ao longo de X, não um
bloco vertical como eu vinha modelando. Só assim atravessa um furo que
olha para o lado. Cada trecho com colisão de caixa igual ao visual.

Efeito colateral: montada na posição de um dedo do gripper (x=+30 mm), a
ponta deixa de ser coaxial com J5. |dponta/dJ5| sai de 0,000 para 0,030
m/rad — J5 sai do espaço nulo e vira grau de liberdade útil.

SEQUÊNCIA, agora com seis fases: aproxima_lateral, atravessa (degrau
entra pelo furo, +90 mm em X), captura (desce e apoia o arame),
arco1/arco2 (acompanha o arco com força pequena em Y) e DESENGATA (sai
lateralmente). A saída lateral não existia — antes a missão ia para o
recolhimento com a ferramenta ainda no anel, o que na bancada arrastaria
a chave.

O MISSION_OK passa a exigir a lâmina acima de 25° medidos, não o ângulo
que a própria missão impôs. Primeira execução com isso: as cinco fases
antigas fechavam em 2,8 mm e a lâmina ficava em 0,0° — a trajetória
estava certa e não havia geometria para prender.

Fica em aberto: o posicionamento com o lado do robô paralelo à parede
(sugestão do Marco) não foi implementado; a fase "atravessa" estaciona em
23,5 mm porque o braço não tem curso lateral a partir de uma postura já
estendida.

Co-Authored-By: Claude Opus 5 <noreply@anthropic.com>

File: src/b166er_robot/urdf/fixtures/chave_seccionadora_lf.urdf.xacro (robot description, xacro)
@@ -46,4 +46,15 @@
     <xacro:property name="ring_t" value="0.006"/>      <!-- espessura do arame -->
     <xacro:property name="ring_seg" value="10"/>       <!-- segmentos do círculo -->
+    <!-- ABERTURA POR CONTATO (2026-08-25). Com isto em true o olhal e a
+         lâmina ganham colisão e a chave passa a abrir porque o gancho
+         PUXA, não porque a missão comanda o ângulo por serviço do
+         Gazebo. É o que precisa valer para a bancada real ter sentido:
+         hoje o MISSION_OK prova que a ponta chegou aos waypoints, não
+         que a chave abriria.
+         Fica parametrizado porque o acoplamento cinemático continua
+         útil como regressão — separa "a trajetória está certa" de "a
+         força é suficiente", que são duas perguntas diferentes. -->
+    <xacro:property name="olhal_colide" value="true"/>
+    <xacro:property name="lamina_colide" value="true"/>
     <!-- Fechada: lâmina vertical, olhal direto acima do pivô. -->
     <xacro:property name="pivot_z" value="${olhal_height - blade_length}"/>
@@ -119,13 +130,20 @@
         <material name="switch_dark"><color rgba="0.22 0.14 0.10 1"/></material>
       </visual>
-      <!-- Lâmina SEM colisão, pelo mesmo motivo do olhal: o anel fica
-           no TOPO dela, então o gancho que mira o centro do anel
-           encosta na lâmina e trava. Medido: J4 cravado enquanto a IK
-           pedia de -41,9° a -2,9° (defasagem crescendo até 30,7°),
-           ponta congelada 5,7 cm aquém.
-           Colisão só faz sentido nas partes ESTRUTURAIS (placa,
-           brackets), que é onde o robô realmente não pode entrar. A
-           lâmina é o alvo da manipulação e sua abertura é acoplada
-           cinematicamente (set_blade_angle), não pelo contato. -->
+      <!-- Lâmina com colisão MAIS ESTREITA que o visual quando a
+           abertura é por contato. Ela ficou sem colisão em 2026-08-13
+           porque o gancho, mirando o centro do anel, encostava nela e
+           travava — mas isso era consequência do olhal ser uma esfera
+           maciça, que empurrava o gancho para trás. Com o anel vazado
+           de verdade o gancho passa pelo furo, e a lâmina precisa de
+           colisão: é ela que transmite o puxão até a junta.
+           A folga (colisão 60% da largura visual) existe porque o
+           contato aqui é lateral e rasante; apertar demais devolve o
+           travamento antigo por outro caminho. -->
+      <xacro:if value="${lamina_colide}">
+        <collision>
+          <origin xyz="0 0 ${blade_length/2}"/>
+          <geometry><box size="0.0096 0.0132 ${blade_length}"/></geometry>
+        </collision>
+      </xacro:if>
       <inertial>
         <mass value="0.5"/>
@@ -144,8 +162,18 @@
       <axis xyz="-1 0 0"/>
       <limit lower="0.0" upper="0.60" effort="40" velocity="1.0"/>
-      <!-- Atrito alto: chave de manobra é dura, não cai sozinha pela
-           gravidade nem oscila. Também deixa a posição estável quando
-           o ângulo é imposto por set_model_configuration. -->
-      <dynamics damping="5.0" friction="8.0"/>
+      <!-- ATRITO: PARÂMETRO A CALIBRAR CONTRA A CHAVE REAL.
+           Com a abertura por contato este número deixa de ser
+           cosmético e passa a decidir se a tarefa é possível.
+           Conta rápida: o olhal fica a ${blade_length} m do pivô, então
+           um atrito de F N·m exige uma força de F/${blade_length} N na
+           ponta do gancho. Com os 8 N·m anteriores seriam 40 N — muito
+           acima do que um RV-M2 entrega (carga útil ~1,2 kg ≈ 12 N).
+           Ou seja: o valor antigo tornava a tarefa infazível pelo braço,
+           e ninguém percebia porque o ângulo era imposto por serviço.
+           Baixado para 1,5 N·m (7,5 N na ponta), dentro do que o braço
+           faz. Se a chave real for mais dura que isso, a força terá de
+           vir da BASE — que é o que o recuo com as rodas já faz, e é
+           onde o whole-body ganha sentido físico. -->
+      <dynamics damping="0.5" friction="1.5"/>
     </joint>
     <!-- ═══ OLHAL: anel no topo da lâmina, a 810 mm do chão. Este é o
@@ -159,9 +187,18 @@
          tarefa é validada por posição do EE, não por contato). ═══ -->
     <link name="${prefix}olhal_link">
+      <!-- PLANO DO ANEL: contém Y e Z, normal em X (2026-08-26).
+           Antes o círculo era desenhado no plano XZ, com a normal em Y —
+           ou seja, o furo encarava o robô. Está errado: o Marco
+           descreveu que o furo olha PARA O LADO, e que atravessar o
+           olhal é um movimento perpendicular ao eixo Y.
+           Não é detalhe de aparência. É essa normal que decide por onde
+           a ferramenta entra: com o furo em X, o degrau do dedo fixo
+           avança paralelo à parede, e não contra ela. Todo o desenho da
+           ferramenta e a sequência de fases dependem disso. -->
       <xacro:macro name="ring_seg_vis" params="i">
         <xacro:property name="a" value="${2*pi*i/ring_seg}"/>
         <visual>
-          <origin xyz="${ring_r*cos(a)} 0 ${ring_r*sin(a)}"
-                  rpy="${pi/2} ${-a} 0"/>
+          <origin xyz="0 ${ring_r*cos(a)} ${ring_r*sin(a)}"
+                  rpy="0 ${pi/2} ${-a}"/>
           <geometry>
             <cylinder radius="${ring_t/2}" length="${2*pi*ring_r/ring_seg*1.15}"/>
@@ -169,4 +206,18 @@
           <material name="galvanized"/>
         </visual>
+        <!-- COLISÃO SEGMENTO A SEGMENTO, não uma primitiva envolvente.
+             É a diferença entre um anel e uma bola para o motor de
+             física: aproximar por esfera fecha o furo, que é justamente
+             por onde o gancho tem de passar. Cada cilindro é barato de
+             testar, e juntos preservam a topologia da peça. -->
+        <xacro:if value="${olhal_colide}">
+          <collision>
+            <origin xyz="0 ${ring_r*cos(a)} ${ring_r*sin(a)}"
+                    rpy="0 ${pi/2} ${-a}"/>
+            <geometry>
+              <cylinder radius="${ring_t/2}" length="${2*pi*ring_r/ring_seg*1.15}"/>
+            </geometry>
+          </collision>
+        </xacro:if>
       </xacro:macro>
       <xacro:ring_seg_vis i="0"/>

File: src/b166er_robot/urdf/movemaster/movemaster.urdf.xacro (robot description, xacro)
@@ -237,4 +237,49 @@
       </visual>
     </link>
+    <!-- ═══ FISHEYE 1 DA T265 — a câmera que o robô REALMENTE tem ═══
+         Acrescentada em 2026-08-26 depois de o Marco reforçar que a
+         bancada não tem a câmera de tarefa: ela foi invenção minha para
+         destravar a percepção em simulação, e tudo que validamos com
+         ela (alcance de detecção, ponto cego no standoff, taxa de
+         acerto do SEARCH) não valia para o robô real.
+         Aqui a simulação passa a exercitar EXATAMENTE o mesmo caminho
+         do hardware: mesmos tópicos (/camera/fisheye1/*), mesmo modelo
+         de lente, mesma resolução.
+         wideanglecamera com lente EQUIDISTANTE: é o modelo da T265
+         (Kannala-Brandt). Usar uma câmera pinhole comum aqui daria
+         números otimistas — a distorção fisheye é justamente o que
+         degrada o PnP longe do centro do quadro.
+         848x800 e ~157° de FOV horizontal são as specs da T265. Isso dá
+         5,4 px/grau contra 7,4 da câmera que inventei: mais campo,
+         menos resolução angular. Consequência já calculada: a detecção
+         confiável com a tag de 220 mm cai de ~3,9 m para ~2,8 m. ═══ -->
+    <gazebo reference="t265_link">
+      <sensor type="wideanglecamera" name="t265_fisheye1">
+        <update_rate>15.0</update_rate>
+        <always_on>1</always_on>
+        <visualize>false</visualize>
+        <camera>
+          <horizontal_fov>2.7367</horizontal_fov>
+          <image><width>848</width><height>800</height><format>R8G8B8</format></image>
+          <clip><near>0.05</near><far>50.0</far></clip>
+          <lens>
+            <type>equidistant</type>
+            <scale_to_hfov>true</scale_to_hfov>
+            <cutoff_angle>1.5707</cutoff_angle>
+            <env_texture_size>512</env_texture_size>
+          </lens>
+        </camera>
+        <plugin name="t265_fisheye1_controller" filename="libgazebo_ros_camera.so">
+          <cameraName>camera/fisheye1</cameraName>
+          <imageTopicName>image_raw</imageTopicName>
+          <!-- O camera_info do Gazebo vai para um tópico MORTO: ele
+               descreve a lente como pinhole e com fx errado. Quem publica
+               o /camera/fisheye1/camera_info é o fisheye_info_fixer. -->
+          <cameraInfoTopicName>camera_info_gazebo</cameraInfoTopicName>
+          <frameName>t265_link</frameName>
+          <hackBaseline>0.0</hackBaseline>
+        </plugin>
+      </sensor>
+    </gazebo>
     <!-- ═══ Câmera de tarefa (detecção de AprilTag) ═══
          Adicionada em 2026-08-12 pra fechar o loop de percepção pedido
@@ -377,7 +422,53 @@
          esse offset ao comandar o T265, não pode simplesmente mirar a
          ponta da ferramenta como se fosse o EE controlado. ═══ -->
-    <xacro:property name="tool_length" value="0.20"/>
+    <!-- ═══════════════════════════════════════════════════════════════
+         DEDO FIXO — ferramenta de manobra do Marco (desenho de
+         2026-08-25, Dedo_Fixo_RVM2_desenho.png).
+         Substitui os DEDOS do gripper, não o gripper: o garfo abraça a
+         lingueta original de 10 mm (vão 10,4 mm, 4 furos M3 por aba em
+         grade 2x2) e a garra não abre nem fecha durante a tarefa — ela
+         só transmite tração. Isso elimina o grau de liberdade que não
+         temos como controlar bem e transforma a garra num ponto de
+         ancoragem rígido.
+         Geometria do desenho (mm), ao longo de -Z a partir da montagem:
+           garfo   25 de altura, 20 de profundidade, abas de 10
+           afunil. 10
+           haste   80, seção 10,4 x 20,0
+           ponta   20 de altura, 30,4 de largura, 20 de profundidade
+           total  135
+         A ponta alargada é o que prende o elo: a haste de 10,4 mm passa
+         pelo olhal, e o degrau de 20 mm (30,4 − 10,4) impede o anel de
+         escapar quando o conjunto traciona. É o mesmo princípio do
+         gancho de vara de manobra convencional, que o Marco descreveu
+         como "gancho puxando um elo".
+         POR QUE ISTO SUBSTITUI O GANCHO EM J ANTERIOR: aquele tinha
+         quatro cilindros de VISUAL e UMA ESFERA de colisão. Uma esfera
+         não engata nada — empurra e escorrega. Foi por isso que a
+         primeira tentativa de abertura por contato terminou com a ponta
+         a 2,8 mm do alvo e a lâmina cravada em 0,0°: a trajetória
+         estava certa e não havia geometria para prender. Aqui cada
+         trecho tem colisão de caixa, com a mesma forma do visual.
+         ═══════════════════════════════════════════════════════════════ -->
+    <!-- Geometria do desenho (mm). A peça é um L: a haste sai do garfo
+         e o DEGRAU vira 90° no plano perpendicular a ela.
+         Corrigido em 2026-08-26 depois de o Marco apontar que a vista
+         superior do desenho é um L, não uma barra com um bloco. Eu vinha
+         lendo a vista superior como se fosse lateral e modelei o degrau
+         como um poste vertical. Ele é um DEDO HORIZONTAL — e só assim
+         atravessa um anel cujo furo olha para o lado (normal em X). -->
+    <xacro:property name="dedo_garfo_h"  value="0.025"/>
+    <xacro:property name="dedo_afun_h"   value="0.010"/>
+    <xacro:property name="dedo_haste_l"  value="0.080"/>
+    <xacro:property name="dedo_haste_x"  value="0.0104"/>
+    <xacro:property name="dedo_haste_y"  value="0.020"/>
+    <!-- Saliência do degrau além da haste: 30,4 − 10,4 = 20 mm. É o
+         comprimento útil que fica atravessado no furo e sustenta o
+         arame do olhal. -->
+    <xacro:property name="dedo_degrau_l" value="0.020"/>
+    <xacro:property name="dedo_degrau_z" value="0.017"/>
+    <xacro:property name="tool_length"
+                    value="${dedo_garfo_h + dedo_afun_h + dedo_haste_l}"/>
     <joint name="JTool" type="fixed">
-      <origin xyz="0 0 -0.08" rpy="0 0 0"/>
+      <origin xyz="0.03 0 -0.08" rpy="0 0 0"/>
       <parent link="GripCube"/>
       <child link="tool_rod"/>
@@ -385,12 +476,34 @@
     <link name="tool_rod">
       <visual>
-        <origin xyz="0 0 ${-tool_length/2}" rpy="0 0 0"/>
-        <geometry><cylinder radius="0.008" length="${tool_length}"/></geometry>
-        <material name="ToolColor"><color rgba="0.95 0.75 0.05 1"/></material>
+        <origin xyz="0 0 ${-dedo_garfo_h/2}"/>
+        <geometry><box size="0.020 0.025 ${dedo_garfo_h}"/></geometry>
+        <material name="ToolColor"><color rgba="0.85 0.75 0.1 1"/></material>
       </visual>
       <collision>
-        <origin xyz="0 0 ${-tool_length/2}" rpy="0 0 0"/>
-        <geometry><cylinder radius="0.008" length="${tool_length}"/></geometry>
+        <origin xyz="0 0 ${-dedo_garfo_h/2}"/>
+        <geometry><box size="0.020 0.025 ${dedo_garfo_h}"/></geometry>
       </collision>
+      <visual>
+        <origin xyz="0 0 ${-dedo_garfo_h - dedo_afun_h/2}"/>
+        <geometry><box size="0.015 0.022 ${dedo_afun_h}"/></geometry>
+        <material name="ToolColor"/>
+      </visual>
+      <collision>
+        <origin xyz="0 0 ${-dedo_garfo_h - dedo_afun_h/2}"/>
+        <geometry><box size="0.015 0.022 ${dedo_afun_h}"/></geometry>
+      </collision>
+      <visual>
+        <origin xyz="0 0 ${-dedo_garfo_h - dedo_afun_h - dedo_haste_l/2}"/>
+        <geometry><box size="${dedo_haste_x} ${dedo_haste_y} ${dedo_haste_l}"/></geometry>
+        <material name="ToolColor"/>
+      </visual>
+      <collision>
+        <origin xyz="0 0 ${-dedo_garfo_h - dedo_afun_h - dedo_haste_l/2}"/>
+        <geometry><box size="${dedo_haste_x} ${dedo_haste_y} ${dedo_haste_l}"/></geometry>
+      </collision>
+      <inertial>
+        <mass value="0.12"/>
+        <inertia ixx="0.0002" ixy="0" ixz="0" iyy="0.0002" iyz="0" izz="0.00002"/>
+      </inertial>
     </link>
     <joint name="JToolTip" type="fixed">
@@ -399,63 +512,26 @@
       <child link="tool_tip"/>
     </joint>
-    <!-- tool_tip: frame no VÃO do gancho — o ponto onde o anel do
-         olhal se aloja quando engatado. É este frame que o controlador
-         mira, então o gancho é desenhado EM VOLTA da origem dele: se o
-         controlador leva tool_tip até o centro do olhal, o anel cai
-         dentro do vão.
-         Formato de gancho pedido pelo Marco (2026-08-13): "para
-         realizar a abertura a ferramenta deve ter na ponta um formato
-         de gancho". Antes era um disco chato, que não engancharia
-         nada. URDF não tem primitiva curva, então o gancho é
-         aproximado por segmentos retos: a haste continua um pouco além
-         do vão, curva e volta, formando um J aberto para o lado — o
-         anel entra pela abertura e fica preso no vão quando a
-         ferramenta puxa. -->
+    <!-- DEGRAU — o dedo horizontal que atravessa o olhal.
+         Sai em −X a partir do eixo da haste; girando J5 a peça aponta
+         para a direita ou para a esquerda, como o Marco descreveu.
+         A ORIGEM DESTE LINK é a referência da tarefa: é aqui que o
+         arame do anel repousa depois da descida de 5 mm. -->
     <link name="tool_tip">
-      <!-- continuação da haste, passando o vão -->
-      <visual>
-        <origin xyz="0 0 -0.018" rpy="0 0 0"/>
-        <geometry><cylinder radius="0.006" length="0.05"/></geometry>
-        <material name="ToolColor"/>
-      </visual>
-      <!-- curva do gancho (dois segmentos inclinados) -->
-      <visual>
-        <origin xyz="0.016 0 -0.045" rpy="0 -0.9 0"/>
-        <geometry><cylinder radius="0.006" length="0.042"/></geometry>
-        <material name="ToolColor"/>
-      </visual>
-      <visual>
-        <origin xyz="0.038 0 -0.026" rpy="0 -2.0 0"/>
-        <geometry><cylinder radius="0.006" length="0.04"/></geometry>
-        <material name="ToolColor"/>
-      </visual>
-      <!-- bico do gancho, apontando de volta para a haste -->
-      <visual>
-        <origin xyz="0.040 0 0.003" rpy="0 -2.7 0"/>
-        <geometry><cylinder radius="0.005" length="0.026"/></geometry>
-        <material name="ToolColor"/>
-      </visual>
-      <!-- Colisão FINA (10 mm), condizente com um gancho de arame. A
-           esfera de 20 mm anterior tratava a ponta como uma bola e
-           batia em tudo perto do olhal. -->
+      <visual>
+        <origin xyz="${-dedo_degrau_l/2} 0 ${-dedo_degrau_z/2}"/>
+        <geometry><box size="${dedo_degrau_l + dedo_haste_x} ${dedo_haste_y} ${dedo_degrau_z}"/></geometry>
+        <material name="ToolColor"><color rgba="0.85 0.75 0.1 1"/></material>
+      </visual>
       <collision>
-        <origin xyz="0.018 0 -0.022"/>
-        <geometry><sphere radius="0.010"/></geometry>
+        <origin xyz="${-dedo_degrau_l/2} 0 ${-dedo_degrau_z/2}"/>
+        <geometry><box size="${dedo_degrau_l + dedo_haste_x} ${dedo_haste_y} ${dedo_degrau_z}"/></geometry>
       </collision>
-    </link>
-    <!-- <material><color> puro do URDF some na fusão de corpo rígido do
-         Gazebo (mesmo comportamento documentado em
-         chave_seccionadora_lf.urdf.xacro) — só os dois links novos da
-         ferramenta ganham <gazebo reference> aqui; o resto da árvore
-         fixa do EE (CameraSupport/GripCube/Grip1/Grip2) já tinha esse
-         problema antes desta mudança e fica fora de escopo. -->
-    <gazebo reference="tool_rod">
-      <material>Gazebo/Yellow</material>
-    </gazebo>
-    <gazebo reference="tool_tip">
-      <material>Gazebo/Yellow</material>
-    </gazebo>
-    <!-- ── Transmissões para ros_control (Gazebo) ───────────────────── -->
-    <!-- VelocityJointInterface: controladores de velocidade para cada junta -->
+      <inertial>
+        <mass value="0.04"/>
+        <inertia ixx="0.00002" ixy="0" ixz="0" iyy="0.00002" iyz="0" izz="0.00002"/>
+      </inertial>
+    </link>
+    <gazebo reference="tool_rod"><material>Gazebo/Yellow</material></gazebo>
+    <gazebo reference="tool_tip"><material>Gazebo/Yellow</material></gazebo>
     <xacro:macro name="arm_transmission" params="joint_name">
       <transmission name="${joint_name}_trans">
