Commit message: fix(b166er_robot): olhal com as medidas de trena da bancada
olhal-dimension.png (2026-08-26) trocou estimativa por medição:

  altura do centro do olhal   0,810 -> 0,805 m
  afastamento da parede       0,08  -> 0,13  m
  furo                        círculo Ø56 -> OVAL 40 (Z) x 30 (Y) mm

O formato do furo é o que importa: o degrau do dedo fixo atravessa com
seção 20 (Y) x 17 (Z) mm, então o furo real dá 5 mm de folga por lado em
Y, contra os 18 mm que o círculo inventado prometia. A simulação estava
escondendo justamente a tolerância que a tarefa precisa vencer.

Corrige também a orientação dos segmentos do anel: a rotação
rpy="0 pi/2 -a" era herdada de quando o anel vivia no plano XZ e, depois
que as posições foram para YZ, apontava os cilindros para FORA do plano
— o "anel" era um punhado de espetos com colisão na boca do furo. Agora
o eixo de cada segmento é a tangente do oval no ponto.

Os braços do pivô e do terminal fixo passam a ter profundidade igual ao
standoff; com 13 cm, a caixa de 20 mm anterior deixaria o pivô no ar.

Co-Authored-By: Claude Opus 5 <noreply@anthropic.com>
Claude-Session: https://claude.ai/code/session_01Ra2BbYQxYWhbcCFkGE7vAN

File: src/b166er_robot/urdf/fixtures/chave_seccionadora_lf.urdf.xacro (robot description, xacro)
@@ -18,32 +18,50 @@
          lâmina encosta no contato fixo de cima; abrir é girá-la 30°
          para fora (curso confirmado pelo Marco).
-       · OLHAL É UM ANEL, não uma barra. É por dentro dele que o gancho
-         da ferramenta passa. URDF não tem primitiva de toroide, então
-         o anel é aproximado por segmentos cilíndricos em círculo, no
-         plano X-Z — furo voltado para o robô, para o gancho entrar de
-         frente e puxar.
+       · OLHAL É UM ANEL OVAL, não uma barra e não um círculo. É por
+         dentro dele que o degrau do dedo fixo passa. URDF não tem
+         primitiva de toroide, então o anel é aproximado por segmentos
+         cilíndricos, no plano Y-Z — FURO VOLTADO PARA O LADO (normal em
+         X), como o Marco descreveu e como a foto da bancada mostra.
        Continua sendo aproximação por primitivas, não réplica de CAD. -->
   <xacro:macro name="chave_seccionadora_lf" params="parent prefix:=chave_ xyz:='0 0 0' rpy:='0 0 0'">
-    <xacro:property name="olhal_height" value="0.810"/>      <!-- altura do olhal (spec do Marco) -->
+    <!-- MEDIDO NA BANCADA REAL em 2026-08-26 (olhal-dimension.png):
+         centro do olhal a 80,5 cm do chão. Era 0,810 por estimativa. -->
+    <xacro:property name="olhal_height" value="0.805"/>
     <xacro:property name="blade_length" value="0.200"/>      <!-- pivô → olhal -->
-    <!-- Afastamento do mecanismo em relação à placa. Subiu de 0,03 m
-         para 0,08 m em 2026-08-13, por dois motivos que convergem:
-         · FÍSICO: a foto da bancada mostra o mecanismo bem destacado da
-           placa (a barra e a articulação se projetam vários cm), não
-           colado como 3 cm sugeriam.
-         · FUNCIONAL: com 3 cm o olhal ficava a 30 mm da face, enquanto
-           o bracket ocupa até 28 mm — o gancho (esfera de colisão de
-           20 mm) não tinha por onde entrar. O J4 travava contra o
-           bracket e a ponta parava 5 cm aquém do alvo, sintoma que
-           levou horas a isolar porque parecia droop ou IK ruim. -->
-    <xacro:property name="wall_standoff" value="0.08"/>
+    <!-- Afastamento do mecanismo em relação à face da placa.
+         Foi 0,03 (estimado da foto) → 0,08 (estimado de novo, para o
+         gancho ter por onde entrar) → 0,13 MEDIDO com trena na bancada
+         em 2026-08-26 (olhal-dimension.png): o centro do olhal está a
+         13 cm da parede.
+         Os 5 cm a mais em relação ao chute anterior não são cosméticos:
+         é a folga entre a ferramenta e a parede durante o engate, e é
+         justamente onde o manipulador vinha entrando dentro da parede
+         nas simulações. -->
+    <xacro:property name="wall_standoff" value="0.13"/>
     <!-- Placa de fundo (a branca da foto, parafusada na parede). -->
     <xacro:property name="plate_w" value="0.16"/>
     <xacro:property name="plate_h" value="0.62"/>
     <xacro:property name="plate_t" value="0.012"/>
-    <!-- Anel do olhal -->
-    <xacro:property name="ring_r" value="0.028"/>      <!-- raio do furo -->
-    <xacro:property name="ring_t" value="0.006"/>      <!-- espessura do arame -->
-    <xacro:property name="ring_seg" value="10"/>       <!-- segmentos do círculo -->
+    <!-- ═══ Anel do olhal — OVAL, medido em 2026-08-26 ═══
+         O anel nunca foi um círculo de 28 mm de raio. Medidas reais
+         (olhal-dimension.png), no plano do anel:
+                       vertical (Z)   horizontal (Y)
+           furo interno   40 mm          30 mm
+           externo        55 mm          40 mm
+           => arame        7,5 mm         5 mm  -> ~6 mm de bitola
+         Os semi-eixos abaixo são da LINHA DE CENTRO do arame
+         (interno + metade da bitola), que é onde os cilindros ficam:
+           Z: 20 + 3 = 23 mm      Y: 15 + 3 = 18 mm
+         Isso devolve externo 52 x 42 mm contra os 55 x 40 medidos.
+         POR QUE O FORMATO IMPORTA: o degrau do dedo fixo atravessa o
+         furo com seção 20 mm (Y) x 17 mm (Z). No furo real de 30 x 40
+         isso passa com 5 mm de folga de cada lado em Y — e Y é a
+         direção apertada. Com o círculo de 56 mm que estava aqui, a
+         simulação dava 18 mm de folga onde a bancada dá 5, ou seja,
+         escondia exatamente a tolerância que a tarefa precisa vencer. -->
+    <xacro:property name="ring_ay" value="0.018"/>     <!-- semi-eixo horizontal (perpendicular à parede) -->
+    <xacro:property name="ring_az" value="0.023"/>     <!-- semi-eixo vertical -->
+    <xacro:property name="ring_t" value="0.006"/>      <!-- bitola do arame -->
+    <xacro:property name="ring_seg" value="12"/>       <!-- segmentos do oval -->
     <!-- ABERTURA POR CONTATO (2026-08-25). Com isto em true o olhal e a
          lâmina ganham colisão e a chave passa a abrir porque o gancho
@@ -80,14 +98,19 @@
       <origin xyz="${xyz}" rpy="${rpy}"/>
     </joint>
-    <!-- ═══ Bracket inferior = PIVÔ ═══ -->
+    <!-- ═══ Bracket inferior = PIVÔ ═══
+         O braço vai da face da placa até o pivô, então sua PROFUNDIDADE
+         é o próprio wall_standoff. Antes era uma caixa de 20 mm plantada
+         a 0,6·standoff, o que com 8 cm quase alcançava o pivô por acaso;
+         com os 13 cm medidos ficaria um bloco solto no ar, com o pivô
+         fora dele. -->
     <link name="${prefix}bracket">
       <visual>
-        <origin xyz="0 ${wall_standoff*0.6} 0"/>
-        <geometry><box size="0.045 0.020 0.14"/></geometry>
+        <origin xyz="0 ${wall_standoff/2} 0"/>
+        <geometry><box size="0.045 ${wall_standoff} 0.14"/></geometry>
         <material name="galvanized"><color rgba="0.55 0.55 0.58 1"/></material>
       </visual>
       <collision>
-        <origin xyz="0 ${wall_standoff*0.6} 0"/>
-        <geometry><box size="0.045 0.020 0.14"/></geometry>
+        <origin xyz="0 ${wall_standoff/2} 0"/>
+        <geometry><box size="0.045 ${wall_standoff} 0.14"/></geometry>
       </collision>
       <inertial>
@@ -105,11 +128,11 @@
     <link name="${prefix}fixed_terminal">
       <visual>
-        <origin xyz="0 ${wall_standoff*0.6} 0"/>
-        <geometry><box size="0.045 0.020 0.19"/></geometry>
+        <origin xyz="0 ${wall_standoff/2} 0"/>
+        <geometry><box size="0.045 ${wall_standoff} 0.19"/></geometry>
         <material name="galvanized"/>
       </visual>
       <collision>
-        <origin xyz="0 ${wall_standoff*0.6} 0"/>
-        <geometry><box size="0.045 0.020 0.19"/></geometry>
+        <origin xyz="0 ${wall_standoff/2} 0"/>
+        <geometry><box size="0.045 ${wall_standoff} 0.19"/></geometry>
       </collision>
       <inertial>
@@ -177,13 +200,12 @@
       <dynamics damping="0.5" friction="1.5"/>
     </joint>
-    <!-- ═══ OLHAL: anel no topo da lâmina, a 810 mm do chão. Este é o
-         frame que o controlador mira, e é por dentro dele que o gancho
-         da ferramenta passa.
-         O anel fica no plano X-Z (normal ao longo de Y), ou seja, com o
-         FURO VOLTADO PARA O ROBÔ — o gancho entra de frente e puxa.
-         Aproximado por ${ring_seg} cilindros curtos em círculo, já que
-         o URDF não tem toroide. A colisão é uma esfera única: o
-         contato fino do gancho no anel não é simulado nesta fase (a
-         tarefa é validada por posição do EE, não por contato). ═══ -->
+    <!-- ═══ OLHAL: anel oval no topo da lâmina, a 805 mm do chão e a
+         130 mm da parede (medidos). Este é o frame que o controlador
+         mira, e é por dentro dele que o degrau do dedo fixo passa.
+         O anel fica no plano Y-Z (normal ao longo de X): o FURO OLHA
+         PARA O LADO, e atravessá-lo é um movimento paralelo à parede.
+         Aproximado por ${ring_seg} cilindros curtos, já que o URDF não
+         tem toroide, e cada um com colisão própria — ver a nota sobre
+         por que uma primitiva envolvente não serve. ═══ -->
     <link name="${prefix}olhal_link">
       <!-- PLANO DO ANEL: contém Y e Z, normal em X (2026-08-26).
@@ -196,11 +218,32 @@
            avança paralelo à parede, e não contra ela. Todo o desenho da
            ferramenta e a sequência de fases dependem disso. -->
+      <!-- ORIENTAÇÃO DOS SEGMENTOS — corrigida em 2026-08-27.
+           A versão anterior tinha rpy="0 pi/2 -a", herdada de quando o
+           anel era desenhado no plano XZ. Depois que as POSIÇÕES foram
+           levadas para o plano YZ, essa rotação passou a apontar os
+           cilindros para FORA do plano do anel (eixo em (cos a, -sen a,
+           0), que vive no plano XY): o "anel" era na verdade um punhado
+           de espetos saindo de lado. Como cada cilindro também tem
+           colisão, isso plantava obstáculos bem na boca do furo.
+           Agora o eixo é a tangente do oval no ponto, obtida do próprio
+           parâmetro: um cilindro alinhado com +Z local vira (0, -sen θ,
+           cos θ) com um roll θ, e θ = atan2(-dy, dz) sobre a corda do
+           segmento. Para o círculo isso dá θ = a; para o oval corrige a
+           inclinação onde os semi-eixos diferem.
+           O comprimento também vem da corda (não de 2πr/n, que só vale
+           para círculo), com 15% de sobreposição para não deixar frestas
+           nas emendas. -->
       <xacro:macro name="ring_seg_vis" params="i">
-        <xacro:property name="a" value="${2*pi*i/ring_seg}"/>
+        <xacro:property name="a"  value="${2*pi*i/ring_seg}"/>
+        <xacro:property name="h"  value="${pi/ring_seg}"/>
+        <xacro:property name="dy" value="${ring_ay*(cos(a+h) - cos(a-h))}"/>
+        <xacro:property name="dz" value="${ring_az*(sin(a+h) - sin(a-h))}"/>
+        <xacro:property name="seg_len" value="${1.15*sqrt(dy*dy + dz*dz)}"/>
+        <xacro:property name="seg_roll" value="${atan2(-dy, dz)}"/>
         <visual>
-          <origin xyz="0 ${ring_r*cos(a)} ${ring_r*sin(a)}"
-                  rpy="0 ${pi/2} ${-a}"/>
+          <origin xyz="0 ${ring_ay*cos(a)} ${ring_az*sin(a)}"
+                  rpy="${seg_roll} 0 0"/>
           <geometry>
-            <cylinder radius="${ring_t/2}" length="${2*pi*ring_r/ring_seg*1.15}"/>
+            <cylinder radius="${ring_t/2}" length="${seg_len}"/>
           </geometry>
           <material name="galvanized"/>
@@ -213,8 +256,8 @@
         <xacro:if value="${olhal_colide}">
           <collision>
-            <origin xyz="0 ${ring_r*cos(a)} ${ring_r*sin(a)}"
-                    rpy="0 ${pi/2} ${-a}"/>
+            <origin xyz="0 ${ring_ay*cos(a)} ${ring_az*sin(a)}"
+                    rpy="${seg_roll} 0 0"/>
             <geometry>
-              <cylinder radius="${ring_t/2}" length="${2*pi*ring_r/ring_seg*1.15}"/>
+              <cylinder radius="${ring_t/2}" length="${seg_len}"/>
             </geometry>
           </collision>
@@ -231,18 +274,16 @@
       <xacro:ring_seg_vis i="8"/>
       <xacro:ring_seg_vis i="9"/>
-      <!-- SEM COLISÃO no olhal (2026-08-13). Havia aqui uma esfera
-           sólida de raio ${ring_r} "aproximando" o anel — mas para a
-           física isso é uma BOLA MACIÇA, não um anel vazado: o gancho
-           batia nela em vez de atravessar. Sintoma medido: durante o
-           engate o J4 ficava cravado em ~-84° por mais que a IK
-           pedisse (-77,8° → -55,5°), a ponta congelada a 3 cm do alvo,
-           e a iteração só aumentava a defasagem (-5,1° → -29,8°).
-           Nada disso era droop nem IK ruim — era o gancho empurrando
-           uma esfera invisível.
-           Modelar o anel como toroide de colisão (vários cilindros)
-           seria caro e inútil aqui: a abertura da chave é acoplada
-           CINEMATICAMENTE (ver set_blade_angle em chave_mission.py),
-           não pelo contato gancho-anel. Sem colisão, o gancho alcança
-           o centro do anel, que é o que o controlador mira. -->
+      <xacro:ring_seg_vis i="10"/>
+      <xacro:ring_seg_vis i="11"/>
+      <!-- HISTÓRICO, para não repetir: em 2026-08-13 havia aqui uma
+           ESFERA sólida "aproximando" o anel. Para a física isso é uma
+           bola maciça, não um anel vazado: o gancho batia nela em vez
+           de atravessar. Sintoma medido — durante o engate o J4 ficava
+           cravado em ~-84° por mais que a IK pedisse (-77,8° → -55,5°),
+           a ponta congelada a 3 cm do alvo, e a iteração só aumentava a
+           defasagem (-5,1° → -29,8°). Não era droop nem IK ruim: era o
+           gancho empurrando uma esfera invisível.
+           Por isso a colisão hoje é segmento a segmento (acima): é a
+           única forma de o furo continuar sendo furo. -->
       <inertial>
         <mass value="0.08"/>

Commit message: feat(b166er_whole_body_control): IK com atitude do degrau; viés de mira corrigido
Primeira execução em que a lâmina SAI de 0,0° (chegou a 17,1°). As sete
fases fecham entre 7,2 e 18,4 mm.

VIÉS DE MIRA — decomposto e corrigido, de −16/−45/−14 mm para +5/+2/+2
(a 1,6 m). Quatro causas independentes, todas medidas:

· a placa da tag fica 22,5 mm à frente da parede (wall_standoff 0,02 +
  metade da espessura) e era tratada como se estivesse no plano;
· a posição da parede era calculada com a rotação CRUA do PnP, cujo tilt
  espúrio era multiplicado por um braço de 0,885 m — o vínculo de
  verticalidade (flatten_wall_R) existia mas era aplicado depois. Agora
  achata ANTES de alavancar. A dispersão do dZ caiu de 2,9 para 0,6 mm;
· cx/cy: a simulação publicava o ponto principal da câmera REAL enquanto
  o Gazebo renderiza centrado — 6,9 px de descasamento = 1,39°, igual ao
  erro de yaw medido. Era um viés que só existia na simulação;
· escala: o detector vê a tag renderizada 1,4% menor (borda sub-pixel).
  Corrigido por ~tag_size no launch de SIMULAÇÃO, não no código — o
  default segue 0,132, a tag física do Marco.

ATITUDE DO DEGRAU — ik_tooltip_nivelado: 2 de posição transversal (a
componente ao longo do eixo do furo pesa 0,15, não zero: é ela que
distingue aproxima_lateral de atravessa) + 3 de orientação. A atitude
pedida põe a LARGURA na vertical, que é a que o braço alcança e dá
folgas mais equilibradas (6,5 e 10 mm contra 5 e 11,5).

A escolha entre a IK nivelada e a de eixo é feita UMA VEZ POR FASE.
Decidir a cada iteração fez a fase aproxima_lateral, que fechava em
8,4 mm, falhar com 58 mm — o braço perseguia alvos que mudavam de
natureza a cada passo.

O terminal fixo volta a ser uma peça de 40 mm: eu tinha lhe dado a
profundidade inteira do standoff por simetria com o bracket do pivô, e
virou um bloco de 130x45x190 mm na trajetória (50 mil contatos numa
missão). Geometria real pendente de medição na bancada.

Co-Authored-By: Claude Opus 5 <noreply@anthropic.com>
Claude-Session: https://claude.ai/code/session_01Ra2BbYQxYWhbcCFkGE7vAN

File: src/b166er_robot/urdf/fixtures/chave_seccionadora_lf.urdf.xacro (robot description, xacro)
@@ -126,13 +126,26 @@
     <!-- ═══ Bracket superior = contato fixo (a lâmina fechada encosta
          nele) ═══ -->
+    <!-- PROFUNDIDADE DO TERMINAL: NÃO MEDIDA, e por isso conservadora.
+         Em 2026-08-27 eu dei a este bloco a profundidade inteira do
+         standoff (130 mm), por simetria com o bracket do pivô. O bracket
+         PRECISA disso — ele vai da parede até o pivô. O terminal fixo
+         não carrega pivô nenhum: é a peça de contato onde a lâmina
+         encosta quando fechada.
+         O resultado foi um bloco maciço de 130x45x190 mm bem na
+         trajetória da ferramenta: ~50 000 contatos ferramenta x terminal
+         numa única missão, e a fase "atravessa" travando com 51,7 mm de
+         resíduo — obstáculo que existe só no meu modelo.
+         Volta a ser uma peça de contato de 40 mm, no plano do mecanismo.
+         A geometria real está na lista de medições da bancada. -->
+    <xacro:property name="terminal_prof" value="0.040"/>
     <link name="${prefix}fixed_terminal">
       <visual>
-        <origin xyz="0 ${wall_standoff/2} 0"/>
-        <geometry><box size="0.045 ${wall_standoff} 0.19"/></geometry>
+        <origin xyz="0 ${wall_standoff} 0"/>
+        <geometry><box size="0.045 ${terminal_prof} 0.19"/></geometry>
         <material name="galvanized"/>
       </visual>
       <collision>
-        <origin xyz="0 ${wall_standoff/2} 0"/>
-        <geometry><box size="0.045 ${wall_standoff} 0.19"/></geometry>
+        <origin xyz="0 ${wall_standoff} 0"/>
+        <geometry><box size="0.045 ${terminal_prof} 0.19"/></geometry>
       </collision>
       <inertial>

Commit message: fix(b166er_robot): lâmina da chave termina antes do olhal
O anel do olhal é fixado em z = blade_length, e a barra da lâmina ia
de 0 até blade_length — ou seja, terminava no CENTRO do furo e tapava
a metade de baixo dele. A ferramenta só tinha uma fresta de ~20 mm por
cima, em vez dos 46 mm de abertura que o oval oferece.

Está errado como modelo: na chave real o olhal é uma alça na PONTA da
lâmina, e a alça é vazada. O Marco apontou olhando a cena.

A barra agora termina em blade_length - ring_az, encostando na borda
inferior do anel. A distância pivô→olhal segue sendo 0,200 m e o
centro do olhal segue a 0,805 m do chão, que são as medidas de
bancada — só a barra deixou de invadir o furo.

Co-Authored-By: Claude Opus 5 <noreply@anthropic.com>
Claude-Session: https://claude.ai/code/session_01Ra2BbYQxYWhbcCFkGE7vAN

File: src/b166er_robot/urdf/fixtures/chave_seccionadora_lf.urdf.xacro (robot description, xacro)
@@ -159,9 +159,22 @@
       <origin xyz="0 0 ${blade_length + 0.14}" rpy="0 0 0"/>
     </joint>
-    <!-- ═══ Lâmina móvel — VERTICAL (posição fechada) ═══ -->
+    <!-- ═══ Lâmina móvel — VERTICAL (posição fechada) ═══
+         A BARRA ACABA ANTES DO OLHAL, e o furo fica livre.
+         Até 2026-09-01 a lâmina ia de 0 a blade_length, e o anel é
+         fixado justamente em z = blade_length — ou seja, a barra
+         terminava no CENTRO do furo e tapava a metade de baixo dele. A
+         ferramenta só tinha uma fresta de 20 mm por cima, em vez dos 46
+         mm de abertura que o oval oferece.
+         Está errado como modelo: na chave real o olhal é uma alça na
+         PONTA da lâmina, e a alça é vazada. O Marco apontou olhando a
+         cena ("o olhal precisa estar livre").
+         Agora a barra termina em blade_length - ring_az, encostando na
+         borda inferior do anel. A distância pivô→olhal segue sendo
+         blade_length (0,200 m), que é a medida de bancada. -->
+    <xacro:property name="blade_bar" value="${blade_length - ring_az}"/>
     <link name="${prefix}blade">
       <visual>
-        <origin xyz="0 0 ${blade_length/2}"/>
-        <geometry><box size="0.016 0.022 ${blade_length}"/></geometry>
+        <origin xyz="0 0 ${blade_bar/2}"/>
+        <geometry><box size="0.016 0.022 ${blade_bar}"/></geometry>
         <material name="switch_dark"><color rgba="0.22 0.14 0.10 1"/></material>
       </visual>
@@ -178,6 +191,6 @@
       <xacro:if value="${lamina_colide}">
         <collision>
-          <origin xyz="0 0 ${blade_length/2}"/>
-          <geometry><box size="0.0096 0.0132 ${blade_length}"/></geometry>
+          <origin xyz="0 0 ${blade_bar/2}"/>
+          <geometry><box size="0.0096 0.0132 ${blade_bar}"/></geometry>
         </collision>
       </xacro:if>

Commit message: fix(robot): olhal com as medidas do lab — furo 40 × 28 mm, arame Ø 8 mm
Remedido pelo Marco em 28 Out 2026: furo interno 40 mm (Z) × 28 mm (Y),
arame de 8 mm. Era 40 × 30 com arame de 6 mm. Linha de centro do arame:
Z 23 → 24 mm, Y 18 mm (inalterado: o furo estreitou 2 mm e o arame
engrossou 2 mm). O centro do olhal continua a 200 mm do pivô.

Co-Authored-By: Claude Opus 5.5 <noreply@anthropic.com>
Claude-Session: https://claude.ai/code/session_01P4v3ZvEh2bwom2DYHA9moN

File: src/b166er_robot/urdf/fixtures/chave_seccionadora_lf.urdf.xacro (robot description, xacro)
@@ -60,7 +60,12 @@
          simulação dava 18 mm de folga onde a bancada dá 5, ou seja,
          escondia exatamente a tolerância que a tarefa precisa vencer. -->
+    <!-- REMEDIDO NO LAB (28 Out 2026, Marco, foto "posições iniciais da
+         chave"): furo interno 40 mm (Z) x 28 mm (Y), arame de Ø 8 mm.
+         Linha de centro: Z 20 + 4 = 24 mm, Y 14 + 4 = 18 mm (Y não muda:
+         o furo estreitou 2 mm e o arame engrossou 2 mm). Externo 56 x 44.
+         Antes: furo 40 x 30, arame 6 mm (estimado pela medida de 26 Ago). -->
     <xacro:property name="ring_ay" value="0.018"/>     <!-- semi-eixo horizontal (perpendicular à parede) -->
-    <xacro:property name="ring_az" value="0.023"/>     <!-- semi-eixo vertical -->
-    <xacro:property name="ring_t" value="0.006"/>      <!-- bitola do arame -->
+    <xacro:property name="ring_az" value="0.024"/>     <!-- semi-eixo vertical (era 0,023) -->
+    <xacro:property name="ring_t" value="0.008"/>      <!-- bitola do arame (era 0,006) -->
     <xacro:property name="ring_seg" value="12"/>       <!-- segmentos do oval -->
     <!-- ABERTURA POR CONTATO (2026-08-25). Com isto em true o olhal e a
