Commit message: fix(sim): move T265 do chassi para o end-effector do braço
Confirmado por foto do robô real: a T265 fica montada no end-effector
do RV-M2, na mesma região do gripper — não no chassi do Pioneer. O
mount de câmera que já existia no CAD do braço (CameraSupport/d400_link)
já estava posicionado exatamente ali, só com nome genérico; renomeado
para t265_link/t265_mount_joint em vez de duplicar a geometria. O
Hokuyo permanece no top_plate do Pioneer, como já estava.

Co-Authored-By: Claude Sonnet 4.6 <noreply@anthropic.com>

File: src/b166er_robot/urdf/b166er.urdf.xacro (robot description, xacro)
@@ -2,28 +2,13 @@
 <robot name="b166er" xmlns:xacro="http://ros.org/wiki/xacro">
   <!-- Modelo unificado do b166er: base Pioneer 3-AT (com sonares e rodas
-       reais) + braço Mitsubishi RV-M2 + câmera T265 + laser Hokuyo
-       UST-05LX. Reaproveita os dois modelos já existentes com malhas
-       reais em vez de recriar geometria do zero. -->
+       reais) + braço Mitsubishi RV-M2 (com a T265 montada no end-effector,
+       na região do gripper) + laser Hokuyo UST-05LX na base superior do
+       Pioneer. Reaproveita os dois modelos já existentes com malhas reais
+       em vez de recriar geometria do zero. -->
   <xacro:include filename="$(find b166er_robot)/urdf/pioneer3at/pioneer3at-m.urdf.xacro"/>
   <xacro:include filename="$(find b166er_robot)/urdf/movemaster/movemaster.urdf.xacro"/>
-  <!-- Braço montado sobre o top_plate do Pioneer -->
+  <!-- Braço montado sobre o top_plate do Pioneer (a T265 vem junto, montada
+       no end-effector do braço — ver t265_mount_joint em movemaster.urdf.xacro) -->
   <xacro:movemaster_rv_m2 parent="top_plate" xyz="0.05 0 0.02" rpy="0 0 0"/>
-  <!-- Intel RealSense T265 — sensor de pose visual-inercial (Pilar 1: navegação) -->
-  <joint name="t265_mount_joint" type="fixed">
-    <parent link="top_plate"/>
-    <child link="t265_link"/>
-    <origin xyz="0.26 0 0.05" rpy="0 0 0"/>
-  </joint>
-  <link name="t265_link">
-    <visual>
-      <origin xyz="0 0 0" rpy="0 0 0"/>
-      <geometry>
-        <mesh filename="package://movemaster_control/3D_Models/realsense.stl"/>
-      </geometry>
-      <material name="t265_color">
-        <color rgba="0.1 0.1 0.1 1.0"/>
-      </material>
-    </visual>
-  </link>
   <!-- Hokuyo UST-05LX (Smart URG) — FOV 270°, alcance 0.06-5.0 m,
        resolução angular 0.25° (1081 amostras). Reaproveita o macro

File: src/b166er_robot/urdf/movemaster/movemaster.urdf.xacro (robot description, xacro)
@@ -128,10 +128,11 @@
       </visual>
     </link>
-    <joint name="DepthCamera" type="fixed">
+    <!-- T265 montada no end-effector, mesma região do gripper (confirmado por foto do robô real) -->
+    <joint name="t265_mount_joint" type="fixed">
       <origin xyz="0 0.075 -0.070" rpy="0 2.1 1.57"/>
       <parent link="CameraSupport"/>
-      <child link="d400_link"/>
+      <child link="t265_link"/>
     </joint>
-    <link name="d400_link">
+    <link name="t265_link">
       <visual>
         <origin xyz="0 0 0" rpy="0 0 0"/>
@@ -139,6 +140,6 @@
           <mesh filename="package://movemaster_control/3D_Models/realsense.stl"/>
         </geometry>
-        <material name="realsensecolor">
-          <color rgba="0.25 0.25 0.25 0"/>
+        <material name="t265_color">
+          <color rgba="0.1 0.1 0.1 1.0"/>
         </material>
       </visual>

Commit message: fix(urdf): posições reais dos sensores conforme foto e medição do robô
- Braço RV-M2: centralizado no meio dos eixos da plataforma (x=0 em top_plate)
- Hokuyo UST-05LX: 2,5 cm da frente da plataforma, assentado no top_plate (z=0.025)
- IMU Sparton AHRS-8: movida para face traseira de L1 (bunda do manipulador,
  eixo 2) em xyz="-0.05 0 0.02", confirmado por foto e ajuste visual no RViz
- b166er_rviz.launch: use_sim_time=false para evitar trava sem roscore do Gazebo

Co-Authored-By: Claude Sonnet 4.6 <noreply@anthropic.com>

File: src/b166er_robot/urdf/b166er.urdf.xacro (robot description, xacro)
@@ -8,13 +8,12 @@
   <xacro:include filename="$(find b166er_robot)/urdf/pioneer3at/pioneer3at-m.urdf.xacro"/>
   <xacro:include filename="$(find b166er_robot)/urdf/movemaster/movemaster.urdf.xacro"/>
-  <!-- Braço montado sobre o top_plate do Pioneer (a T265 vem junto, montada
-       no end-effector do braço — ver t265_mount_joint em movemaster.urdf.xacro) -->
-  <xacro:movemaster_rv_m2 parent="top_plate" xyz="0.05 0 0.02" rpy="0 0 0"/>
-  <!-- Hokuyo UST-05LX (Smart URG) — FOV 270°, alcance 0.06-5.0 m,
-       resolução angular 0.25° (1081 amostras). Reaproveita o macro
-       custom_laser já existente no xacro do Pioneer (placeholder visual
-       em caixa, sem malha própria do sensor). -->
+  <!-- Braço montado sobre o top_plate do Pioneer, centralizado no meio dos
+       eixos da plataforma original (x≈0 no base_link, z=0.02 de folga de
+       montagem). A T265 vem junto, no end-effector — ver movemaster.urdf.xacro. -->
+  <xacro:movemaster_rv_m2 parent="top_plate" xyz="0 0 0.02" rpy="0 0 0"/>
+  <!-- Hokuyo UST-05LX — centralizado (y=0), 2.5 cm da frente da plataforma
+       em direção ao centro. FOV 270°, alcance 0.06-5.0 m, 0.25°/amostra. -->
   <xacro:custom_laser name="hokuyo" color="Black"
-                      x="0.24" y="0" z="0.05" roll="0" pitch="0" yaw="0"
+                      x="0.215" y="0" z="0.025" roll="0" pitch="0" yaw="0"
                       samples="1081" resolution="1"
                       min_angle="${-3*PI/4}" max_angle="${3*PI/4}"

File: src/b166er_robot/urdf/movemaster/movemaster.urdf.xacro (robot description, xacro)
@@ -55,8 +55,9 @@
       </inertial>
     </link>
-    <!-- Sparton AHRS-8 IMU — montada na face traseira de L1, primeiro elo
-         do braço logo após a torre giratória (confirmado por foto do robô real) -->
+    <!-- Sparton AHRS-8 — face traseira de L1 (bunda do manipulador, eixo 2),
+         confirmado por foto do robô real. Offset: 5 cm atrás do eixo J1,
+         10 cm abaixo; orientado 180° em yaw (face para trás do braço). -->
     <joint name="imu_mount_joint" type="fixed">
-      <origin xyz="-0.05 0 -0.1" rpy="0 0 ${PI}"/>
+      <origin xyz="-0.05 0 0.02" rpy="0 0 ${PI}"/>
       <parent link="L1"/>
       <child link="ahrs8_link"/>

Commit message: fix(b166er_robot): plataforma alongada 92 mm e Hokuyo na borda medida
O Marco alongou a plataforma do Pioneer PARA A FRENTE: 508,2 mm de
fábrica -> 600 mm. Chassi e entre-eixos não mudaram. Modelado como link
próprio (front_plate_ext), com colisão, para o pioneer3at-m.urdf.xacro
continuar descrevendo o robô de fábrica.

O Hokuyo está a 3 cm da nova borda, o que o põe 10 cm à frente de onde o
modelo o desenhava. Esse era o erro que fazia o laser_safety reportar a
parede 10 cm mais longe do que está — e é o sintoma que o Marco relatou
de o robô encostar demais na parede.

laser_offset_x: 0,215 -> 0,3189 (= 0,003 base_link->top_plate + 0,3159).

Co-Authored-By: Claude Opus 5 <noreply@anthropic.com>
Claude-Session: https://claude.ai/code/session_01Ra2BbYQxYWhbcCFkGE7vAN

File: src/b166er_robot/urdf/b166er.urdf.xacro (robot description, xacro)
@@ -12,8 +12,54 @@
        montagem). A T265 vem junto, no end-effector — ver movemaster.urdf.xacro. -->
   <xacro:movemaster_rv_m2 parent="top_plate" xyz="0 0 0.02" rpy="0 0 0"/>
-  <!-- Hokuyo UST-05LX — centralizado (y=0), 2.5 cm da frente da plataforma
-       em direção ao centro. FOV 270°, alcance 0.06-5.0 m, 0.25°/amostra. -->
+  <!-- ═══ Prolongamento frontal da plataforma (medido 2026-08-26) ═══
+       O Marco alongou a plataforma do Pioneer PARA A FRENTE. O chassi e
+       o entre-eixos NÃO mudaram — só o prato de cima:
+         top.stl original ....... 508,2 mm  (±254,1 no frame top_plate)
+         plataforma real hoje ... 600   mm
+         acréscimo .............. 91,8 mm, todo à frente
+       Modelado como um link próprio em vez de mexer no mesh do Pioneer:
+       o pioneer3at-m.urdf.xacro é o modelo de fábrica e deve continuar
+       descrevendo o robô de fábrica. Tem COLISÃO porque é ela que a
+       parede enxerga — sem isso o Gazebo deixaria a parede invadir 9 cm
+       de plataforma antes de tocar em qualquer coisa. -->
+  <xacro:property name="ext_len"   value="0.0918"/>
+  <xacro:property name="plate_x0"  value="0.25410"/>
+  <xacro:property name="plate_hw"  value="0.19154"/>
+  <xacro:property name="plate_t"   value="0.00658"/>
+  <!-- Face frontal da plataforma, no frame do top_plate. -->
+  <xacro:property name="plate_front" value="${plate_x0 + ext_len}"/>
+  <joint name="front_plate_ext_joint" type="fixed">
+    <origin xyz="${plate_x0 + ext_len/2} 0 0" rpy="0 0 0"/>
+    <parent link="top_plate"/>
+    <child link="front_plate_ext"/>
+  </joint>
+  <link name="front_plate_ext">
+    <visual>
+      <origin xyz="0 0 0" rpy="0 0 0"/>
+      <geometry><box size="${ext_len} ${2*plate_hw} ${plate_t}"/></geometry>
+      <material name="TopBlack"/>
+    </visual>
+    <collision>
+      <origin xyz="0 0 0" rpy="0 0 0"/>
+      <geometry><box size="${ext_len} ${2*plate_hw} ${plate_t}"/></geometry>
+    </collision>
+    <inertial>
+      <mass value="0.25"/>
+      <inertia ixx="0.003" ixy="0" ixz="0" iyy="0.0002" iyz="0" izz="0.003"/>
+    </inertial>
+  </link>
+  <gazebo reference="front_plate_ext"><material>Gazebo/Black</material></gazebo>
+  <!-- Hokuyo UST-05LX — centralizado (y=0), 3 cm atrás da borda frontal
+       do prato (medido na bancada em 2026-08-26). Com a plataforma
+       alongada isso o põe em x=0,3159 no frame do top_plate, ou seja
+       0,3189 do centro da base — 10 cm mais à frente do que o modelo
+       antigo supunha. Esse era o erro que fazia o laser_safety achar que
+       a parede estava 10 cm mais longe do que está, e é por isso que o
+       robô encostava demais. laser_safety.py:~laser_offset_x precisa
+       casar com este número.
+       FOV 270°, alcance 0.06-5.0 m, 0.25°/amostra. -->
   <xacro:custom_laser name="hokuyo" color="Black"
-                      x="0.215" y="0" z="0.025" roll="0" pitch="0" yaw="0"
+                      x="${plate_front - 0.030}" y="0" z="0.025"
+                      roll="0" pitch="0" yaw="0"
                       samples="1081" resolution="1"
                       min_angle="${-3*PI/4}" max_angle="${3*PI/4}"

Commit message: feat(b166er_robot): Hokuyo UST-05LX modelado e em laranja, visível na simulação
O Marco: "o hokuyo precisa ser renderizado/modelado, e mudado de cor
para que possamos enxergar na simulação" / "o nosso é o UST-05LX". Era
um cubo preto de 25 mm, invisível sobre o chassi.

Malha: hokuyo.dae do gazebo_plugins (BSD), a forma da família URG/UST,
cujo envelope já é 50 x 50 x 70 mm — o do UST-05LX — sem escala. Estava
deitada no arquivo; convertida para STL em pé, base em z = 0, centrada.
O lado de cima foi acertado pelo Marco com o sensor real na mão (a
heurística pela faixa branca tinha posto de ponta-cabeça). STL sem
materiais de propósito: com os materiais do .dae o Gazebo ignora o
<material> do link, e a cor é o pedido. Laranja (Gazebo/Orange e RViz),
distinto do verde da T265, do amarelo da ferramenta e do azul da placa.

A origem do laser_hokuyo_link é o plano de varredura (o sensor ray
emite dali): a malha desce 34 mm (a janela da malha) para a base
assentar na placa, e a instanciação sobe o link de 0,025 para 0,034 —
plano de varredura de 0,299 para 0,308 m do base_link. A altura real
da janela na bancada não foi medida; está assumida pela malha.
Colisão: caixa 50 x 50 x 70, inteira dentro do alcance mínimo (0,06 m),
então sem retorno espúrio do próprio corpo.

Sensor já estava com os parâmetros do UST-05LX (0,06-5,0 m, ±135°,
1081 passos, 40 Hz); só os comentários ao lado falavam de outro modelo
e foram corrigidos. Conferido no stack novo: 40 Hz, 1081 passos, 270°,
154 retornos finitos (parede e fixture a 1,96-2,58 m).

Co-Authored-By: Claude Fable 5.1 <noreply@anthropic.com>
Claude-Session: https://claude.ai/code/session_01P4v3ZvEh2bwom2DYHA9moN

File: src/b166er_robot/urdf/b166er.urdf.xacro (robot description, xacro)
@@ -59,6 +59,11 @@
        casar com este número.
        FOV 270°, alcance 0.06-5.0 m, 0.25°/amostra. -->
-  <xacro:custom_laser name="hokuyo" color="Black"
-                      x="${plate_front - 0.030}" y="0" z="0.025"
+  <!-- z = 0,034: a origem do link é o PLANO DE VARREDURA, e a malha do
+       UST-05LX tem a janela a 34 mm da base — assim a base assenta na
+       placa (era 0,025 para um cubo de 25 mm). Sobe o plano 9 mm; a
+       altura real da janela na bancada não foi medida (assumida pela
+       malha). Laranja para ser visível sobre o chassi escuro. -->
+  <xacro:custom_laser name="hokuyo" color="Orange"
+                      x="${plate_front - 0.030}" y="0" z="0.034"
                       roll="0" pitch="0" yaw="0"
                       samples="1081" resolution="1"

File: src/b166er_robot/urdf/pioneer3at/pioneer3at-m.urdf.xacro (robot description, xacro)
@@ -422,19 +422,31 @@
     </joint>
     <link name="laser_${name}_link">
+        <!-- HOKUYO UST-05LX MODELADO (2026-09-02, pedido do Marco: "o hokuyo
+             precisa ser renderizado/modelado, e mudado de cor para que
+             possamos enxergar na simulação"). Era um cubo de 25 mm preto,
+             invisível sobre o chassi. A malha é a hokuyo.dae do gazebo_plugins
+             (forma da família URG/UST, mesmo envelope de 50 x 50 x 70 mm do
+             UST-05LX), convertida para STL em pé, base em z = 0, e a janela
+             de varredura a 34 mm da base (o lado de cima foi conferido pelo Marco
+             contra o sensor real: a heurística pela faixa branca errou) — ver
+             meshes/hokuyo/README.md.
+             A ORIGEM DESTE LINK É O PLANO DE VARREDURA (é onde o sensor ray
+             emite), então a malha desce 36 mm para a base assentar na placa.
+             STL e não DAE de propósito: com materiais embutidos o Gazebo
+             ignora o <material> do link, e a cor é o pedido. -->
         <collision>
-          <origin xyz="0 0 0" rpy="0 0 0"/>
+          <origin xyz="0 0 -0.001" rpy="0 0 0"/>
           <geometry>
-            <box size="0.025 0.025 0.025"/>
+            <box size="0.050 0.050 0.070"/>
           </geometry>
         </collision>
         <visual>
-          <origin xyz="0 0 0" rpy="0 0 0"/>
+          <origin xyz="0 0 -0.034" rpy="0 0 0"/>
           <geometry>
-            <box size="0.025 0.025 0.025"/>
+            <mesh filename="package://b166er_robot/meshes/hokuyo/hokuyo_ust05lx.stl"/>
           </geometry>
-          <!-- "red" sem <color> = material indefinido no RViz → link renderizado branco.
-               Definição explícita garante cor vermelha em vez do branco padrão. -->
-          <material name="red">
-            <color rgba="0.8 0.1 0.1 1"/>
+          <!-- RViz lê este <material>; o Gazebo lê o <gazebo reference> abaixo. -->
+          <material name="hokuyo_laranja">
+            <color rgba="1.0 0.5 0.0 1"/>
           </material>
         </visual>
@@ -456,5 +468,5 @@
             <scan>
               <horizontal>
-                <samples>${samples}</samples> <!-- 720 -->
+                <samples>${samples}</samples> <!-- UST-05LX: 1081 (0,25°) -->
                 <resolution>${resolution}</resolution> <!-- 1 -->
                 <min_angle>${min_angle}</min_angle> <!-- minus 1.570796 -->
@@ -463,6 +475,6 @@
             </scan>
             <range>
-              <min>${min_range}</min> <!-- 0.10 -->
-              <max>${max_range}</max> <!-- 30.0 -->
+              <min>${min_range}</min> <!-- UST-05LX: 0.06 -->
+              <max>${max_range}</max> <!-- UST-05LX: 5.0 -->
               <resolution>${range_resolution}</resolution> <!-- 0.01 -->
             </range>
