Commit message: feat(sim): adiciona IMU Sparton AHRS-8 no URDF, montada no braço
Confirmado por foto do robô real: a AHRS-8 fica fixada na face
traseira de L1, primeiro elo do braço logo após a torre giratória —
não no chassi do Pioneer. Placeholder visual em caixa (sem malha
própria), no mesmo padrão usado para os outros sensores adicionados.

Co-Authored-By: Claude Sonnet 4.6 <noreply@anthropic.com>

File: src/b166er_robot/urdf/movemaster/movemaster.urdf.xacro (robot description, xacro)
@@ -40,4 +40,27 @@
       </visual>
     </link>
+    <!-- Sparton AHRS-8 IMU — montada na face traseira de L1, primeiro elo
+         do braço logo após a torre giratória (confirmado por foto do robô real) -->
+    <joint name="imu_mount_joint" type="fixed">
+      <origin xyz="-0.05 0 -0.1" rpy="0 0 ${PI}"/>
+      <parent link="L1"/>
+      <child link="ahrs8_link"/>
+    </joint>
+    <link name="ahrs8_link">
+      <visual>
+        <origin xyz="0 0 0" rpy="0 0 0"/>
+        <geometry>
+          <box size="0.025 0.025 0.025"/>
+        </geometry>
+        <material name="imu_color">
+          <color rgba="1.0 1.0 0.0 1.0"/>
+        </material>
+      </visual>
+      <inertial>
+        <mass value="1e-5"/>
+        <origin xyz="0 0 0" rpy="0 0 0"/>
+        <inertia ixx="1e-6" ixy="0" ixz="0" iyy="1e-6" iyz="0" izz="1e-6"/>
+      </inertial>
+    </link>
     <joint name="J2" type="revolute">
       <axis xyz="0 0 1"/>

Commit message: feat(sim): inércias provisórias no braço e launch do Gazebo (Fase 2, preview)
Adiciona <inertial> placeholder em Base/L1-L5 (únicos elos com junta
revolute, exigem massa para o Gazebo) e um novo launch
simulation/b166er_gazebo.launch, exclusivamente para preview estético
do spawn — sem controle e sem validação de física real. Os valores de
massa/inércia são estimativas e devem ser substituídos pelos dados
reais quando o usuário medir os componentes no laboratório.

gzserver não sobe neste ambiente conda: crash fatal
"pthread_mutex_lock assertion failed" ao carregar
libgazebo_ros_api_plugin.so, reproduzido isoladamente sem nenhum
robô/world customizado — bug de empacotamento do gazebo_ros nesta env
RoboStack, não relacionado ao URDF/launch. Necessário corrigir a
instalação do Gazebo (rebuild/repin de gazebo+gazebo_ros) antes de
validar a Fase 2.

Co-Authored-By: Claude Sonnet 4.6 <noreply@anthropic.com>

File: src/b166er_robot/urdf/movemaster/movemaster.urdf.xacro (robot description, xacro)
@@ -21,4 +21,11 @@
         </material>
       </visual>
+      <!-- Massa/inércia provisórias, só para o Gazebo não instabilizar.
+           Substituir pelos valores reais quando medidos no laboratório. -->
+      <inertial>
+        <mass value="2.0"/>
+        <origin xyz="0 0 0" rpy="0 0 0"/>
+        <inertia ixx="0.02" ixy="0" ixz="0" iyy="0.02" iyz="0" izz="0.02"/>
+      </inertial>
     </link>
     <joint name="J1" type="revolute">
@@ -39,4 +46,9 @@
         </material>
       </visual>
+      <inertial>
+        <mass value="1.5"/>
+        <origin xyz="0 0 -0.16" rpy="0 0 0"/>
+        <inertia ixx="0.015" ixy="0" ixz="0" iyy="0.015" iyz="0" izz="0.015"/>
+      </inertial>
     </link>
     <!-- Sparton AHRS-8 IMU — montada na face traseira de L1, primeiro elo
@@ -80,4 +92,9 @@
         </material>
       </visual>
+      <inertial>
+        <mass value="1.2"/>
+        <origin xyz="0 0 0" rpy="0 0 0"/>
+        <inertia ixx="0.012" ixy="0" ixz="0" iyy="0.012" iyz="0" izz="0.012"/>
+      </inertial>
     </link>
     <joint name="J3" type="revolute">
@@ -98,4 +115,9 @@
         </material>
       </visual>
+      <inertial>
+        <mass value="1.0"/>
+        <origin xyz="0 0 0" rpy="0 0 0"/>
+        <inertia ixx="0.01" ixy="0" ixz="0" iyy="0.01" iyz="0" izz="0.01"/>
+      </inertial>
     </link>
     <joint name="J4" type="revolute">
@@ -116,4 +138,9 @@
         </material>
       </visual>
+      <inertial>
+        <mass value="0.6"/>
+        <origin xyz="0 0 0" rpy="0 0 0"/>
+        <inertia ixx="0.006" ixy="0" ixz="0" iyy="0.006" iyz="0" izz="0.006"/>
+      </inertial>
     </link>
     <joint name="J5" type="revolute">
@@ -134,4 +161,9 @@
         </material>
       </visual>
+      <inertial>
+        <mass value="0.4"/>
+        <origin xyz="0 0 -0.08" rpy="0 0 0"/>
+        <inertia ixx="0.004" ixy="0" ixz="0" iyy="0.004" iyz="0" izz="0.004"/>
+      </inertial>
     </link>
     <joint name="JCam" type="fixed">

Commit message: fix(sim): limites de junta e massa do RV-M2 conforme manual oficial
Dados extraídos do manual de instruções Mitsubishi (BFP-A5296) e da
dissertação do Cerbaro sobre o Movemaster modernizado, que o usuário
trouxe do laboratório:

- Limites de junta reais (manual, tabela 1.3.1) substituem o
  placeholder de ±360° (quase sem limite): cintura ±150° (300° total),
  ombro ±65° (130°), cotovelo ±60° (120°), punho pitch ±110°, punho
  roll ±180°. Os ranges de J1-J3 só têm o total documentado, não o
  zero exato — assumido simétrico por ora, a confirmar com o robô real.
- Massa total escalada de ~6.7kg (placeholder) para ~28kgf (peso real
  do braço, mesma tabela), mantendo a distribuição proporcional entre
  os elos — ainda uma estimativa, não a massa real por elo.
- Comprimentos dos elos (120/250/200mm) já confirmados corretos contra
  o manual e a tabela de parâmetros DH da dissertação.

Co-Authored-By: Claude Sonnet 4.6 <noreply@anthropic.com>

File: src/b166er_robot/urdf/movemaster/movemaster.urdf.xacro (robot description, xacro)
@@ -21,10 +21,12 @@
         </material>
       </visual>
-      <!-- Massa/inércia provisórias, só para o Gazebo não instabilizar.
-           Substituir pelos valores reais quando medidos no laboratório. -->
-      <inertial>
-        <mass value="2.0"/>
-        <origin xyz="0 0 0" rpy="0 0 0"/>
-        <inertia ixx="0.02" ixy="0" ixz="0" iyy="0.02" iyz="0" izz="0.02"/>
+      <!-- Massa/inércia: distribuição proporcional ao placeholder original,
+           escalada para somar ~28kgf (peso total real do RV-M2, manual de
+           instruções Mitsubishi BFP-A5296, tabela 1.3.1). Distribuição por
+           elo ainda é estimada — substituir quando medido no laboratório. -->
+      <inertial>
+        <mass value="8.4"/>
+        <origin xyz="0 0 0" rpy="0 0 0"/>
+        <inertia ixx="0.084" ixy="0" ixz="0" iyy="0.084" iyz="0" izz="0.084"/>
       </inertial>
     </link>
@@ -34,5 +36,6 @@
       <parent link="Base"/>
       <child link="L1"/>
-      <limit upper="6.28" lower="-6.28" effort="10" velocity="10" />
+      <!-- Cintura (waist): 300° de curso total no manual, assumido ±150° -->
+      <limit upper="2.61799" lower="-2.61799" effort="10" velocity="10" />
     </joint>
     <link name="L1">
@@ -47,7 +50,7 @@
       </visual>
       <inertial>
-        <mass value="1.5"/>
+        <mass value="6.3"/>
         <origin xyz="0 0 -0.16" rpy="0 0 0"/>
-        <inertia ixx="0.015" ixy="0" ixz="0" iyy="0.015" iyz="0" izz="0.015"/>
+        <inertia ixx="0.063" ixy="0" ixz="0" iyy="0.063" iyz="0" izz="0.063"/>
       </inertial>
     </link>
@@ -80,5 +83,6 @@
       <parent link="L1"/>
       <child link="L2"/>
-      <limit upper="6.28" lower="-6.28" effort="10" velocity="10" />
+      <!-- Ombro (shoulder): 130° de curso total no manual, assumido ±65° -->
+      <limit upper="1.13446" lower="-1.13446" effort="10" velocity="10" />
     </joint>
     <link name="L2">
@@ -93,7 +97,7 @@
       </visual>
       <inertial>
-        <mass value="1.2"/>
-        <origin xyz="0 0 0" rpy="0 0 0"/>
-        <inertia ixx="0.012" ixy="0" ixz="0" iyy="0.012" iyz="0" izz="0.012"/>
+        <mass value="5.0"/>
+        <origin xyz="0 0 0" rpy="0 0 0"/>
+        <inertia ixx="0.050" ixy="0" ixz="0" iyy="0.050" iyz="0" izz="0.050"/>
       </inertial>
     </link>
@@ -103,5 +107,6 @@
       <parent link="L2"/>
       <child link="L3"/>
-      <limit upper="6.28" lower="-6.28" effort="10" velocity="10" />
+      <!-- Cotovelo (elbow): 120° de curso total no manual, assumido ±60° -->
+      <limit upper="1.04720" lower="-1.04720" effort="10" velocity="10" />
     </joint>
     <link name="L3">
@@ -116,7 +121,7 @@
       </visual>
       <inertial>
-        <mass value="1.0"/>
-        <origin xyz="0 0 0" rpy="0 0 0"/>
-        <inertia ixx="0.01" ixy="0" ixz="0" iyy="0.01" iyz="0" izz="0.01"/>
+        <mass value="4.2"/>
+        <origin xyz="0 0 0" rpy="0 0 0"/>
+        <inertia ixx="0.042" ixy="0" ixz="0" iyy="0.042" iyz="0" izz="0.042"/>
       </inertial>
     </link>
@@ -126,5 +131,6 @@
       <parent link="L3"/>
       <child link="L4"/>
-      <limit upper="6.28" lower="-6.28" effort="10" velocity="10" />
+      <!-- Punho pitch (wrist pitch): ±110° no manual -->
+      <limit upper="1.91986" lower="-1.91986" effort="10" velocity="10" />
     </joint>
     <link name="L4">
@@ -139,7 +145,7 @@
       </visual>
       <inertial>
-        <mass value="0.6"/>
-        <origin xyz="0 0 0" rpy="0 0 0"/>
-        <inertia ixx="0.006" ixy="0" ixz="0" iyy="0.006" iyz="0" izz="0.006"/>
+        <mass value="2.5"/>
+        <origin xyz="0 0 0" rpy="0 0 0"/>
+        <inertia ixx="0.025" ixy="0" ixz="0" iyy="0.025" iyz="0" izz="0.025"/>
       </inertial>
     </link>
@@ -149,5 +155,6 @@
       <parent link="L4"/>
       <child link="L5"/>
-      <limit upper="6.28" lower="-6.28" effort="10" velocity="10" />
+      <!-- Punho roll (wrist roll): ±180° no manual -->
+      <limit upper="3.14159" lower="-3.14159" effort="10" velocity="10" />
     </joint>
     <link name="L5">
@@ -162,7 +169,7 @@
       </visual>
       <inertial>
-        <mass value="0.4"/>
+        <mass value="1.7"/>
         <origin xyz="0 0 -0.08" rpy="0 0 0"/>
-        <inertia ixx="0.004" ixy="0" ixz="0" iyy="0.004" iyz="0" izz="0.004"/>
+        <inertia ixx="0.017" ixy="0" ixz="0" iyy="0.017" iyz="0" izz="0.017"/>
       </inertial>
     </link>

Commit message: feat(control): Fase 2 — arm_vel_integrator + validação Gazebo
Hardware path:
- arm_vel_integrator.py: integra /b166er/arm_vel_cmd (rad/s) → /setpoints
  (graus) para o Arduino via rosserial; warm-start com q estimado pelo
  state_estimator; timeout de segurança de 0,5 s sem comando → velocidade
  zerada; saturação em JOINT_LOWER/JOINT_UPPER

Gazebo path (mode:=gazebo):
- movemaster.urdf.xacro: adiciona transmissões VelocityJointInterface
  (J1..J5) + plugin gazebo_ros_control
- config/arm_controllers.yaml: joint_state_controller + 5
  velocity_controllers para as juntas do braço
- gazebo_sensor_sim.py: sintetiza /t265/odom/sample (FK das juntas
  simuladas) e republica /pioneer/pose a partir do diff-drive do Pioneer
- gazebo_arm_bridge.py: encaminha /b166er/arm_vel_cmd (JointState) →
  /Jx_velocity_controller/command (Float64) individuais
- b166er_wb.launch: modo gazebo completo (spawn + controllers + bridges +
  stack WBC); arm_vel_integrator ativado apenas em mode:=hardware

Co-Authored-By: Claude Sonnet 4.6 <noreply@anthropic.com>

File: src/b166er_robot/urdf/movemaster/movemaster.urdf.xacro (robot description, xacro)
@@ -256,4 +256,30 @@
       </visual>
     </link>
+    <!-- ── Transmissões para ros_control (Gazebo) ───────────────────── -->
+    <!-- VelocityJointInterface: controladores de velocidade para cada junta -->
+    <xacro:macro name="arm_transmission" params="joint_name">
+      <transmission name="${joint_name}_trans">
+        <type>transmission_interface/SimpleTransmission</type>
+        <joint name="${joint_name}">
+          <hardwareInterface>hardware_interface/VelocityJointInterface</hardwareInterface>
+        </joint>
+        <actuator name="${joint_name}_motor">
+          <hardwareInterface>hardware_interface/VelocityJointInterface</hardwareInterface>
+          <mechanicalReduction>1</mechanicalReduction>
+        </actuator>
+      </transmission>
+    </xacro:macro>
+    <xacro:arm_transmission joint_name="J1"/>
+    <xacro:arm_transmission joint_name="J2"/>
+    <xacro:arm_transmission joint_name="J3"/>
+    <xacro:arm_transmission joint_name="J4"/>
+    <xacro:arm_transmission joint_name="J5"/>
+    <!-- Plugin gazebo_ros_control para ativar as transmissões acima -->
+    <gazebo>
+      <plugin name="gazebo_ros_control" filename="libgazebo_ros_control.so">
+        <robotNamespace>/</robotNamespace>
+        <robotSimType>gazebo_ros_control/DefaultRobotHWSim</robotSimType>
+      </plugin>
+    </gazebo>
   </xacro:macro>
 </robot>

Commit message: fix(urdf): adiciona collision boxes/cylinders ao braço RV-M2
Sem <collision> o Gazebo não tem geometria para simular física dos elos
— os joints colapsam sob gravidade e as links atravessam objetos.
Geometrias aproximadas (box/cylinder) adicionadas em Base, L1-L5.
As geometrias visuais (STL) permanecem inalteradas.

Co-Authored-By: Claude Sonnet 4.6 <noreply@anthropic.com>

File: src/b166er_robot/urdf/movemaster/movemaster.urdf.xacro (robot description, xacro)
@@ -21,4 +21,8 @@
         </material>
       </visual>
+      <collision>
+        <origin xyz="0 0 0.20" rpy="0 0 0"/>
+        <geometry><box size="0.12 0.12 0.40"/></geometry>
+      </collision>
       <!-- Massa/inércia: distribuição proporcional ao placeholder original,
            escalada para somar ~28kgf (peso total real do RV-M2, manual de
@@ -49,4 +53,8 @@
         </material>
       </visual>
+      <collision>
+        <origin xyz="0.06 0 -0.16" rpy="0 0 0"/>
+        <geometry><box size="0.20 0.10 0.30"/></geometry>
+      </collision>
       <inertial>
         <mass value="6.3"/>
@@ -97,4 +105,8 @@
         </material>
       </visual>
+      <collision>
+        <origin xyz="0.125 0 0" rpy="0 1.5708 0"/>
+        <geometry><cylinder radius="0.04" length="0.25"/></geometry>
+      </collision>
       <inertial>
         <mass value="5.0"/>
@@ -121,4 +133,8 @@
         </material>
       </visual>
+      <collision>
+        <origin xyz="0.100 0 0" rpy="0 1.5708 0"/>
+        <geometry><cylinder radius="0.035" length="0.20"/></geometry>
+      </collision>
       <inertial>
         <mass value="4.2"/>
@@ -145,4 +161,8 @@
         </material>
       </visual>
+      <collision>
+        <origin xyz="0.04 0 0" rpy="0 1.5708 0"/>
+        <geometry><cylinder radius="0.03" length="0.08"/></geometry>
+      </collision>
       <inertial>
         <mass value="2.5"/>
@@ -169,4 +189,8 @@
         </material>
       </visual>
+      <collision>
+        <origin xyz="0 0 -0.06" rpy="0 0 0"/>
+        <geometry><cylinder radius="0.03" length="0.12"/></geometry>
+      </collision>
       <inertial>
         <mass value="1.7"/>

Commit message: fix(sim): aumenta effort limits e ganhos PID do braço RV-M2
effort=10 Nm era insuficiente para sustentar o braço de 28 kg contra
a gravidade (J2 precisa de ~39 Nm só para segurar o ombro).
Novos valores: J1=30, J2=80, J3=50, J4=20, J5=10 Nm.
Velocidades corrigidas para os valores reais do manual.

Ganhos PID aumentados proporcionalmente para que o controlador
de posição consiga comandar torque dentro dos novos limites.

Co-Authored-By: Claude Sonnet 4.6 <noreply@anthropic.com>

File: src/b166er_robot/urdf/movemaster/movemaster.urdf.xacro (robot description, xacro)
@@ -41,5 +41,5 @@
       <child link="L1"/>
       <!-- Cintura (waist): 300° de curso total no manual, assumido ±150° -->
-      <limit upper="2.61799" lower="-2.61799" effort="10" velocity="10" />
+      <limit upper="2.61799" lower="-2.61799" effort="30" velocity="3.14" />
     </joint>
     <link name="L1">
@@ -93,5 +93,5 @@
       <child link="L2"/>
       <!-- Ombro (shoulder): 130° de curso total no manual, assumido ±65° -->
-      <limit upper="1.13446" lower="-1.13446" effort="10" velocity="10" />
+      <limit upper="1.13446" lower="-1.13446" effort="80" velocity="2.09" />
     </joint>
     <link name="L2">
@@ -121,5 +121,5 @@
       <child link="L3"/>
       <!-- Cotovelo (elbow): 120° de curso total no manual, assumido ±60° -->
-      <limit upper="1.04720" lower="-1.04720" effort="10" velocity="10" />
+      <limit upper="1.04720" lower="-1.04720" effort="50" velocity="2.09" />
     </joint>
     <link name="L3">
@@ -149,5 +149,5 @@
       <child link="L4"/>
       <!-- Punho pitch (wrist pitch): ±110° no manual -->
-      <limit upper="1.91986" lower="-1.91986" effort="10" velocity="10" />
+      <limit upper="1.91986" lower="-1.91986" effort="20" velocity="3.14" />
     </joint>
     <link name="L4">
@@ -177,5 +177,5 @@
       <child link="L5"/>
       <!-- Punho roll (wrist roll): ±180° no manual -->
-      <limit upper="3.14159" lower="-3.14159" effort="10" velocity="10" />
+      <limit upper="3.14159" lower="-3.14159" effort="10" velocity="6.28" />
     </joint>
     <link name="L5">

Commit message: fix(sim): damping físico nas juntas + reverte tracking do bridge
- Adiciona <dynamics damping friction> em J1-J5: amortecimento viscoso
  simulado pelo Gazebo, independente do PID (J2=15, J3=10, J1/J4=5, J5=2 Nm·s/rad)
- Reverte tracking de posição real no bridge: causava feedback positivo
  que fazia J2 desandar (bridge aceitava posição em queda como setpoint)

Co-Authored-By: Claude Sonnet 4.6 <noreply@anthropic.com>

File: src/b166er_robot/urdf/movemaster/movemaster.urdf.xacro (robot description, xacro)
@@ -42,4 +42,5 @@
       <!-- Cintura (waist): 300° de curso total no manual, assumido ±150° -->
       <limit upper="2.61799" lower="-2.61799" effort="30" velocity="3.14" />
+      <dynamics damping="5.0" friction="1.0"/>
     </joint>
     <link name="L1">
@@ -94,4 +95,5 @@
       <!-- Ombro (shoulder): 130° de curso total no manual, assumido ±65° -->
       <limit upper="1.13446" lower="-1.13446" effort="80" velocity="2.09" />
+      <dynamics damping="15.0" friction="2.0"/>
     </joint>
     <link name="L2">
@@ -122,4 +124,5 @@
       <!-- Cotovelo (elbow): 120° de curso total no manual, assumido ±60° -->
       <limit upper="1.04720" lower="-1.04720" effort="50" velocity="2.09" />
+      <dynamics damping="10.0" friction="1.5"/>
     </joint>
     <link name="L3">
@@ -150,4 +153,5 @@
       <!-- Punho pitch (wrist pitch): ±110° no manual -->
       <limit upper="1.91986" lower="-1.91986" effort="20" velocity="3.14" />
+      <dynamics damping="5.0" friction="1.0"/>
     </joint>
     <link name="L4">
@@ -178,4 +182,5 @@
       <!-- Punho roll (wrist roll): ±180° no manual -->
       <limit upper="3.14159" lower="-3.14159" effort="10" velocity="6.28" />
+      <dynamics damping="2.0" friction="0.5"/>
     </joint>
     <link name="L5">

Commit message: fix(urdf): remove collision boxes do braço — causavam forças explosivas
As collision boxes adicionadas se sobrepunham (Base/L1 intersectavam),
gerando forças de contato ODE gigantes no spawn. Para ros_control com
PositionJointInterface, collision geometry não é necessária — apenas
inércias e joint damping importam para a simulação de controle.

Co-Authored-By: Claude Sonnet 4.6 <noreply@anthropic.com>

File: src/b166er_robot/urdf/movemaster/movemaster.urdf.xacro (robot description, xacro)
@@ -21,8 +21,4 @@
         </material>
       </visual>
-      <collision>
-        <origin xyz="0 0 0.20" rpy="0 0 0"/>
-        <geometry><box size="0.12 0.12 0.40"/></geometry>
-      </collision>
       <!-- Massa/inércia: distribuição proporcional ao placeholder original,
            escalada para somar ~28kgf (peso total real do RV-M2, manual de
@@ -54,8 +50,4 @@
         </material>
       </visual>
-      <collision>
-        <origin xyz="0.06 0 -0.16" rpy="0 0 0"/>
-        <geometry><box size="0.20 0.10 0.30"/></geometry>
-      </collision>
       <inertial>
         <mass value="6.3"/>
@@ -107,8 +99,4 @@
         </material>
       </visual>
-      <collision>
-        <origin xyz="0.125 0 0" rpy="0 1.5708 0"/>
-        <geometry><cylinder radius="0.04" length="0.25"/></geometry>
-      </collision>
       <inertial>
         <mass value="5.0"/>
@@ -136,8 +124,4 @@
         </material>
       </visual>
-      <collision>
-        <origin xyz="0.100 0 0" rpy="0 1.5708 0"/>
-        <geometry><cylinder radius="0.035" length="0.20"/></geometry>
-      </collision>
       <inertial>
         <mass value="4.2"/>
@@ -165,8 +149,4 @@
         </material>
       </visual>
-      <collision>
-        <origin xyz="0.04 0 0" rpy="0 1.5708 0"/>
-        <geometry><cylinder radius="0.03" length="0.08"/></geometry>
-      </collision>
       <inertial>
         <mass value="2.5"/>
@@ -194,8 +174,4 @@
         </material>
       </visual>
-      <collision>
-        <origin xyz="0 0 -0.06" rpy="0 0 0"/>
-        <geometry><cylinder radius="0.03" length="0.12"/></geometry>
-      </collision>
       <inertial>
         <mass value="1.7"/>

Commit message: fix(sim): damping ODE-safe (0.1-1.0) + PID conservador
damping > 5 Nm·s/rad é numericamente instável no ODE com dt=1ms
(equivale a rigidez de 5000+ Nm/rad em discreto). Valores típicos
para Gazebo: 0.1-1.0. friction=0 elimina stick-slip.
PID D reduzido para não somar com o damping físico.

Co-Authored-By: Claude Sonnet 4.6 <noreply@anthropic.com>

File: src/b166er_robot/urdf/movemaster/movemaster.urdf.xacro (robot description, xacro)
@@ -38,5 +38,5 @@
       <!-- Cintura (waist): 300° de curso total no manual, assumido ±150° -->
       <limit upper="2.61799" lower="-2.61799" effort="30" velocity="3.14" />
-      <dynamics damping="5.0" friction="1.0"/>
+      <dynamics damping="0.5" friction="0.0"/>
     </joint>
     <link name="L1">
@@ -87,5 +87,5 @@
       <!-- Ombro (shoulder): 130° de curso total no manual, assumido ±65° -->
       <limit upper="1.13446" lower="-1.13446" effort="80" velocity="2.09" />
-      <dynamics damping="15.0" friction="2.0"/>
+      <dynamics damping="1.0" friction="0.0"/>
     </joint>
     <link name="L2">
@@ -112,5 +112,5 @@
       <!-- Cotovelo (elbow): 120° de curso total no manual, assumido ±60° -->
       <limit upper="1.04720" lower="-1.04720" effort="50" velocity="2.09" />
-      <dynamics damping="10.0" friction="1.5"/>
+      <dynamics damping="0.5" friction="0.0"/>
     </joint>
     <link name="L3">
@@ -137,5 +137,5 @@
       <!-- Punho pitch (wrist pitch): ±110° no manual -->
       <limit upper="1.91986" lower="-1.91986" effort="20" velocity="3.14" />
-      <dynamics damping="5.0" friction="1.0"/>
+      <dynamics damping="0.3" friction="0.0"/>
     </joint>
     <link name="L4">
@@ -162,5 +162,5 @@
       <!-- Punho roll (wrist roll): ±180° no manual -->
       <limit upper="3.14159" lower="-3.14159" effort="10" velocity="6.28" />
-      <dynamics damping="2.0" friction="0.5"/>
+      <dynamics damping="0.1" friction="0.0"/>
     </joint>
     <link name="L5">
