Commit message: feat(b166er_robot): adiciona ferramenta (vara+gancho) no end-effector
Decisão do Marco (2026-08-12): vara rígida (sem atuação própria) com
gancho na ponta, ~35cm de comprimento, montada no mesmo ponto do
gripper visual (GripCube). Existe pra dar folga real entre o
chassi/braço e a parede — o RV-M2 sozinho (~0,5-0,7m de alcance) já
forçou a base a colidir com a parede numa simulação de teste, tombando
o robô, ao tentar alcançar o olhal da chave seccionadora sem essa
extensão. Mesma lógica de uma vara de manobra real (hot stick).

Novos links: tool_rod (haste) + tool_tip (gancho na ponta), ambos
fixed a partir de GripCube (JTool/JToolTip), com <gazebo reference>
para não perder a cor na fusão de corpo rígido do Gazebo (mesmo
comportamento já documentado no fixture da chave).

kinematics.py: adiciona T_T265_TOOLTIP (offset fixo e conhecido de
t265_link até a ponta da ferramenta, calculado pela mesma cadeia
JCam+JGripCube+JTool+JToolTip do xacro) e duas funções de conversão:
- tooltip_target_to_t265_target: quando a ORIENTAÇÃO desejada é da
  ponta da ferramenta.
- tooltip_position_to_t265_position: quando só a POSIÇÃO da ponta da
  ferramenta importa e a orientação do T265 fica fixa (caso usado por
  task_sequencer.py — a rotação não-trivial do mount da ferramenta faz
  essas duas contas darem resultados diferentes, documentado em
  kinematics.py).

task_sequencer.py: os alvos de fase (engage/release/pos1/pos2)
continuam pensados para a ponta da ferramenta alcançar o olhal, mas
agora convertidos para o alvo equivalente do T265 antes de publicar
em /b166er/ee_target e antes de checar convergência (ee_pose é o
T265, não a ferramenta, que não é observada diretamente — arquitetura
sem encoders).

Co-Authored-By: Claude Sonnet 5 <noreply@anthropic.com>

File: src/b166er_robot/urdf/movemaster/movemaster.urdf.xacro (robot description, xacro)
@@ -261,4 +261,78 @@
       </visual>
     </link>
+    <!-- ═══ Ferramenta de operação (vara rígida + gancho na ponta) ═══
+         Decisão do Marco (2026-08-12): vara rígida (sem junta própria,
+         sem atuação — só extensão fixa do EE), ~35cm de comprimento,
+         com gancho na ponta pra engatar no olhal da chave seccionadora
+         (ver urdf/fixtures/chave_seccionadora_lf.urdf.xacro). Existe
+         pra dar folga real entre o chassi/braço e a parede — o RV-M2
+         sozinho (~0,5-0,7m de alcance) força a base a chegar quase
+         colada na parede pra alcançar o olhal, o que já derrubou o
+         robô numa simulação de teste (base colidindo com a parede).
+         Mesma lógica de uma vara de manobra real (hot stick): manter
+         distância do ponto energizado.
+         Montada no mesmo ponto que o gripper visual (GripCube, ponta
+         em z=-0.08 no frame do GripCube, mesmo offset dos meshes
+         Grip1/Grip2) — SEM junta própria (fixed), então herda a fusão
+         de corpo rígido do Gazebo junto com L5/CameraSupport/GripCube
+         (mesmo comportamento já documentado nas fixtures: um
+         <gazebo reference> por link, não <material><color> puro).
+         IMPORTANTE: o T265 (t265_link) continua sendo o único sensor
+         de pose do EE (arquitetura sem encoders) — a ponta da
+         ferramenta (tool_tip) NÃO é observada diretamente, é um offset
+         FIXO e conhecido a partir de t265_link (mesmo CameraSupport
+         rígido). Ver kinematics.py (T_T265_TOOLTIP) para essa
+         transformação — quem consome alvos Cartesianos pensando na
+         ponta da ferramenta (ex.: task_sequencer.py) precisa aplicar
+         esse offset ao comandar o T265, não pode simplesmente mirar a
+         ponta da ferramenta como se fosse o EE controlado. ═══ -->
+    <xacro:property name="tool_length" value="0.35"/>
+    <joint name="JTool" type="fixed">
+      <origin xyz="0 0 -0.08" rpy="0 0 0"/>
+      <parent link="GripCube"/>
+      <child link="tool_rod"/>
+    </joint>
+    <link name="tool_rod">
+      <visual>
+        <origin xyz="0 0 ${-tool_length/2}" rpy="0 0 0"/>
+        <geometry><cylinder radius="0.008" length="${tool_length}"/></geometry>
+        <material name="ToolColor"><color rgba="0.95 0.75 0.05 1"/></material>
+      </visual>
+      <collision>
+        <origin xyz="0 0 ${-tool_length/2}" rpy="0 0 0"/>
+        <geometry><cylinder radius="0.008" length="${tool_length}"/></geometry>
+      </collision>
+    </link>
+    <joint name="JToolTip" type="fixed">
+      <origin xyz="0 0 ${-tool_length}" rpy="0 0 0"/>
+      <parent link="tool_rod"/>
+      <child link="tool_tip"/>
+    </joint>
+    <!-- tool_tip: frame na ponta do gancho — este é o frame que precisa
+         coincidir com chave_olhal_link quando a tarefa "engage"
+         converge. URDF não tem primitiva de toroide; o gancho é
+         aproximado por um disco fino, mesma convenção já usada em
+         chave_olhal_link (chave_seccionadora_lf.urdf.xacro). -->
+    <link name="tool_tip">
+      <visual>
+        <geometry><cylinder radius="0.015" length="0.006"/></geometry>
+        <material name="ToolColor"/>
+      </visual>
+      <collision>
+        <geometry><sphere radius="0.018"/></geometry>
+      </collision>
+    </link>
+    <!-- <material><color> puro do URDF some na fusão de corpo rígido do
+         Gazebo (mesmo comportamento documentado em
+         chave_seccionadora_lf.urdf.xacro) — só os dois links novos da
+         ferramenta ganham <gazebo reference> aqui; o resto da árvore
+         fixa do EE (CameraSupport/GripCube/Grip1/Grip2) já tinha esse
+         problema antes desta mudança e fica fora de escopo. -->
+    <gazebo reference="tool_rod">
+      <material>Gazebo/Yellow</material>
+    </gazebo>
+    <gazebo reference="tool_tip">
+      <material>Gazebo/Yellow</material>
+    </gazebo>
     <!-- ── Transmissões para ros_control (Gazebo) ───────────────────── -->
     <!-- VelocityJointInterface: controladores de velocidade para cada junta -->

Commit message: feat(b166er): pipeline de localização por AprilTag (substitui trapaça de ground-truth)
Pedido explícito do Marco (2026-08-12): "a tag deve ser utilizada
para aproximação do robot até a chave" / "porque vc não faz o
cálculo com a ajuda da tag?" — o task_sequencer usava
/gazebo/get_link_state direto, uma trapaça de ground-truth que
nenhum robô real teria, e que escondia o problema de fundo: o
whole-body controller perseguia um ponto cego, sem nenhuma noção do
ambiente, e colidia com a parede.

- movemaster.urdf.xacro: adiciona task_camera_link (câmera pinhole
  simples no Gazebo, montada no mesmo ponto/direção da ferramenta via
  GripCube) — proxy de simulação para o stream de imagem que a câmera
  fisheye do T265 real também forneceria (pipeline já validado com
  hardware real, ver memória project_fase4_apriltag_validacao). NÃO
  substitui t265_link, que continua sendo o único sensor de POSE do
  EE.

- apriltag_localizer.py (novo nó): detecta a tag 36h11 id0 via
  cv2.aruco (OpenCV ≥4.7 tem DICT_APRILTAG_36H11 nativo — não precisei
  instalar apriltag_ros nem o pacote apriltag, nenhum dos dois
  disponível neste ambiente), estima a pose via solvePnP, e compõe
  com a pose do T265 (kinematics.T_T265_TASKCAMERA, mesmo padrão de
  T_T265_TOOLTIP) para publicar wall_link no mundo em
  /b166er/wall_pose.

- kinematics.py: adiciona T_T265_TASKCAMERA (offset fixo T265→câmera
  de tarefa).

- task_sequencer.py: troca a fonte de wall_link de
  /gazebo/get_link_state para /b166er/wall_pose por padrão.
  ~use_ground_truth:=true mantém o caminho antigo, só para
  debug/calibração (comparar a estimativa por visão com a verdade do
  simulador).

STATUS HONESTO: código completo e compila, mas AINDA NÃO VALIDADO com
detecção ao vivo — não consegui, nesta sessão, posicionar a tag no
campo de visão da câmera de forma controlada pra conferir os números
(braço com muitos graus de liberdade, geometria de montagem da câmera
não trivial, e o controlador whole-body brigando com tentativas de
posicionamento manual via /gazebo/set_model_configuration). A
convenção de eixos do PnP em apriltag_localizer.py é a melhor
estimativa, não uma correspondência confirmada — documentado
explicitamente no próprio nó. Próximo passo: validar comparando
/b166er/wall_pose com /gazebo/get_link_state numa pose com a tag
visível.

Co-Authored-By: Claude Sonnet 5 <noreply@anthropic.com>

File: src/b166er_robot/urdf/movemaster/movemaster.urdf.xacro (robot description, xacro)
@@ -213,4 +213,56 @@
       </visual>
     </link>
+    <!-- ═══ Câmera de tarefa (detecção de AprilTag) ═══
+         Adicionada em 2026-08-12 pra fechar o loop de percepção pedido
+         pelo Marco: "a tag deve ser utilizada para aproximação do
+         robot até a chave" — sem isso, task_sequencer.py só sabia onde
+         a chave estava porque perguntava direto pro Gazebo
+         (/gazebo/get_link_state, trapaça de ground-truth que nenhum
+         robô real teria).
+         NÃO é o T265 de novo — o t265_link continua sendo o único
+         sensor de POSE do EE (VIO, arquitetura sem encoders,
+         inalterado). Esta é uma câmera pinhole simples, proxy de
+         simulação para o STREAM DE IMAGEM que a câmera fisheye do
+         T265 real também forneceria (mesmo pipeline já validado com
+         hardware real — ver memória project_fase4_apriltag_validacao:
+         T265 real + AprilTag 36h11, regra tag≥d/11, tag física de
+         132mm — mesmo tamanho usado aqui). Modelar o FOV fisheye real
+         do T265 é desnecessário pra essa demonstração; pinhole padrão
+         do Gazebo já resolve.
+         Montada no mesmo ponto/direção do JTool (offset z=-0.08 a
+         partir do GripCube, mesmo "para frente" que a ferramenta
+         aponta) — olhando para onde o robô vai manipular, não para
+         onde o T265 fisicamente aponta (rotação tortuosa,
+         rpy="0 2.1 1.57", inconveniente para uma câmera de tarefa). ═══ -->
+    <joint name="JTaskCamera" type="fixed">
+      <origin xyz="0 0 -0.08" rpy="0 0 0"/>
+      <parent link="GripCube"/>
+      <child link="task_camera_link"/>
+    </joint>
+    <link name="task_camera_link">
+      <visual>
+        <geometry><box size="0.02 0.02 0.02"/></geometry>
+        <material name="ToolColor"/>
+      </visual>
+    </link>
+    <gazebo reference="task_camera_link">
+      <material>Gazebo/Yellow</material>
+      <sensor type="camera" name="task_camera">
+        <update_rate>15.0</update_rate>
+        <camera>
+          <!-- FOV largo (~86°) — compensar não ter as duas câmeras
+               fisheye do T265 real, que juntas cobrem bem mais campo. -->
+          <horizontal_fov>1.5</horizontal_fov>
+          <image><width>640</width><height>480</height><format>R8G8B8</format></image>
+          <clip><near>0.05</near><far>15.0</far></clip>
+        </camera>
+        <plugin name="task_camera_controller" filename="libgazebo_ros_camera.so">
+          <cameraName>task_camera</cameraName>
+          <imageTopicName>image_raw</imageTopicName>
+          <cameraInfoTopicName>camera_info</cameraInfoTopicName>
+          <frameName>task_camera_link</frameName>
+        </plugin>
+      </sensor>
+    </gazebo>
     <joint name="JGripCube" type="fixed">
       <origin xyz="0 0 -0.005" rpy="0 0 0"/>

Commit message: tune(b166er_robot): reduz ferramenta do EE de 35cm para 20cm
Pedido do Marco (2026-08-13). Atualizado nos dois lugares que definem
o comprimento — tool_length no xacro e o termo JToolTip em
_T_L5_TOOLTIP (kinematics.py) — que precisam ficar em sincronia
manual. Offset T265→ponta recalculado e conferido numericamente:
(0.353, 0, 0.120) → (0.224, 0, 0.044).

Co-Authored-By: Claude Fable 5 <noreply@anthropic.com>

File: src/b166er_robot/urdf/movemaster/movemaster.urdf.xacro (robot description, xacro)
@@ -315,5 +315,6 @@
     <!-- ═══ Ferramenta de operação (vara rígida + gancho na ponta) ═══
          Decisão do Marco (2026-08-12): vara rígida (sem junta própria,
-         sem atuação — só extensão fixa do EE), ~35cm de comprimento,
+         sem atuação — só extensão fixa do EE), 20cm de comprimento
+         (reduzida de 35cm por pedido do Marco em 2026-08-13),
          com gancho na ponta pra engatar no olhal da chave seccionadora
          (ver urdf/fixtures/chave_seccionadora_lf.urdf.xacro). Existe
@@ -339,5 +340,5 @@
          esse offset ao comandar o T265, não pode simplesmente mirar a
          ponta da ferramenta como se fosse o EE controlado. ═══ -->
-    <xacro:property name="tool_length" value="0.35"/>
+    <xacro:property name="tool_length" value="0.20"/>
     <joint name="JTool" type="fixed">
       <origin xyz="0 0 -0.08" rpy="0 0 0"/>

Commit message: fix(b166er_robot): remove o dedo que a garra real não tem
As fotos da bancada (IMG_0593/IMG_0599) mostram só UMA castanha da HM-01
com dedo montado — é nela que a placa em L do dedo fixo é parafusada. A
castanha oposta está nua.

O modelo mantinha os dois meshes originais, então a simulação desenhava
um dedo azul em -X que não existe no robô. Como a garra não abre nem
fecha durante a tarefa, era geometria fantasma.

Grip1 (mesma origem do JTool) fica: é a lingueta que o garfo abraça.

Co-Authored-By: Claude Opus 5 <noreply@anthropic.com>
Claude-Session: https://claude.ai/code/session_01Ra2BbYQxYWhbcCFkGE7vAN

File: src/b166er_robot/urdf/movemaster/movemaster.urdf.xacro (robot description, xacro)
@@ -254,5 +254,26 @@
          menos resolução angular. Consequência já calculada: a detecção
          confiável com a tag de 220 mm cai de ~3,9 m para ~2,8 m. ═══ -->
-    <gazebo reference="t265_link">
+    <!-- A FISHEYE1 NÃO ESTÁ NO CENTRO DA T265 (medido em 2026-08-26).
+         O driver publica a extrínseca t265_link -> fisheye1_optical como
+         translação de 32 mm em Y, rotação [-90°, 0°, -90°] (a convenção
+         óptica padrão).
+         O modelo assumia os dois no mesmo ponto. Um deslocamento fixo na
+         origem do raio de projeção produz erro de pose que cresce com a
+         distância angular à tag — candidato direto ao erro proporcional
+         que travou a simulação em 2026-08-26.
+         Aqui o sensor é declarado num link próprio, deslocado, em vez de
+         pendurado direto no t265_link. -->
+    <joint name="JFisheye1" type="fixed">
+      <origin xyz="0 0.032 0" rpy="0 0 0"/>
+      <parent link="t265_link"/>
+      <child link="t265_fisheye1_frame"/>
+    </joint>
+    <link name="t265_fisheye1_frame">
+      <inertial>
+        <mass value="0.001"/>
+        <inertia ixx="1e-7" ixy="0" ixz="0" iyy="1e-7" iyz="0" izz="1e-7"/>
+      </inertial>
+    </link>
+    <gazebo reference="t265_fisheye1_frame">
       <sensor type="wideanglecamera" name="t265_fisheye1">
         <update_rate>15.0</update_rate>
@@ -260,5 +281,11 @@
         <visualize>false</visualize>
         <camera>
-          <horizontal_fov>2.7367</horizontal_fov>
+          <!-- 170,3° — MEDIDO na T265 real em 2026-08-26, não a
+               especificação. Invertendo fx=285,32 do camera_info do
+               driver para 848 px com r=f·θ: hfov = 2·(w/2)/fx = 2,9724
+               rad. A especificação de 163° diagonal me levara a assumir
+               157° horizontais; a lente é mais aberta que isso, o que
+               reduz a resolução angular de 5,41 para 4,98 px/grau. -->
+          <horizontal_fov>2.9724</horizontal_fov>
           <image><width>848</width><height>800</height><format>R8G8B8</format></image>
           <clip><near>0.05</near><far>50.0</far></clip>
@@ -277,5 +304,5 @@
                o /camera/fisheye1/camera_info é o fisheye_info_fixer. -->
           <cameraInfoTopicName>camera_info_gazebo</cameraInfoTopicName>
-          <frameName>t265_link</frameName>
+          <frameName>t265_fisheye1_frame</frameName>
           <hackBaseline>0.0</hackBaseline>
         </plugin>
@@ -368,9 +395,15 @@
       <child link="Grip1"/>
     </joint>
-    <joint name="JGrip2" type="fixed">
-      <origin xyz="0 0 0" rpy="0 0 0"/>
-      <parent link="GripCube"/>
-      <child link="Grip2"/>
-    </joint>
+    <!-- Grip2 REMOVIDO em 2026-08-27.
+         Nas fotos da bancada (IMG_0593 / IMG_0599, 2026-08-26) só UMA
+         das castanhas da HM-01 tem dedo montado — é nela que a placa em
+         L do dedo fixo é parafusada (4 parafusos, grade 2x2). A castanha
+         oposta está NUA, apenas com os furos roscados à vista.
+         O modelo mantinha os dois meshes originais, então a simulação
+         desenhava um dedo azul em −X que não existe no robô. Como a
+         garra não abre nem fecha na tarefa (ver o bloco do DEDO FIXO
+         abaixo), esse dedo é massa e geometria fantasma: some daqui.
+         Grip1 (em +0.03, mesma origem do JTool) fica: é a lingueta que o
+         garfo do dedo fixo abraça. -->
     <link name="Grip1">
       <visual>
@@ -378,15 +411,4 @@
         <geometry>
           <mesh filename="package://movemaster_control/3D_Models/Grip1.stl" scale="0.001 0.001 0.001"/>
-        </geometry>
-        <material name="L1Color">
-          <color rgba="0.15 0.2 0.8 1"/>
-        </material>
-      </visual>
-    </link>
-    <link name="Grip2">
-      <visual>
-        <origin xyz="-0.03 0 -0.08" rpy="0 1.57 -1.57" />
-        <geometry>
-          <mesh filename="package://movemaster_control/3D_Models/Grip2.stl" scale="0.001 0.001 0.001"/>
         </geometry>
         <material name="L1Color">
@@ -409,5 +431,5 @@
          Montada no mesmo ponto que o gripper visual (GripCube, ponta
          em z=-0.08 no frame do GripCube, mesmo offset dos meshes
-         Grip1/Grip2) — SEM junta própria (fixed), então herda a fusão
+         Grip1) — SEM junta própria (fixed), então herda a fusão
          de corpo rígido do Gazebo junto com L5/CameraSupport/GripCube
          (mesmo comportamento já documentado nas fixtures: um

Commit message: fix(b166er_robot): degrau não colide mais com a própria haste
A caixa de colisão do degrau tinha a largura do VISUAL (para desenhar o
L inteiro), o que a fazia compartilhar uma face de 10,4 mm com a haste
do tool_rod, em z=0. Duas faces coincidentes geram contato continuamente:
a captura de contatos de 2026-08-27 registrou 1,1 MILHÃO de pares
tool_rod x tool_tip em ~90 s de simulação.

É o suspeito do travamento do J1 numa execução anterior — J1 comandado
subindo de 6,4 para 23,6 graus, medido parado, defasagem crescendo até
16 graus enquanto J2..J5 seguiam dentro de 1 grau.

A colisão agora cobre só o trecho que se projeta, com 0,5 mm de recuo.
A face superior do degrau (z=0) é preservada: é ela que sustenta o arame.

Co-Authored-By: Claude Opus 5 <noreply@anthropic.com>
Claude-Session: https://claude.ai/code/session_01Ra2BbYQxYWhbcCFkGE7vAN

File: src/b166er_robot/urdf/movemaster/movemaster.urdf.xacro (robot description, xacro)
@@ -545,7 +545,22 @@
         <material name="ToolColor"><color rgba="0.85 0.75 0.1 1"/></material>
       </visual>
+      <!-- COLISÃO SÓ DA PARTE QUE SE PROJETA, não da largura visual.
+           A caixa visual acima vai de x=+5,2 mm a x=-25,2 mm para
+           desenhar o L inteiro — mas isso faz ela compartilhar uma FACE
+           inteira (z=0, de x=-5,2 a +5,2) com a haste do tool_rod. Duas
+           faces coincidentes no mesmo corpo rígido geram contato
+           permanentemente: a captura de 2026-08-27 registrou 1,1 MILHÃO
+           de pares tool_rod x tool_tip em ~90 s de simulação, e é o
+           suspeito do travamento do J1 numa execução anterior (J1
+           comandado subindo, medido parado, defasagem crescendo até 16°
+           enquanto J2..J5 seguiam dentro de 1°).
+           Aqui a caixa começa onde a haste termina, com 0,5 mm de
+           recuo, de modo que os dois sólidos se encostem no máximo por
+           uma aresta. A face SUPERIOR do degrau (z=0) é preservada
+           porque é ela que sustenta o arame do anel. -->
+      <xacro:property name="degrau_gap" value="0.0005"/>
       <collision>
-        <origin xyz="${-dedo_degrau_l/2} 0 ${-dedo_degrau_z/2}"/>
-        <geometry><box size="${dedo_degrau_l + dedo_haste_x} ${dedo_haste_y} ${dedo_degrau_z}"/></geometry>
+        <origin xyz="${-(dedo_degrau_l/2 + dedo_haste_x/2 + degrau_gap)} 0 ${-dedo_degrau_z/2}"/>
+        <geometry><box size="${dedo_degrau_l} ${dedo_haste_y} ${dedo_degrau_z}"/></geometry>
       </collision>
       <inertial>
