Commit message: feat(b166er_robot): remonta a T265 nos furos do suporte com a malha oficial
A T265 estava 4 cm à frente do suporte, olhando 30,3° fora da direção da
ferramenta, e desenhada com uma malha (realsense.stl, 148x30x28 mm) que
não é uma T265. O Marco comparou a simulação com a câmera da bancada e
apontou os três problemas em sequência: posição, modelo e o lado do
conector.

Posição pelos furos, não pelo berço: a malha do suporte tem dois furos
M3 (⌀3,5 mm) espaçados 50,50 mm sobre um plano de apoio em z=6,50 mm —
o padrão de montagem da T265. Face das lentes = apoio + 12,5 mm de
espessura. A origem do t265_link é o centro de rastreamento, que a doc
da Intel define como o ponto médio entre as duas fisheyes.

Malha oficial: common/res/sources/T265.obj do librealsense (Apache-2.0,
verificada), convertida para STL. Mede 108,00 x 24,49 x 12,50 mm. As
fisheyes estão nela separadas por 64,74 mm (baseline nominal 64 mm), e
posicionando pelo ponto médio delas caem em y = ±0,03237 m no link —
contra os +0,032 m que JFisheye1 usa desde 2026-08-26, medidos na
bancada com o driver real. 0,4 mm entre a malha da Intel e a régua.

Rolagem: 180° em torno do eixo óptico em relação à primeira tentativa,
porque o conector USB-C caía do lado errado. É a única rotação rígida
que troca o lado do conector sem tirar a câmera de mira.

kinematics.py (_T_L5_T265) acompanha o URDF: é uma cópia desatualizada
desse tipo que já pôs a parede 0,795 m fora do lugar.

Consequência: o sensor andou 51,8 mm, o eixo óptico girou 30,3° e a
fisheye1 atravessou 64 mm de lado. T_T265_TOOLTIP foi de 0,1531 m para
0,2024 m. As poses calibradas contra a montagem antiga precisam ser
revalidadas.

Co-Authored-By: Claude Fable 5.1 <noreply@anthropic.com>
Claude-Session: https://claude.ai/code/session_01P4v3ZvEh2bwom2DYHA9moN

File: src/b166er_robot/urdf/movemaster/movemaster.urdf.xacro (robot description, xacro)
@@ -220,15 +220,97 @@
       </visual>
     </link>
-    <!-- T265 montada no end-effector, mesma região do gripper (confirmado por foto do robô real) -->
+    <!-- T265 NO BERÇO DE CIMA DO SUPORTE — posição MEDIDA na malha, não
+         estimada (2026-09-02, a pedido do Marco: "a T265 deve ir para o
+         suporte na posição superior").
+         O suporte_movemaster_com_cameras.stl tem DUAS câmeras modeladas
+         nele (o nome do arquivo não é acidente), ambas de 90x25x25 mm com
+         três lentes espaçadas de 50 mm — geometria de D435, uma no berço
+         de baixo (inclinada) e outra no de cima (alinhada aos eixos). A
+         T265 vai no de cima.
+         MAS A POSIÇÃO NÃO É O BERÇO: é onde os FUROS põem a T265. O
+         Marco: "ela fixou-se na mesma posição dos furos do suporte". A
+         câmera modelada no berço de cima é uma D435 (90x25x25 mm, três
+         lentes espaçadas de 50 mm); a T265 da bancada tem 108x24,5x12,5
+         mm — METADE da espessura. Apoiar a T265 no mesmo plano e assumir
+         a face da D435 punha a origem 12,8 mm à frente do lugar.
+         Medido na malha, separada em componentes conectadas e
+         transformada pelo <visual> do CameraSupport (escala 1e-3,
+         rpy 0 3.14 0, xyz 0.255 -0.18 0):
+           furos de fixação (⌀3,5 mm = M3)  x_stl 230.92 e 281.42
+                                            y_stl 266.03 (mesma linha)
+           espaçamento entre furos          50,50 mm
+           plano de apoio da peça           z_stl 6,50
+         Os 50,50 mm entre furos são o padrão de montagem da T265 — é o
+         que confirma que estes furos são dela, e não do berço da D435.
+         Face das lentes = apoio + espessura = 6,50 + 12,5 = 19,00 mm.
+         A ORIGEM DO t265_link É O CENTRO DE RASTREAMENTO, e a doc da
+         Intel (doc/t265.md do librealsense) é explícita: "the center of
+         tracking corresponds to the center location between the right and
+         left monochrome imagers on the PCB" — nem o centro do corpo, nem
+         um canto. É por isso que JFisheye1 desloca 32 mm logo abaixo:
+         metade da baseline de 64 mm. Origem, então, no meio dos furos em
+         X e Y, no plano das lentes em Z.
+         ORIENTAÇÃO: rpy="-1.5708 1.5708 0" põe o eixo óptico (+X) em -Z
+         do CameraSupport — exatamente para onde a ferramenta aponta. A
+         montagem anterior (rpy="0 2.1 1.57") olhava 30,3° fora de -Z, e
+         era a tal "rotação tortuosa" que o comentário da câmera de tarefa
+         menciona logo abaixo.
+         ROLAGEM: 180° em torno do EIXO ÓPTICO em relação ao que estava
+         aqui até 2026-09-02. Eu tinha preservado a rolagem antiga por
+         conservadorismo, e ficou errado — o Marco viu na simulação e
+         corrigiu: "a conexão da camera fica do outro lado". O conector
+         USB-C fica na ponta -X da malha (a face de lá tem 338 triângulos
+         em 231 mm², contra 120 em 331 mm² do outro lado: mais geometria
+         em menos área é o recorte do conector), e essa ponta estava
+         caindo em +X do CameraSupport quando deveria cair em -X.
+         O giro é em torno do eixo óptico porque é a ÚNICA rotação rígida
+         que troca o conector de lado sem tirar a câmera de mira: o eixo
+         óptico continua em -Z. Em troca, a câmera fica de cabeça para
+         baixo em relação a antes — que é a montagem real da bancada.
+         CONSEQUÊNCIA QUE NÃO É COSMÉTICA: a fisheye1 fica 32 mm em +Y do
+         link, então ela atravessou 64 mm para o outro lado do suporte. A
+         câmera que enxerga mudou de lugar, e com ela a geometria da
+         detecção. A extrínseca interna (JFisheye1, medida na bancada em
+         2026-08-26) não muda com isso: ela descreve o dispositivo por
+         dentro, não como ele foi parafusado.
+         ATENÇÃO: esta transformada é duplicada em kinematics.py
+         (_T_L5_T265). As duas TÊM que andar juntas — foi uma cópia
+         desatualizada desse tipo que pôs a parede 0,795 m fora do lugar e
+         ainda assim terminou a missão em MISSION_OK. -->
     <joint name="t265_mount_joint" type="fixed">
-      <origin xyz="0 0.075 -0.070" rpy="0 2.1 1.57"/>
+      <origin xyz="-0.0011 0.0860 -0.0194" rpy="1.5708 1.5708 0"/>
       <parent link="CameraSupport"/>
       <child link="t265_link"/>
     </joint>
     <link name="t265_link">
-      <visual>
-        <origin xyz="0 0 0" rpy="0 0 0"/>
-        <geometry>
-          <mesh filename="package://movemaster_control/3D_Models/realsense.stl"/>
+      <!-- MALHA OFICIAL DA INTEL, não uma aproximação.
+           A realsense.stl que estava aqui mede 148x30x28 mm e não é uma
+           T265 — o Marco reparou olhando a simulação ("a modelagem da
+           T265 que vc está simulando é um pouco diferente da T265 que
+           tenho na bancada") e mandou a foto da peça e o repositório.
+           Esta malha vem de common/res/sources/T265.obj do librealsense
+           (Apache-2.0), convertida para STL binário, e mede
+           108,00 x 24,49 x 12,50 mm — a T265 de verdade.
+           POSE DA MALHA, e por que não é arbitrária: a origem do link é o
+           CENTRO DE RASTREAMENTO, que a doc da Intel define como o ponto
+           médio entre as duas fisheyes. Achei as duas na malha (as
+           concavidades da face frontal) em X = -30,86 e X = +33,88 mm,
+           separadas por 64,74 mm — a baseline nominal de 64 mm. O rpy
+           gira os eixos da malha (X = linha das fisheyes, Y = altura,
+           Z = frente) para os do link (X = eixo óptico, Y = linha das
+           fisheyes, Z = altura), e o xyz leva o ponto médio delas para a
+           origem.
+           A CONFERÊNCIA QUE IMPORTA: com esta pose, as fisheyes caem em
+           y = ±0,03237 m no t265_link. O JFisheye1 logo abaixo usa
+           +0,032, medido na bancada em 2026-08-26, por outro caminho e
+           em outro dia. 0,4 mm de diferença entre a malha da Intel e a
+           régua da bancada — as duas descrevem a mesma peça.
+           O corpo fica assimétrico em torno da origem (y de -0,0636 a
+           +0,0444) e isso está certo: o centro de rastreamento não é o
+           centro do corpo, as fisheyes não são simétricas nas pontas. -->
+      <visual>
+        <origin xyz="0 -0.00151 0.00033" rpy="1.5708 0 1.5708"/>
+        <geometry>
+          <mesh filename="package://b166er_robot/meshes/movemaster/t265.stl" scale="0.001 0.001 0.001"/>
         </geometry>
         <material name="t265_color">
@@ -328,7 +410,11 @@
          Montada no mesmo ponto/direção do JTool (offset z=-0.08 a
          partir do GripCube, mesmo "para frente" que a ferramenta
-         aponta) — olhando para onde o robô vai manipular, não para
-         onde o T265 fisicamente aponta (rotação tortuosa,
-         rpy="0 2.1 1.57", inconveniente para uma câmera de tarefa). ═══ -->
+         aponta) — olhando para onde o robô vai manipular.
+         NOTA (2026-09-02): a justificativa original era que o T265
+         apontava para outro lado (a "rotação tortuosa" rpy="0 2.1 1.57").
+         Isso deixou de valer: remontado nos furos do berço de cima, o
+         T265 olha reto para -Z, a MESMA direção desta câmera. O que
+         separa as duas hoje é só o sensor — fisheye equidistante contra
+         pinhole — e esta continua não existindo na bancada. ═══ -->
     <joint name="JTaskCamera" type="fixed">
       <origin xyz="0 0 -0.08" rpy="0 0 0"/>
@@ -571,4 +657,13 @@
     <gazebo reference="tool_rod"><material>Gazebo/Yellow</material></gazebo>
     <gazebo reference="tool_tip"><material>Gazebo/Yellow</material></gazebo>
+    <!-- T265 em VERDE no Gazebo (pedido do Marco, 2026-09-02). O
+         <material> do URDF, logo acima no t265_link, vale só para o
+         RViz; o Gazebo ignora e usa este bloco. Em cinza escuro a
+         câmera se confundia com o corpo do punho nas capturas de tela,
+         que é como acompanhamos a manipulação. Verde e não laranja
+         porque a haste e o degrau já são amarelos: laranja ficava perto
+         demais deles na paleta, e o que precisa se distinguir é
+         justamente câmera x ferramenta. -->
+    <gazebo reference="t265_link"><material>Gazebo/Green</material></gazebo>
     <xacro:macro name="arm_transmission" params="joint_name">
       <transmission name="${joint_name}_trans">

Commit message: chore(b166er_robot): remove as câmeras decorativas da malha do suporte
A malha suporte_movemaster_com_cameras.stl traz duas D435 desenhadas
sobre a chapa (90x25x25 mm, três lentes espaçadas de 50 mm cada).
Nenhuma existe na bancada: o robô tem uma T265, declarada como link
próprio. Câmera desenhada que não é sensor engana quem olha a simulação
justamente para conferir a montagem — foi uma delas que se confundiu
com a T265 nesta sessão. O Marco pediu para retirar.

Gerada por componentes conectadas, removendo toda componente contida em
y_stl > 220 (a faixa das duas D435): 268.832 dos 269.936 triângulos
saíram, sobrando só a estrutura. Os furos de fixação da T265 foram
preservados e conferidos. A malha nova vive em b166er_robot/meshes, e a
original segue intocada no submódulo movemaster_control.

Co-Authored-By: Claude Fable 5.1 <noreply@anthropic.com>
Claude-Session: https://claude.ai/code/session_01P4v3ZvEh2bwom2DYHA9moN

File: src/b166er_robot/urdf/movemaster/movemaster.urdf.xacro (robot description, xacro)
@@ -213,5 +213,16 @@
         <origin xyz="0.255 -0.18 0" rpy="0 3.14 0" />
         <geometry>
-          <mesh filename="package://movemaster_control/3D_Models/suporte_movemaster_com_cameras.stl" scale="0.001 0.001 0.001"/>
+          <!-- SEM AS CÂMERAS DECORATIVAS (2026-09-02, a pedido do Marco).
+               A malha original, suporte_movemaster_com_cameras.stl, traz
+               DUAS D435 desenhadas em cima da chapa. Nenhuma delas existe
+               na bancada: o robô tem uma T265, e ela é declarada como
+               link próprio logo abaixo. Câmera desenhada que não é sensor
+               engana quem olha a simulação para conferir a montagem — foi
+               exatamente uma delas que a gente confundiu com a T265.
+               Aqui ficou só a estrutura: 1104 triângulos contra 269936,
+               e os furos de fixação preservados (é por eles que a T265 se
+               posiciona). Gerada por componentes conectadas; a original
+               segue intocada no submódulo. -->
+          <mesh filename="package://b166er_robot/meshes/movemaster/suporte_movemaster.stl" scale="0.001 0.001 0.001"/>
         </geometry>
         <material name="CameraSupportColor">

Commit message: feat(b166er_robot): dedo fixo com haste e degrau de 10 x 10 e afunilamento em rampa
Revisão da ferramenta com o Marco (2026-09-02). Três mudanças na peça:

Seção da haste: 10,4 x 20 -> 10 x 10. A redução é no plano Y, o que o
afunilamento já não reduzia; os 10,4 em X eram escolha minha e "10 ou
10,4 não fará muita diferença".

Degrau: 20 x 17 -> 10 x 10, acompanhando a haste, altura inclusive. A
projeção de 20 mm em -X não muda, nem o comprimento garfo + afunil +
haste (0,115), então JToolTip e toda a cinemática ficam como estão.

Afunilamento: o bloco 15 x 22 de cantos vivos vira uma rampa contínua
de 20 x 25 para 10 x 10 (malha gerada em código, 12 triângulos). A
colisão fica como caixa 10 x 10 — a rampa nunca encosta em nada.

O que a redução compra: o degrau 20 x 17 num oval de 30 x 40 tinha
limite de ~20° de rolagem antes de o canto sair do contorno, e foi isso
que decidiu 0,54 contra 0,62 na distância de engate. Um 10 x 10 tem
diagonal de 14,1 mm e cabe no vão de 30 em qualquer rolagem: a
restrição que mandava na tarefa deixa de existir na geometria. O que
custa: rigidez à flexão em Y cai por 8 e a face de apoio do arame
encurta de 20 para 10 mm.

Dependências ajustadas pela fórmula que o próprio YAML declara: a
descida da captura passa de 11,5 para 15 mm e o alvo de -3,0 para
-10,0 mm (face de baixo do degrau na aba inferior do anel, em -20).
Calculado, ainda não medido com a peça nova. As tolerâncias por eixo
NÃO foram relaxadas: as folgas dobraram, mas afrouxar sem medir é o que
o arquivo existe para impedir — fica para a revalidação.

Co-Authored-By: Claude Fable 5.1 <noreply@anthropic.com>
Claude-Session: https://claude.ai/code/session_01P4v3ZvEh2bwom2DYHA9moN

File: src/b166er_robot/urdf/movemaster/movemaster.urdf.xacro (robot description, xacro)
@@ -550,10 +550,13 @@
          temos como controlar bem e transforma a garra num ponto de
          ancoragem rígido.
-         Geometria do desenho (mm), ao longo de -Z a partir da montagem:
-           garfo   25 de altura, 20 de profundidade, abas de 10
-           afunil. 10
-           haste   80, seção 10,4 x 20,0
-           ponta   20 de altura, 30,4 de largura, 20 de profundidade
-           total  135
+         Geometria (mm), ao longo de -Z a partir da montagem — REVISADA
+         em 2026-09-02 com o Marco (ver o bloco de propriedades abaixo):
+           garfo   25 de altura, 20 x 25 de seção, abas de 10
+           afunil. 10, RAMPA de 20 x 25 para 10 x 10 (inclinada, sem
+                   canto vivo — o bloco 15 x 22 que estava aqui era erro
+                   de modelagem meu, a peça é uma transição contínua)
+           haste   80, seção 10 x 10
+           degrau  10 de altura, 10 de largura, 20 de projeção em -X
+           total  125
          A ponta alargada é o que prende o elo: a haste de 10,4 mm passa
          pelo olhal, e o degrau de 20 mm (30,4 − 10,4) impede o anel de
@@ -579,11 +582,24 @@
     <xacro:property name="dedo_afun_h"   value="0.010"/>
     <xacro:property name="dedo_haste_l"  value="0.080"/>
-    <xacro:property name="dedo_haste_x"  value="0.0104"/>
-    <xacro:property name="dedo_haste_y"  value="0.020"/>
-    <!-- Saliência do degrau além da haste: 30,4 − 10,4 = 20 mm. É o
+    <!-- SEÇÃO 10 x 10 (2026-09-02). O Marco reduziu a haste e o degrau
+         no plano Y de 20 para 10 mm — "teremos uma haste 10 mm x 10 mm, e
+         o degrau vai acompanhar essa medida também", altura do degrau
+         inclusive. Os 10,4 em X eram escolha minha (lingueta de 10 +
+         folga); "10 ou 10,4 não fará muita diferença", então 10.
+         O QUE ISSO COMPRA: o degrau era 20 x 17 num oval de 30 x 40, e
+         a ROLAGEM em torno do próprio eixo decidia se ele passava — além
+         de ~20° o canto saía do contorno (foi isso que fixou a distância
+         de engate em 0,54 contra 0,62, ver chave_mission.py). Um 10 x 10
+         tem diagonal de 14,1 mm: cabe no vão de 30 em QUALQUER rolagem.
+         A restrição que mandava na tarefa deixa de existir.
+         O QUE CUSTA: rigidez à flexão no plano Y cai por 8 (I ∝ h³), e a
+         face de apoio do arame encurta de 20 para 10 mm. -->
+    <xacro:property name="dedo_haste_x"  value="0.010"/>
+    <xacro:property name="dedo_haste_y"  value="0.010"/>
+    <!-- Projeção do degrau além da haste: 20 mm, inalterada. É o
          comprimento útil que fica atravessado no furo e sustenta o
          arame do olhal. -->
     <xacro:property name="dedo_degrau_l" value="0.020"/>
-    <xacro:property name="dedo_degrau_z" value="0.017"/>
+    <xacro:property name="dedo_degrau_z" value="0.010"/>
     <xacro:property name="tool_length"
                     value="${dedo_garfo_h + dedo_afun_h + dedo_haste_l}"/>
@@ -603,12 +619,20 @@
         <geometry><box size="0.020 0.025 ${dedo_garfo_h}"/></geometry>
       </collision>
-      <visual>
-        <origin xyz="0 0 ${-dedo_garfo_h - dedo_afun_h/2}"/>
-        <geometry><box size="0.015 0.022 ${dedo_afun_h}"/></geometry>
+      <!-- AFUNILAMENTO INCLINADO. Tronco de pirâmide gerado em código
+           (meshes/movemaster/dedo_afunilamento.stl, em METROS, já no
+           frame deste link: topo 20 x 25 em z = -0,025, base 10 x 10 em
+           z = -0,035). Se dedo_garfo_h ou dedo_afun_h mudarem, a malha
+           tem que ser regerada — ela não lê as propriedades.
+           A colisão fica como CAIXA 10 x 10, a seção menor: a rampa
+           nunca encosta em nada (fica 90 mm acima do degrau), e caixa é
+           mais barata e mais estável no ODE que trimesh. -->
+      <visual>
+        <origin xyz="0 0 0"/>
+        <geometry><mesh filename="package://b166er_robot/meshes/movemaster/dedo_afunilamento.stl"/></geometry>
         <material name="ToolColor"/>
       </visual>
       <collision>
         <origin xyz="0 0 ${-dedo_garfo_h - dedo_afun_h/2}"/>
-        <geometry><box size="0.015 0.022 ${dedo_afun_h}"/></geometry>
+        <geometry><box size="${dedo_haste_x} ${dedo_haste_y} ${dedo_afun_h}"/></geometry>
       </collision>
       <visual>

Commit message: feat(b166er_robot): limita o esforço do J4 simulado a 4,2 N·m pela especificação do RV-M2
Os manuais não dão torque de junta; dão carga nominal 1,0 kg e a
estimativa estática de ~1,2 N·m no punho (12 N a 0,1 m). O limite do
atuador simulado passa a ser o peso próprio do punho na pior postura
(L5 1,7 kg a 0,08 m + ferramenta 0,16 kg a ~0,25 m ≈ 1,7 N·m) mais duas
vezes a referência estática (2,4 N·m): 4,2 N·m, contra os 20 N·m de
antes. A bateria de contato diz se o híbrido ainda abre a chave com um
punho desse tamanho.

Co-Authored-By: Claude Fable 5.1 <noreply@anthropic.com>
Claude-Session: https://claude.ai/code/session_01P4v3ZvEh2bwom2DYHA9moN

File: src/b166er_robot/urdf/movemaster/movemaster.urdf.xacro (robot description, xacro)
@@ -160,5 +160,23 @@
       <child link="L4"/>
       <!-- Punho pitch (wrist pitch): ±110° no manual -->
-      <limit upper="1.91986" lower="-1.91986" effort="20" velocity="3.14" />
+      <!-- ESFORÇO LIMITADO PELA ESPECIFICAÇÃO (2026-09-08, decisão do
+           Marco: "limita o J4 e roda as baterias"). Os manuais do RV-M2
+           não dão torque de junta; dão carga nominal 1,0 kg (máx. 2,0) e
+           a estimativa estática do Marco: 12 N a 0,1 m = 1,2 N·m no
+           punho. Esse número é o que o punho suporta ALÉM do próprio
+           peso, então o limite do atuador simulado = peso próprio do
+           punho na pior postura (horizontal) + 2 × 1,2 N·m:
+             L5 1,7 kg a 0,08 m          1,33 N·m
+             ferramenta 0,16 kg a ~0,25 m 0,40 N·m
+             (L4 2,5 kg tem CG no eixo; câmera e suporte sem inércia)
+             margem 2 × 1,2               2,40 N·m
+             total                        4,2 N·m
+           Antes era 20 N·m: o destrava íntegro simulado exigia 2–3 N·m no
+           J4 (RELATORIO6), e ao ser retro-acionado pelo anel o J4 saturava
+           nos 20 e colapsava para 110°. Com 4,2 a pergunta que a bateria
+           responde é se o híbrido ainda abre a chave com um punho do
+           tamanho do real; se não abrir, o destrava tem que vir de J2/J3
+           com o punho travado. -->
+      <limit upper="1.91986" lower="-1.91986" effort="4.2" velocity="3.14" />
       <dynamics damping="0.3" friction="0.0"/>
     </joint>
