Commit message: feat(b166er_robot): dedo v2 — degrau girado 90°, sai em +Y no sentido das abas
Pedido do Marco (2026-09-29): "o degrau tem que rotacionar 90 graus",
opção B do desenho de alternativas. A direção do degrau passa a viver
numa constante só, kinematics.DEGRAU_DIR_TIP = +Y (era −X implícito em
degrau_dir, na _feat da ik_tooltip_com_degrau e na _alvo_R da
ik_tooltip_nivelado). No URDF as caixas visual e de colisão do tool_tip
acompanham (+Y, mesma projeção de 20 mm e seção 10 × 10). A missão e o
YAML das fases não mudam: o vínculo é degrau ∥ eixo do furo no frame da
parede. Validado em simulação: MISSION_OK, chave 30,0°, DEPLOY com J5 a
79,7° (o punho rodou os 90° esperados), destrava com lingueta 12,4 mm.

Co-Authored-By: Claude Fable 5.1 <noreply@anthropic.com>
Claude-Session: https://claude.ai/code/session_01P4v3ZvEh2bwom2DYHA9moN

File: src/b166er_robot/urdf/movemaster/movemaster.urdf.xacro (robot description, xacro)
@@ -575,5 +575,7 @@
                    de modelagem meu, a peça é uma transição contínua)
            haste   80, seção 10 x 10
-           degrau  10 de altura, 10 de largura, 20 de projeção em -X
+           degrau  10 de altura, 10 de largura, 20 de projeção em +Y
+                   (DEDO v2, 2026-09-29: girado 90° em torno da haste —
+                   sai no sentido das ABAS do garfo. Na v1 saía em -X.)
            total  125
          A ponta alargada é o que prende o elo: a haste de 10,4 mm passa
@@ -674,17 +676,22 @@
     </joint>
     <!-- DEGRAU — o dedo horizontal que atravessa o olhal.
-         Sai em −X a partir do eixo da haste; girando J5 a peça aponta
-         para a direita ou para a esquerda, como o Marco descreveu.
+         DEDO v2 (2026-09-29, "o degrau tem que rotacionar 90 graus",
+         opção B): sai em +Y a partir do eixo da haste, no sentido das
+         abas do garfo em U. Na v1 saía em −X. Girando J5 a peça aponta
+         para a direita ou para a esquerda, como o Marco descreveu — só
+         que agora com o punho 90° rodado em relação à v1. A direção
+         que a cinemática usa é kinematics.DEGRAU_DIR_TIP = +Y: os dois
+         têm que casar.
          A ORIGEM DESTE LINK é a referência da tarefa: é aqui que o
          arame do anel repousa depois da descida de 5 mm. -->
     <link name="tool_tip">
       <visual>
-        <origin xyz="${-dedo_degrau_l/2} 0 ${-dedo_degrau_z/2}"/>
-        <geometry><box size="${dedo_degrau_l + dedo_haste_x} ${dedo_haste_y} ${dedo_degrau_z}"/></geometry>
+        <origin xyz="0 ${dedo_degrau_l/2} ${-dedo_degrau_z/2}"/>
+        <geometry><box size="${dedo_haste_x} ${dedo_degrau_l + dedo_haste_y} ${dedo_degrau_z}"/></geometry>
         <material name="ToolColor"><color rgba="0.85 0.75 0.1 1"/></material>
       </visual>
       <!-- COLISÃO SÓ DA PARTE QUE SE PROJETA, não da largura visual.
-           A caixa visual acima vai de x=+5,2 mm a x=-25,2 mm para
-           desenhar o L inteiro — mas isso faz ela compartilhar uma FACE
+           A caixa visual acima vai de y=-5 mm a y=+25 mm (v2; na v1
+           era x=+5,2 a x=-25,2) para desenhar o L inteiro — mas isso faz ela compartilhar uma FACE
            inteira (z=0, de x=-5,2 a +5,2) com a haste do tool_rod. Duas
            faces coincidentes no mesmo corpo rígido geram contato
@@ -700,6 +707,6 @@
       <xacro:property name="degrau_gap" value="0.0005"/>
       <collision>
-        <origin xyz="${-(dedo_degrau_l/2 + dedo_haste_x/2 + degrau_gap)} 0 ${-dedo_degrau_z/2}"/>
-        <geometry><box size="${dedo_degrau_l} ${dedo_haste_y} ${dedo_degrau_z}"/></geometry>
+        <origin xyz="0 ${dedo_degrau_l/2 + dedo_haste_y/2 + degrau_gap} ${-dedo_degrau_z/2}"/>
+        <geometry><box size="${dedo_haste_x} ${dedo_degrau_l} ${dedo_degrau_z}"/></geometry>
       </collision>
       <inertial>

Commit message: feat(whole_body): garra_dx — posição da castanha do dedo (aberta 0,03 / fechada 0,0)
A garra não tem junta na simulação; o que muda entre "aberta" e
"fechada" é onde a castanha com o dedo fica travada no eixo transversal
do GripCube (curso 0–60 mm da mão DC do RV-M2, 30 mm por castanha).
O valor entra por um só argumento: xacro:arg garra_dx no URDF (JTool e
visual Grip1), GARRA_DX em kinematics.py via B166ER_GARRA_DX, e o arg
garra_dx em b166er_wb.launch (xacro, env e repasse a b166er_gazebo.launch,
que recarrega o robot_description e sobrescrevia o valor) e em
chave_mission.launch. A missão confere o JTool do robot_description
contra a cinemática e aborta se discordarem. Default continua 0,03.

Co-Authored-By: Claude Fable 5.1 <noreply@anthropic.com>
Claude-Session: https://claude.ai/code/session_01P4v3ZvEh2bwom2DYHA9moN

File: src/b166er_robot/urdf/movemaster/movemaster.urdf.xacro (robot description, xacro)
@@ -5,4 +5,19 @@
        movemaster_state_publisher real, para que o mesmo /joint_states
        sirva tanto a simulação quanto o hardware. -->
+  <!-- POSIÇÃO DA CASTANHA onde o dedo fixo monta (2026-09-30). A mão DC
+       do RV-M2 (folheto Mitsubishi, "DC motor hand") tem curso de 0 a
+       60 mm entre as faces internas das castanhas: cada castanha anda
+       30 mm no eixo transversal (x do GripCube). A garra NÃO tem junta
+       neste modelo — ela não abre nem fecha na tarefa — então a posição
+       em que ela fica travada entra como argumento:
+         garra_dx = 0.03  → garra ABERTA (valor histórico do modelo;
+                            dedo 30 mm fora do eixo do J5)
+         garra_dx = 0.0   → garra FECHADA (dedo no eixo do J5; o rolamento
+                            do punho deixa de mover a ponta)
+       Tem que casar com B166ER_GARRA_DX lido por kinematics.py
+       (_T_L5_TOOLTIP): b166er_wb.launch passa os dois a partir do mesmo
+       arg garra_dx, e chave_mission.py confere no robot_description. -->
+  <xacro:arg name="garra_dx" default="0.03"/>
+  <xacro:property name="garra_dx" value="$(arg garra_dx)"/>
   <xacro:macro name="movemaster_rv_m2" params="parent xyz:='0 0 0' rpy:='0 0 0'">
     <joint name="movemaster_mount_joint" type="fixed">
@@ -519,9 +534,9 @@
          garra não abre nem fecha na tarefa (ver o bloco do DEDO FIXO
          abaixo), esse dedo é massa e geometria fantasma: some daqui.
-         Grip1 (em +0.03, mesma origem do JTool) fica: é a lingueta que o
+         Grip1 (em +garra_dx, mesma origem do JTool) fica: é a lingueta que o
          garfo do dedo fixo abraça. -->
     <link name="Grip1">
       <visual>
-        <origin xyz="0.03 0 -0.08" rpy="0 1.57 -1.57" />
+        <origin xyz="${garra_dx} 0 -0.08" rpy="0 1.57 -1.57" />
         <geometry>
           <mesh filename="package://movemaster_control/3D_Models/Grip1.stl" scale="0.001 0.001 0.001"/>
@@ -625,5 +640,5 @@
                     value="${dedo_garfo_h + dedo_afun_h + dedo_haste_l}"/>
     <joint name="JTool" type="fixed">
-      <origin xyz="0.03 0 -0.08" rpy="0 0 0"/>
+      <origin xyz="${garra_dx} 0 -0.08" rpy="0 0 0"/>
       <parent link="GripCube"/>
       <child link="tool_rod"/>

Commit message: feat(b166er_robot): dedo v3 — STL da peça impressa como visual, colisões em caixas como antes
O tool_rod passa a desenhar meshes/movemaster/dedo_fixo_v3.stl (mm, já
no frame do link: z=0 no topo do garfo, degrau em +Y), no lugar das três
caixas + malha da rampa; o tool_tip fica sem visual próprio. As caixas de
colisão não mudaram (garfo 20 x 25, rampa 10 x 10, haste, degrau), para
a bateria aberta x fechada comparar só a garra.

Co-Authored-By: Claude Fable 5.1 <noreply@anthropic.com>
Claude-Session: https://claude.ai/code/session_01P4v3ZvEh2bwom2DYHA9moN

File: src/b166er_robot/urdf/movemaster/movemaster.urdf.xacro (robot description, xacro)
@@ -645,7 +645,21 @@
     </joint>
     <link name="tool_rod">
-      <visual>
-        <origin xyz="0 0 ${-dedo_garfo_h/2}"/>
-        <geometry><box size="0.020 0.025 ${dedo_garfo_h}"/></geometry>
+      <!-- VISUAL = a peça impressa (dedo v3, REV. C, 2026-09-30, pedido
+           do Marco: "usa o STL da v3 no visual"). meshes/movemaster/
+           dedo_fixo_v3.stl é gerado por scripts/gera_dedo.py (versao 3)
+           em mm, já no frame deste link: z=0 no topo do garfo, z=-125 na
+           face de baixo do degrau, degrau em +Y (y de -5 a +25), garfo
+           20 x 30 com rasgo e furos. Cobre também o tool_tip, que por
+           isso não tem visual próprio. As COLISÕES continuam em caixas
+           (garfo, rampa, haste aqui; degrau no tool_tip): caixa é mais
+           barata e estável no ODE que trimesh, e é o que o contato com
+           o olhal e o gatilho usa. As caixas ficaram EXATAMENTE como
+           antes (garfo 20 x 25, a peça tem 20 x 30; o garfo fica 90 mm
+           acima de qualquer contato), para a bateria aberta x fechada
+           comparar só a garra. Se a v3 mudar, regenerar o STL e
+           conferir que as caixas ainda batem com ele. -->
+      <visual>
+        <origin xyz="0 0 0"/>
+        <geometry><mesh filename="package://b166er_robot/meshes/movemaster/dedo_fixo_v3.stl" scale="0.001 0.001 0.001"/></geometry>
         <material name="ToolColor"><color rgba="0.85 0.75 0.1 1"/></material>
       </visual>
@@ -654,26 +668,14 @@
         <geometry><box size="0.020 0.025 ${dedo_garfo_h}"/></geometry>
       </collision>
-      <!-- AFUNILAMENTO INCLINADO. Tronco de pirâmide gerado em código
-           (meshes/movemaster/dedo_afunilamento.stl, em METROS, já no
-           frame deste link: topo 20 x 25 em z = -0,025, base 10 x 10 em
-           z = -0,035). Se dedo_garfo_h ou dedo_afun_h mudarem, a malha
-           tem que ser regerada — ela não lê as propriedades.
+      <!-- AFUNILAMENTO INCLINADO (rampa). O visual em malha própria
+           (meshes/movemaster/dedo_afunilamento.stl) saiu em 2026-09-30:
+           a rampa agora é desenhada pela malha da peça inteira acima.
            A colisão fica como CAIXA 10 x 10, a seção menor: a rampa
            nunca encosta em nada (fica 90 mm acima do degrau), e caixa é
            mais barata e mais estável no ODE que trimesh. -->
-      <visual>
-        <origin xyz="0 0 0"/>
-        <geometry><mesh filename="package://b166er_robot/meshes/movemaster/dedo_afunilamento.stl"/></geometry>
-        <material name="ToolColor"/>
-      </visual>
       <collision>
         <origin xyz="0 0 ${-dedo_garfo_h - dedo_afun_h/2}"/>
         <geometry><box size="${dedo_haste_x} ${dedo_haste_y} ${dedo_afun_h}"/></geometry>
       </collision>
-      <visual>
-        <origin xyz="0 0 ${-dedo_garfo_h - dedo_afun_h - dedo_haste_l/2}"/>
-        <geometry><box size="${dedo_haste_x} ${dedo_haste_y} ${dedo_haste_l}"/></geometry>
-        <material name="ToolColor"/>
-      </visual>
       <collision>
         <origin xyz="0 0 ${-dedo_garfo_h - dedo_afun_h - dedo_haste_l/2}"/>
@@ -701,12 +703,9 @@
          arame do anel repousa depois da descida de 5 mm. -->
     <link name="tool_tip">
-      <visual>
-        <origin xyz="0 ${dedo_degrau_l/2} ${-dedo_degrau_z/2}"/>
-        <geometry><box size="${dedo_haste_x} ${dedo_degrau_l + dedo_haste_y} ${dedo_degrau_z}"/></geometry>
-        <material name="ToolColor"><color rgba="0.85 0.75 0.1 1"/></material>
-      </visual>
-      <!-- COLISÃO SÓ DA PARTE QUE SE PROJETA, não da largura visual.
-           A caixa visual acima vai de y=-5 mm a y=+25 mm (v2; na v1
-           era x=+5,2 a x=-25,2) para desenhar o L inteiro — mas isso faz ela compartilhar uma FACE
+      <!-- Sem visual próprio: a malha dedo_fixo_v3.stl do tool_rod já
+           desenha o degrau (2026-09-30). -->
+      <!-- COLISÃO SÓ DA PARTE QUE SE PROJETA, não da largura do degrau.
+           O degrau inteiro vai de y=-5 mm a y=+25 mm (v2/v3; na v1
+           era x=+5,2 a x=-25,2) — mas uma caixa assim compartilharia uma FACE
            inteira (z=0, de x=-5,2 a +5,2) com a haste do tool_rod. Duas
            faces coincidentes no mesmo corpo rígido geram contato

Commit message: feat(b166er_robot): arm_iface no URDF (Position|VelocityJointInterface) + preflight aceita o modo malha aberta
Os controladores de velocidade não inicializavam porque as transmissões
declaravam PositionJointInterface. O xacro ganha arg arm_iface, passado
pelos dois launches a partir de braco; sim_stack.sh confere
arm_openloop_sim + arm_joint_servo no lugar da ponte quando é o caso.

Co-Authored-By: Claude Fable 5.1 <noreply@anthropic.com>
Claude-Session: https://claude.ai/code/session_01P4v3ZvEh2bwom2DYHA9moN

File: src/b166er_robot/urdf/movemaster/movemaster.urdf.xacro (robot description, xacro)
@@ -740,12 +740,20 @@
          justamente câmera x ferramenta. -->
     <gazebo reference="t265_link"><material>Gazebo/Green</material></gazebo>
+    <!-- INTERFACE DAS JUNTAS no gazebo_ros_control (2026-10-06): position
+         (histórico, controladores de posição) ou velocity (braco:=malha_aberta
+         — o braço real não tem encoder; a placa só aplica velocidade/PWM, e
+         a simulação passa a executar igual). Vem do arg arm_iface, que o
+         b166er_wb.launch e o b166er_gazebo.launch passam ao xacro. -->
+    <xacro:arg name="arm_iface" default="position"/>
+    <xacro:property name="arm_hw_iface"
+                    value="${'hardware_interface/VelocityJointInterface' if '$(arg arm_iface)' == 'velocity' else 'hardware_interface/PositionJointInterface'}"/>
     <xacro:macro name="arm_transmission" params="joint_name">
       <transmission name="${joint_name}_trans">
         <type>transmission_interface/SimpleTransmission</type>
         <joint name="${joint_name}">
-          <hardwareInterface>hardware_interface/PositionJointInterface</hardwareInterface>
+          <hardwareInterface>${arm_hw_iface}</hardwareInterface>
         </joint>
         <actuator name="${joint_name}_motor">
-          <hardwareInterface>hardware_interface/PositionJointInterface</hardwareInterface>
+          <hardwareInterface>${arm_hw_iface}</hardwareInterface>
           <mechanicalReduction>1</mechanicalReduction>
         </actuator>

Commit message: feat(robot): dedo fixo monta girado +90° na castanha (JTool yaw + JTOOL_YAW na cinemática)
Marco, de trás do robô com o braço recolhido: "vc posicionou o dedo errado,
ele tem q virar 90 graus para esquerda" — "o dedo completo gira, toda a
peça". A v3 não muda; a peça inteira monta girada +90° em torno da haste.
No stow o degrau aponta para a esquerda do robô e o garfo passa a abraçar
a lingueta da castanha no eixo em que ela anda (antes ficava de lado).
checa_garra_dx passa a conferir também o yaw do JTool. Na tarefa a IK
compensa no J5 (−11° em vez de +79°); missão e YAML não mudam.

Co-Authored-By: Claude Fable 5.1 <noreply@anthropic.com>
Claude-Session: https://claude.ai/code/session_01P4v3ZvEh2bwom2DYHA9moN

File: src/b166er_robot/urdf/movemaster/movemaster.urdf.xacro (robot description, xacro)
@@ -639,6 +639,18 @@
     <xacro:property name="tool_length"
                     value="${dedo_garfo_h + dedo_afun_h + dedo_haste_l}"/>
+    <!-- MONTAGEM DA PEÇA (2026-10-07). O Marco, olhando o Gazebo com o
+         braço recolhido e de trás do robô: "vc posicionou o dedo errado,
+         ele tem q virar 90 graus para esquerda" — "o dedo completo gira,
+         toda a peça" (desenho scratchpad dedo_90_esquerda.png, leitura 2).
+         A peça v3 NÃO muda (garfo, rasgo, furos, degrau em +Y do próprio
+         frame): o que estava errado era como ela monta na castanha. O
+         yaw de +90° gira o frame tool_rod/tool_tip inteiro em torno da
+         haste; no braço recolhido o degrau passa a apontar para a
+         ESQUERDA do robô (base +Y), e o rasgo do garfo fica no eixo
+         transversal da garra (x do GripCube), que é o eixo em que a
+         castanha anda. kinematics._T_L5_TOOLTIP leva o mesmo _rotz;
+         checa_garra_dx confere os dois. -->
     <joint name="JTool" type="fixed">
-      <origin xyz="${garra_dx} 0 -0.08" rpy="0 0 0"/>
+      <origin xyz="${garra_dx} 0 -0.08" rpy="0 0 1.5708"/>
       <parent link="GripCube"/>
       <child link="tool_rod"/>

Commit message: feat(robot): limites de junta do RV-M2 retrofitado no URDF (Cerbaro, Tab. 2/3)
Eram os cursos do manual repartidos ao meio (±150/±65/±60/±110). O robô
retrofitado tem os fins de curso onde o Cerbaro os instalou (dissertação,
Tabela 2 limites, Tabela 3 home): J1 ±100°, J2 −30…+100° com o switch de
trás em 106° (16° depois da vertical, como na foto do Marco de 14 Out),
J3 −120…0° com o switch em −123° (o cotovelo só dobra para um lado),
J4 ±100°, J5 ±180°. Batentes do URDF nos switches.

Co-Authored-By: Claude Fable 5.1 <noreply@anthropic.com>
Claude-Session: https://claude.ai/code/session_01P4v3ZvEh2bwom2DYHA9moN

File: src/b166er_robot/urdf/movemaster/movemaster.urdf.xacro (robot description, xacro)
@@ -51,6 +51,10 @@
       <parent link="Base"/>
       <child link="L1"/>
-      <!-- Cintura (waist): 300° de curso total no manual, assumido ±150° -->
-      <limit upper="2.61799" lower="-2.61799" effort="30" velocity="3.14" />
+      <!-- Cintura (waist): 300° no manual, mas o robô retrofitado tem os fins
+           de curso em ±100° (Cerbaro, dissertação, Tabela 2 — chapa do
+           switch invertida para o operador atrás do robô). Batente = switch.
+           14 Out 2026: limites do Cerbaro em todas as juntas (eram os do
+           manual repartidos ao meio). -->
+      <limit upper="1.74533" lower="-1.74533" effort="30" velocity="3.14" />
       <dynamics damping="0.5" friction="0.0"/>
     </joint>
@@ -124,6 +128,9 @@
       <parent link="L1"/>
       <child link="L2"/>
-      <!-- Ombro (shoulder): 130° de curso total no manual, assumido ±65° -->
-      <limit upper="1.13446" lower="-1.13446" effort="80" velocity="2.09" />
+      <!-- Ombro (shoulder): trabalho −30° … +100° (Cerbaro, Tabela 2); o
+           switch de trás (home) fica em +106° (Tabela 3) — ~16° depois da
+           vertical, como na foto do Marco de 14 Out 2026. Batentes nos
+           switches: −31,5° (o da frente fecha em −30°) e +106°. -->
+      <limit upper="1.85005" lower="-0.54978" effort="80" velocity="2.09" />
       <dynamics damping="1.0" friction="0.0"/>
     </joint>
@@ -149,6 +156,8 @@
       <parent link="L2"/>
       <child link="L3"/>
-      <!-- Cotovelo (elbow): 120° de curso total no manual, assumido ±60° -->
-      <limit upper="1.04720" lower="-1.04720" effort="50" velocity="2.09" />
+      <!-- Cotovelo (elbow): trabalho −120° … 0° (Cerbaro, Tabela 2): o
+           cotovelo só dobra para UM lado, não há ramo. Switch (home) em
+           −123° (Tabela 3); batente de cima em +1,5° (fecha em 0°). -->
+      <limit upper="0.02618" lower="-2.14675" effort="50" velocity="2.09" />
       <dynamics damping="0.5" friction="0.0"/>
     </joint>
@@ -193,5 +202,8 @@
            tamanho do real; se não abrir, o destrava tem que vir de J2/J3
            com o punho travado. -->
-      <limit upper="1.91986" lower="-1.91986" effort="4.2" velocity="3.14" />
+      <!-- Arfagem do punho: ±100° (Cerbaro, Tabela 2 — chapa do switch
+           movida para o suporte da câmera não bater no corpo); o manual
+           diz ±110°. -->
+      <limit upper="1.74533" lower="-1.74533" effort="4.2" velocity="3.14" />
       <dynamics damping="0.3" friction="0.0"/>
     </joint>

Commit message: exp(robot): degrau de 30 mm na colisão do dedo (experimento, era 20)
Marco: "se aumentarmos o tamanho do degrau, isso ajudaria?". A sonda
mostrou o degrau curto em X (ponta 2–8 mm antes do plano do olhal) nos
casos em que a chave não abre. Só a caixa de colisão muda; a malha
visual continua com 20 mm.

Co-Authored-By: Claude Opus 5.5 <noreply@anthropic.com>
Claude-Session: https://claude.ai/code/session_01P4v3ZvEh2bwom2DYHA9moN

File: src/b166er_robot/urdf/movemaster/movemaster.urdf.xacro (robot description, xacro)
@@ -647,5 +647,10 @@
          comprimento útil que fica atravessado no furo e sustenta o
          arame do olhal. -->
-    <xacro:property name="dedo_degrau_l" value="0.020"/>
+    <!-- EXPERIMENTO 28 Out 2026 (Marco: "se aumentarmos o tamanho do
+         degrau, isso ajudaria?"): 20 → 30 mm só na COLISÃO; a malha visual
+         dedo_fixo_v3.stl continua desenhando 20 mm. Os batentes da lingueta
+         ficam a ≥ 19 mm do centro do furo em Y e o degrau a ≤ 8 mm: alongar
+         em X não muda essa folga. -->
+    <xacro:property name="dedo_degrau_l" value="0.030"/>
     <xacro:property name="dedo_degrau_z" value="0.010"/>
     <xacro:property name="tool_length"

Commit message: feat(robot): dedo v4 (REV. D) — degrau de 30 mm, malha e prancha; URDF usa a v4
gera_dedo.py ganha a versão 4 (padrão): a v3 com o degrau de 30 mm em vez
de 20, o resto igual. Gera dedo_fixo_v4.stl (24,4 cm³, bbox Y −15..35) e a
prancha cotada REV. D em docs/. O movemaster.urdf.xacro passa a desenhar
a malha v4, e colisão e visual voltam a ser a mesma peça. Para imprimir:
dedo_fixo_v4.stl, deitado, como na nota 4 da prancha.

Co-Authored-By: Claude Opus 5.5 <noreply@anthropic.com>
Claude-Session: https://claude.ai/code/session_01P4v3ZvEh2bwom2DYHA9moN

File: src/b166er_robot/urdf/movemaster/movemaster.urdf.xacro (robot description, xacro)
@@ -647,7 +647,8 @@
          comprimento útil que fica atravessado no furo e sustenta o
          arame do olhal. -->
-    <!-- EXPERIMENTO 28 Out 2026 (Marco: "se aumentarmos o tamanho do
-         degrau, isso ajudaria?"): 20 → 30 mm só na COLISÃO; a malha visual
-         dedo_fixo_v3.stl continua desenhando 20 mm. Os batentes da lingueta
+    <!-- DEGRAU DE 30 mm (dedo v4, REV. D, 30 Out 2026; Marco: "se
+         aumentarmos o tamanho do degrau, isso ajudaria?" — RELATORIO44,
+         14/25 → 17/25). Colisão e malha visual dedo_fixo_v4.stl
+         (gera_dedo.py, versão 4) agora concordam. Os batentes da lingueta
          ficam a ≥ 19 mm do centro do furo em Y e o degrau a ≤ 8 mm: alongar
          em X não muda essa folga. -->
@@ -676,5 +677,5 @@
       <!-- VISUAL = a peça impressa (dedo v3, REV. C, 2026-09-30, pedido
            do Marco: "usa o STL da v3 no visual"). meshes/movemaster/
-           dedo_fixo_v3.stl é gerado por scripts/gera_dedo.py (versao 3)
+           dedo_fixo_v4.stl é gerado por scripts/gera_dedo.py (versao 4; v3 = degrau de 20 mm)
            em mm, já no frame deste link: z=0 no topo do garfo, z=-125 na
            face de baixo do degrau, degrau em +Y (y de -5 a +25), garfo
@@ -690,5 +691,5 @@
       <visual>
         <origin xyz="0 0 0"/>
-        <geometry><mesh filename="package://b166er_robot/meshes/movemaster/dedo_fixo_v3.stl" scale="0.001 0.001 0.001"/></geometry>
+        <geometry><mesh filename="package://b166er_robot/meshes/movemaster/dedo_fixo_v4.stl" scale="0.001 0.001 0.001"/></geometry>
         <material name="ToolColor"><color rgba="0.85 0.75 0.1 1"/></material>
       </visual>
@@ -732,5 +733,5 @@
          arame do anel repousa depois da descida de 5 mm. -->
     <link name="tool_tip">
-      <!-- Sem visual próprio: a malha dedo_fixo_v3.stl do tool_rod já
+      <!-- Sem visual próprio: a malha dedo_fixo_v4.stl do tool_rod já
            desenha o degrau (2026-09-30). -->
       <!-- COLISÃO SÓ DA PARTE QUE SE PROJETA, não da largura do degrau.
